Commit message: Simulator updated to use URDF exclusively, working on ground truth publishing now

File: spirit_simulator/spirit_description/urdf/spirit_gazebo.urdf (robot description, URDF)
Before this commit: robot spirit, 17 links, 16 joints
Links:
- added link body_dummy
- added link imu_link; visual box size=0.05 0.05 0.02
Joints:
- added joint dummy_joint: type fixed, parent body_dummy, child body, origin xyz=0 0.07 0, axis 0 0 0
- added joint imu_joint: type fixed, parent body, child imu_link, origin xyz=0 0 0 rpy=0 0 0
