Commit message: Fix error in foot plan velocity, make rviz and matlab scripts real pretty

File: spirit_simulator/spirit_description/urdf/spirit_meshes_temp.urdf (robot description, URDF)
Before this commit: robot spirit, 17 links, 16 joints
Links:
- added link dummy
- added link t265_pose_frame
Joints:
- added joint body_to_t265: type fixed, parent body, child t265_pose_frame, origin xyz=0.0 0.0 0.0 rpy=0 0 0, axis 1 0 0
- added joint dummy_joint: type fixed, parent dummy, child body
