Commit message: Update sensor data passing and urdf to work on the robot

File: spirit_simulator/spirit_description/urdf/spirit_meshes.urdf (robot description, URDF)
Before this commit: robot spirit, 19 links, 18 joints
Links:
- link body: geometry collision box size=0.335 0.24 0.104; visual mesh filename=package://spirit_description/meshes/Spirit40_Body_Mesh_tran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 scale=1 1 1
- link hip0: geometry collision cylinder length=0.08 radius=0.055; visual mesh filename=package://spirit_description/meshes/Spirit40_Hip_Module_tra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 scale=1 1 1
- link hip1: geometry collision cylinder length=0.08 radius=0.055; visual mesh filename=package://spirit_description/meshes/Spirit40_Hip_Module_tra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 scale=1 1 1
- link hip2: geometry collision cylinder length=0.08 radius=0.055; visual mesh filename=package://spirit_description/meshes/Spirit40_Hip_Module_tra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 scale=1 1 1
- link hip3: geometry collision cylinder length=0.08 radius=0.055; visual mesh filename=package://spirit_description/meshes/Spirit40_Hip_Module_tra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 scale=1 1 1
- link lower0: geometry collision cylinder length=0.206 radius=0.013; visual mesh filename=package://spirit_description/meshes/Spirit40_Lower_Leg_tran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 scale=1 1 1
- link lower1: geometry collision cylinder length=0.206 radius=0.013; visual mesh filename=package://spirit_description/meshes/Spirit40_Lower_Leg_tran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 scale=1 1 1
- link lower2: geometry collision cylinder length=0.206 radius=0.013; visual mesh filename=package://spirit_description/meshes/Spirit40_Lower_Leg_tran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 scale=1 1 1
- link lower3: geometry collision cylinder length=0.206 radius=0.013; visual mesh filename=package://spirit_description/meshes/Spirit40_Lower_Leg_tran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 scale=1 1 1
- link upper0: geometry collision box size=0.206 0.022 0.055; visual mesh filename=package://spirit_description/meshes/Spirit40_Upper_leg_tran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 scale=1 1 1
- link upper1: geometry collision box size=0.206 0.022 0.055; visual mesh filename=package://spirit_description/meshes/Spirit40_Upper_leg_tran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 scale=1 1 1
- link upper2: geometry collision box size=0.206 0.022 0.055; visual mesh filename=package://spirit_description/meshes/Spirit40_Upper_leg_tran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 scale=1 1 1
- link upper3: geometry collision box size=0.206 0.022 0.055; visual mesh filename=package://spirit_description/meshes/Spirit40_Upper_leg_tran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 scale=1 1 1
Joints:
- removed joint j0
- removed joint j1
- removed joint j10
- removed joint j11
- removed joint j2
- removed joint j3
- removed joint j4
- removed joint j5
- removed joint j6
- removed joint j7
- removed joint j8
- removed joint j9
- added joint 0: type revolute, parent hip0, child upper0, origin xyz=0 0.10098 0, axis 0 -1 0, limit lower=-6.28318530718 upper=6.28318530718 effort=40 velocity=30
- added joint 1: type revolute, parent upper0, child lower0, origin xyz=-0.206 0 0, axis 0 1 0, limit lower=0 upper=3.14159265359 effort=40 velocity=30
- added joint 10: type revolute, parent body, child hip2, origin xyz=0.2263 -0.07 0, axis 1 0 0, limit lower=-0.707 upper=0.707 effort=40 velocity=30
- added joint 11: type revolute, parent body, child hip3, origin xyz=-0.2263 -0.07 0, axis 1 0 0, limit lower=-0.707 upper=0.707 effort=40 velocity=30
- added joint 2: type revolute, parent hip1, child upper1, origin xyz=0 0.10098 0, axis 0 -1 0, limit lower=-6.28318530718 upper=6.28318530718 effort=40 velocity=30
- added joint 3: type revolute, parent upper1, child lower1, origin xyz=-0.206 0 0, axis 0 1 0, limit lower=0 upper=3.14159265359 effort=40 velocity=30
- added joint 4: type revolute, parent hip2, child upper2, origin xyz=0 -0.10098 0, axis 0 -1 0, limit lower=-6.28318530718 upper=6.28318530718 effort=40 velocity=30
- added joint 5: type revolute, parent upper2, child lower2, origin xyz=-0.206 0 0, axis 0 1 0, limit lower=0 upper=3.14159265359 effort=40 velocity=30
- added joint 6: type revolute, parent hip3, child upper3, origin xyz=0 -0.10098 0, axis 0 -1 0, limit lower=-6.28318530718 upper=6.28318530718 effort=40 velocity=30
- added joint 7: type revolute, parent upper3, child lower3, origin xyz=-0.206 0 0, axis 0 1 0, limit lower=0 upper=3.14159265359 effort=40 velocity=30
- added joint 8: type revolute, parent body, child hip0, origin xyz=0.2263 0.07 0, axis 1 0 0, limit lower=-0.707 upper=0.707 effort=40 velocity=30
- added joint 9: type revolute, parent body, child hip1, origin xyz=-0.2263 0.07 0, axis 1 0 0, limit lower=-0.707 upper=0.707 effort=40 velocity=30

Commit message: Initial tail version * Tail is assembled to robot in URDF and SDF * Add tail in Gazebo control and estimator plugins * Add tail_controller nodes * Open-loop trajectory tracking toy implemented in tail_controller
* TODO: clean the variable names
* TODO: have a seperate launch file for tail
* TODO: merge to the main stream codes
* TODO: add ODrive_convertor nodes
* TODO: port MPC tail controller

File: spirit_simulator/spirit_description/urdf/spirit_meshes.urdf (robot description, URDF)
Before this commit: robot spirit, 19 links, 18 joints
Links:
- added link tail_link_0, mass 1e-03; collision sphere radius=0.02; visual sphere radius=0.02
- added link tail_link_1, mass 0.025; collision cylinder length=1 radius=0.02; visual cylinder length=1 radius=0.02
- added link tail_mass, mass 0.25; collision sphere radius=0.04; visual sphere radius=0.04
Joints:
- added joint body_tail_joint_0: type revolute, parent body, child tail_link_0, origin xyz=-0.1675 0 0.052, axis 1 0 0, limit lower=-1.79769e+308 upper=1.79769e+308 effort=40 velocity=30
- added joint body_tail_joint_1: type revolute, parent tail_link_0, child tail_link_1, origin xyz=0 0 0, axis 0 1 0, limit lower=-3.14159 upper=1.57080 effort=40 velocity=30
- added joint tail_link_mass_joint: type fixed, parent tail_link_1, child tail_mass, origin xyz=0 0 1
