Commit message: modify sdf and urdf make the tail mass and length match the real one, modify tail_controller for setpoint stablize and trajectory tracking test

File: spirit_simulator/spirit_description/urdf/spirit_meshes_tail.urdf (robot description, URDF)
Before this commit: robot spirit, 20 links, 19 joints
Links:
- link tail_link_1: geometry collision cylinder length=0.64 radius=0.02; visual cylinder length=0.64 radius=0.02
- link tail_mass: mass 0.25 -> 0.7
Joints:
- joint tail_link_mass_joint: origin xyz=0 0 1 -> xyz=0 0 0.64

Commit message: fix rviz for tail, add centralized MPC for tailed robot with global planner

File: spirit_simulator/spirit_description/urdf/spirit_meshes_tail.urdf (robot description, URDF)
Before this commit: robot spirit, 20 links, 19 joints
Links:
- link tail_link_1: geometry collision cylinder length=1 radius=0.02; visual cylinder length=1 radius=0.02
- link tail_mass: mass 0.7 -> 0.25
Joints:
- joint body_tail_joint_0: limit lower=-1.79769e+308 upper=1.79769e+308 effort=40 velocity=30 -> lower=-1.79769e+308 upper=1.79769e+308 effort=10 velocity=30
- joint body_tail_joint_1: limit lower=-3.14159 upper=1.57080 effort=40 velocity=30 -> lower=-3.14159 upper=1.57080 effort=10 velocity=30
- joint tail_link_mass_joint: origin xyz=0 0 0.64 -> xyz=0 0 1

File: spirit_simulator/spirit_description/urdf/spirit_tail.urdf (robot description, URDF)
Before this commit: robot ngr, 20 links, 19 joints
Links:
- link tail_link_1: geometry collision cylinder length=1.0 radius=0.02; visual cylinder length=1.0 radius=0.02
- link tail_mass: mass 0.7 -> 0.25
Joints:
- joint body_tail_joint_0: limit lower=-1.79769e+308 upper=1.79769e+308 effort=40 velocity=30 -> lower=-1.79769e+308 upper=1.79769e+308 effort=10 velocity=30
- joint body_tail_joint_1: limit lower=-3.14159 upper=1.57080 effort=40 velocity=30 -> lower=-3.14159 upper=1.57080 effort=10 velocity=30
- joint tail_link_mass_joint: origin xyz=0 0 0.64 -> xyz=0 0 1

Commit message: update tail physics to match the real hardware, update torque limit to make the feedback work

File: spirit_simulator/spirit_description/urdf/spirit_meshes_tail.urdf (robot description, URDF)
Before this commit: robot spirit, 20 links, 19 joints
Links:
- link tail_link_1: geometry collision cylinder length=0.54 radius=0.02; visual cylinder length=0.54 radius=0.02
- link tail_mass: mass 0.25 -> 0.6
Joints:
- joint body_tail_joint_0: limit lower=-1.79769e+308 upper=1.79769e+308 effort=10 velocity=30 -> lower=-1.79769e+308 upper=1.79769e+308 effort=15 velocity=30
- joint body_tail_joint_1: limit lower=-3.14159 upper=1.57080 effort=10 velocity=30 -> lower=-3.14159 upper=1.57080 effort=15 velocity=30
- joint tail_link_mass_joint: origin xyz=0 0 1 -> xyz=0 0 0.54

File: spirit_simulator/spirit_description/urdf/spirit_tail.urdf (robot description, URDF)
Before this commit: robot spirit, 21 links, 20 joints
Links:
- link tail_link_1: geometry collision cylinder length=0.54 radius=0.02; visual cylinder length=0.54 radius=0.02
- link tail_mass: mass 0.25 -> 0.6
Joints:
- joint body_tail_joint_0: limit lower=-1.79769e+308 upper=1.79769e+308 effort=10 velocity=30 -> lower=-1.79769e+308 upper=1.79769e+308 effort=15 velocity=30
- joint body_tail_joint_1: limit lower=-3.14159 upper=1.57080 effort=10 velocity=30 -> lower=-3.14159 upper=1.57080 effort=15 velocity=30
- joint tail_link_mass_joint: origin xyz=0 0 1 -> xyz=0 0 0.54

Commit message: real tail model, fix leg extension threshold, add logger, avoid mpc fail by feedback

File: spirit_simulator/spirit_description/urdf/spirit_meshes_tail.urdf (robot description, URDF)
Before this commit: robot spirit, 20 links, 19 joints
Joints:
- joint body_tail_joint_0: origin xyz=-0.1675 0 0.052 -> xyz=0 0 0.052
- joint body_tail_joint_1: limit lower=-3.14159 upper=1.57080 effort=15 velocity=30 -> lower=-1.79769e+308 upper=1.79769e+308 effort=15 velocity=30

File: spirit_simulator/spirit_description/urdf/spirit_tail.urdf (robot description, URDF)
Before this commit: robot spirit, 21 links, 20 joints
Joints:
- joint body_tail_joint_0: origin xyz=-0.1675 0 0.052 -> xyz=0 0 0.052
- joint body_tail_joint_1: limit lower=-3.14159 upper=1.57080 effort=15 velocity=30 -> lower=-1.79769e+308 upper=1.79769e+308 effort=15 velocity=30

Commit message: align initial time step, relax constraints

File: spirit_simulator/spirit_description/urdf/spirit_meshes_tail.urdf (robot description, URDF)
Before this commit: robot spirit, 20 links, 19 joints
Joints:
- joint body_tail_joint_0: limit lower=-1.79769e+308 upper=1.79769e+308 effort=15 velocity=30 -> lower=-1.79769e+308 upper=1.79769e+308 effort=10 velocity=30
- joint body_tail_joint_1: limit lower=-1.79769e+308 upper=1.79769e+308 effort=15 velocity=30 -> lower=-1.79769e+308 upper=1.79769e+308 effort=10 velocity=30

File: spirit_simulator/spirit_description/urdf/spirit_tail.urdf (robot description, URDF)
Before this commit: robot spirit, 21 links, 20 joints
Joints:
- joint body_tail_joint_0: limit lower=-1.79769e+308 upper=1.79769e+308 effort=15 velocity=30 -> lower=-1.79769e+308 upper=1.79769e+308 effort=10 velocity=30
- joint body_tail_joint_1: limit lower=-1.79769e+308 upper=1.79769e+308 effort=15 velocity=30 -> lower=-1.79769e+308 upper=1.79769e+308 effort=10 velocity=30

Commit message: unify initial time, adjustable terminal scale factor, more terrain

File: spirit_simulator/spirit_description/urdf/spirit_meshes_tail.urdf (robot description, URDF)
Before this commit: robot spirit, 20 links, 19 joints
Joints:
- joint body_tail_joint_0: limit lower=-1.79769e+308 upper=1.79769e+308 effort=10 velocity=30 -> lower=-1.79769e+308 upper=1.79769e+308 effort=10 velocity=1.79769e+308
- joint body_tail_joint_1: limit lower=-1.79769e+308 upper=1.79769e+308 effort=10 velocity=30 -> lower=-1.79769e+308 upper=1.79769e+308 effort=10 velocity=1.79769e+308

File: spirit_simulator/spirit_description/urdf/spirit_tail.urdf (robot description, URDF)
Before this commit: robot spirit, 21 links, 20 joints
Joints:
- joint body_tail_joint_0: limit lower=-1.79769e+308 upper=1.79769e+308 effort=10 velocity=30 -> lower=-1.79769e+308 upper=1.79769e+308 effort=10 velocity=1.79769e+308
- joint body_tail_joint_1: limit lower=-1.79769e+308 upper=1.79769e+308 effort=10 velocity=30 -> lower=-1.79769e+308 upper=1.79769e+308 effort=10 velocity=1.79769e+308
