Commit message: add centralized, distributed, decentralized tail

File: spirit_simulator/spirit_description/urdf/spirit_tail.urdf (robot description, URDF)
Before this commit: robot ngr, 20 links, 19 joints
Links:
- added link dummy
- link tail_link_1: geometry collision cylinder length=1 radius=0.02; visual cylinder length=1 radius=0.02
Joints:
- added joint dummy_joint: type fixed, parent dummy, child body
- joint 0: origin xyz=0.0 0.10098 0 -> xyz=0 0.10098 0
- joint 2: origin xyz=-0.0 0.10098 0 -> xyz=0 0.10098 0
- joint 4: origin xyz=0.0 -0.10098 0 -> xyz=0 -0.10098 0
- joint 6: origin xyz=-0.0 -0.10098 0 -> xyz=0 -0.10098 0

Commit message: bunch fix

File: spirit_simulator/spirit_description/urdf/spirit_tail.urdf (robot description, URDF)
Before this commit: robot spirit, 21 links, 20 joints
Links:
- link tail_link_0: geometry visual sphere radius=0.02
- link tail_link_1: mass 0.025 -> 1e-03; geometry visual cylinder length=0.54 radius=0.02
- link tail_mass: geometry visual sphere radius=0.04
Joints:
- joint body_tail_joint_0: limit lower=-1.79769e+308 upper=1.79769e+308 effort=10 velocity=1.79769e+308 -> lower=-1.57 upper=1.57 effort=10 velocity=1.79769e+308
- joint body_tail_joint_1: limit lower=-1.79769e+308 upper=1.79769e+308 effort=10 velocity=1.79769e+308 -> lower=-1.57 upper=1.57 effort=10 velocity=1.79769e+308
