Commit message: Unify urdf/sdf parameter loading, fix quad_mpc test bug

File: spirit_simulator/spirit_description/urdf/archive/spirit_no_meshes.urdf (robot description, URDF)
Before this commit: robot spirit, 17 links, 16 joints
Joints:
- joint 0: origin xyz=0 0.10098 0 -> xyz=0.0 0.10098 0
- joint 2: origin xyz=0 0.10098 0 -> xyz=-0.0 0.10098 0
- joint 4: origin xyz=0 -0.10098 0 -> xyz=0.0 -0.10098 0
- joint 6: origin xyz=0 -0.10098 0 -> xyz=-0.0 -0.10098 0
