Commit message: leg control checked

File: quad_simulator/spirit_description/urdf/spirit_meshes_tail.urdf (robot description, URDF)
Before this commit: robot spirit, 20 links, 19 joints
Links:
- link tail_link_1: geometry visual cylinder length=0.6706 radius=0.02
Joints:
- joint tail_link_mass_joint: origin xyz=0 0 0.6613 -> xyz=0 0 0.6706

File: quad_simulator/spirit_description/urdf/spirit_tail.urdf (robot description, URDF)
Before this commit: robot spirit, 20 links, 19 joints
Links:
- link tail_link_1: geometry visual cylinder length=0.6706 radius=0.02
Joints:
- joint tail_link_mass_joint: origin xyz=0 0 0.6613 -> xyz=0 0 0.6706
