Commit message: small changes

File: quad_simulator/spirit_description/urdf/spirit_tail.urdf (robot description, URDF)
Before this commit: robot spirit, 20 links, 19 joints
Links:
- link tail_mass: mass 0.6 -> 0.3

Commit message: fix bugs

File: quad_simulator/spirit_description/urdf/spirit_tail.urdf (robot description, URDF)
Before this commit: robot spirit, 20 links, 19 joints
Links:
- link body: mass 5.75 -> 7.388

Commit message: backup

File: quad_simulator/spirit_description/urdf/spirit_tail.urdf (robot description, URDF)
Before this commit: robot spirit, 20 links, 19 joints
Links:
- link tail_link_1: geometry visual cylinder length=0.6613 radius=0.02
- link tail_mass: mass 0.3 -> 0.2764
Joints:
- joint body_tail_joint_0: limit lower=-1.57 upper=1.57 effort=10 velocity=1.79769e+308 -> lower=-1.57 upper=1.57 effort=20 velocity=30
- joint body_tail_joint_1: limit lower=-1.57 upper=1.57 effort=10 velocity=1.79769e+308 -> lower=-1.57 upper=1.57 effort=20 velocity=30
- joint tail_link_mass_joint: origin xyz=0 0 0.54 -> xyz=0 0 0.6613

Commit message: add old flat terrain assumption codes, rewrite swing foot trajectory computation, add temporary foothold history for missing contact, add old swing leg codes for missing foot

File: quad_simulator/spirit_description/urdf/spirit_tail.urdf (robot description, URDF)
Before this commit: robot spirit, 20 links, 19 joints
Joints:
- joint body_tail_joint_0: limit lower=-1.57 upper=1.57 effort=20 velocity=30 -> lower=-1.57 upper=1.57 effort=10 velocity=30
- joint body_tail_joint_1: limit lower=-1.57 upper=1.57 effort=20 velocity=30 -> lower=-1.57 upper=1.57 effort=10 velocity=30

Commit message: State machine improve

File: quad_simulator/spirit_description/urdf/spirit_tail.urdf (robot description, URDF)
Before this commit: robot spirit, 20 links, 19 joints
Joints:
- joint body_tail_joint_0: limit lower=-1.57 upper=1.57 effort=10 velocity=30 -> lower=-1.57 upper=1.57 effort=35 velocity=1000000
- joint body_tail_joint_1: limit lower=-1.57 upper=1.57 effort=10 velocity=30 -> lower=-1.57 upper=1.57 effort=35 velocity=1000000

Commit message: Final

File: quad_simulator/spirit_description/urdf/spirit_tail.urdf (robot description, URDF)
Before this commit: robot spirit, 20 links, 19 joints
Links:
- link tail_link_1: geometry visual cylinder length=0.8816 radius=0.02
Joints:
- joint tail_link_mass_joint: origin xyz=0 0 0.6706 -> xyz=0 0 0.8816
