Commit message: Put identified leg inertial parameters into spirit.sdf and spirit.urdf files.

File: quad_simulator/spirit_description/urdf/spirit_gazebo.urdf (robot description, URDF)
Before this commit: robot spirit, 19 links, 18 joints
Links:
- link lower0: mass 0.075 -> 0.096
- link lower1: mass 0.075 -> 0.096
- link lower2: mass 0.075 -> 0.096
- link lower3: mass 0.075 -> 0.096
- link upper0: mass 0.775 -> 0.792
- link upper1: mass 0.775 -> 0.792
- link upper2: mass 0.775 -> 0.792
- link upper3: mass 0.775 -> 0.792

Commit message: Revert to before merge attempt, commit 55fc5a2

File: quad_simulator/spirit_description/urdf/spirit_gazebo.urdf (robot description, URDF)
Before this commit: robot spirit, 19 links, 18 joints
Links:
- link lower0: mass 0.096 -> 0.075
- link lower1: mass 0.096 -> 0.075
- link lower2: mass 0.096 -> 0.075
- link lower3: mass 0.096 -> 0.075
- link upper0: mass 0.792 -> 0.775
- link upper1: mass 0.792 -> 0.775
- link upper2: mass 0.792 -> 0.775
- link upper3: mass 0.792 -> 0.775
