Commit message: Modified estimater plugin to work with new xacro templates. Removed some of the dummy links. Added an alternative xacro template, which split the robot along the longer center line.

File: quad_simulator/testbot_description/sdf_mesh/spine_robot_alt.urdf.xacro (robot description, xacro)
@@ -65,19 +65,19 @@
 	<xacro:property name="jointEffortLimit" value="40"/>
 	<!-- Additional limb: tail or neck-->
-	<xacro:property name="spineDirection" value="0 1 0"/>
-	<xacro:property name="spineLB" value="-0.4"/>
-	<xacro:property name="spineUB" value="0.4"/>
+	<xacro:property name="spineDirection" value="1 0 0"/>
+	<xacro:property name="spineLB" value="-1"/>
+	<xacro:property name="spineUB" value="1"/>
 	<!-- Body -->
 	<link name="body">
 		<visual>
-			<origin rpy="0 0 0" xyz="${bodyLength/4} 0 0"/>
+			<origin rpy="0 0 0" xyz="0 ${bodyWidth/4} 0"/>
 			<geometry>
-				<box size="${bodyLength/2} ${bodyWidth} ${bodyHeight}"/>
+				<box size="${bodyLength} ${bodyWidth/2} ${bodyHeight}"/>
 			</geometry>
 			<material name="darkgray"/>
 		</visual>
 		<inertial>
-			<origin rpy="0 0 0" xyz="${bodyLength/4} 0 0"/>
-			<mass value="${bodyMass}"/>
+			<origin rpy="0 0 0" xyz="0 ${bodyWidth/4} 0"/>
+			<mass value="${bodyMass/2}"/>
 			<!-- Uniform box -->
 			<!-- <inertia ixx="1/12*${bodyMass}*(${bodyWidth}*${bodyWidth} + ${bodyHeight}*${bodyHeight})"  ixy="0"  ixz="0" iyy="1/12*${bodyMass}*(${bodyLength}*${bodyLength} + ${bodyHeight}*${bodyHeight})" iyz="0" izz="1/12*${bodyMass}*(${bodyLength}*${bodyLength} + ${bodyWidth}*${bodyWidth})"/> -->
@@ -86,5 +86,5 @@
 		<!-- Just copy geometry for collision -->
 		<collision>
-			<origin rpy="0 0 0" xyz="${bodyLength/4} 0 0"/>
+			<origin rpy="0 0 0" xyz="0 ${bodyWidth/4} 0"/>
 			<geometry>
 				<box size="${bodyLength/2} ${bodyWidth} ${bodyHeight}"/>
@@ -99,13 +99,13 @@
 	<link name="body2">
 		<visual>
-			<origin rpy="0 0 0" xyz="${-bodyLength/4} 0 0"/>
+			<origin rpy="0 0 0" xyz="0 ${-bodyWidth/4} 0"/>
 			<geometry>
-				<box size="${bodyLength/2} ${bodyWidth} ${bodyHeight}"/>
+				<box size="${bodyLength} ${bodyWidth/2} ${bodyHeight}"/>
 			</geometry>
 			<material name="darkgray"/>
 		</visual>
 		<inertial>
-			<origin rpy="0 0 0" xyz="${-bodyLength/4} 0 0"/>
-			<mass value="${bodyMass}"/>
+			<origin rpy="0 0 0" xyz="0 ${-bodyWidth/4} 0"/>
+			<mass value="${bodyMass/2}"/>
 			<!-- Uniform box -->
 			<!-- <inertia ixx="1/12*${bodyMass}*(${bodyWidth}*${bodyWidth} + ${bodyHeight}*${bodyHeight})"  ixy="0"  ixz="0" iyy="1/12*${bodyMass}*(${bodyLength}*${bodyLength} + ${bodyHeight}*${bodyHeight})" iyz="0" izz="1/12*${bodyMass}*(${bodyLength}*${bodyLength} + ${bodyWidth}*${bodyWidth})"/> -->
@@ -114,5 +114,5 @@
 		<!-- Just copy geometry for collision -->
 		<collision>
-			<origin rpy="0 0 0" xyz="${-bodyLength/4} 0 0"/>
+			<origin rpy="0 0 0" xyz="0 ${-bodyWidth/4} 0"/>
 			<geometry>
 				<box size="${bodyLength/2} ${bodyWidth} ${bodyHeight}"/>
@@ -343,6 +343,6 @@
 	</xacro:macro>
 	<xacro:leg suffix="0" hipJointName="0" kneeJointName="1" abductionJointName="8" front="1" left="1" hipJointLowerLimit="${-2*pi}" hipJointUpperLimit="${2*pi}" color="darkgray" bodylink="body"/>
- 	<xacro:leg suffix="1" hipJointName="2" kneeJointName="3" abductionJointName="9" front="-1" left="1" hipJointLowerLimit="${-2*pi}" hipJointUpperLimit="${2*pi}" color="darkgray" bodylink="body2"/>
- 	<xacro:leg suffix="2" hipJointName="4" kneeJointName="5" abductionJointName="10" front="1" left="-1" hipJointLowerLimit="${-2*pi}" hipJointUpperLimit="${2*pi}" color="red" bodylink="body"/>
+ 	<xacro:leg suffix="1" hipJointName="2" kneeJointName="3" abductionJointName="9" front="-1" left="1" hipJointLowerLimit="${-2*pi}" hipJointUpperLimit="${2*pi}" color="darkgray" bodylink="body"/>
+ 	<xacro:leg suffix="2" hipJointName="4" kneeJointName="5" abductionJointName="10" front="1" left="-1" hipJointLowerLimit="${-2*pi}" hipJointUpperLimit="${2*pi}" color="red" bodylink="body2"/>
  	<xacro:leg suffix="3" hipJointName="6" kneeJointName="7" abductionJointName="11" front="-1" left="-1" hipJointLowerLimit="${-2*pi}" hipJointUpperLimit="${2*pi}" color="darkgray" bodylink="body2"/>
   	<link name="imu::link">
