Commit message: Migrated the melodic_devel_designOpt to noetic by changing some setup_deps.sh files, still need testing. Added a new package quad_pybullet, an interface to pybullet simulator as an alternative to Gazebo. Still in progress.

File: quad_simulator/testbot_description/sdf_mesh/test.urdf (robot description, URDF)
Before this commit: robot spirit, 18 links, 17 joints
Links:
- added link body2, mass 5.75; collision box size=0.1675 0.24 0.104; visual box size=0.1675 0.24 0.104
- link body: geometry collision box size=0.1675 0.24 0.104; visual box size=0.1675 0.24 0.104
Joints:
- added joint spine: type revolute, parent body, child body2, origin xyz=0 0 0, axis 0 1 0, limit lower=-0.4 upper=0.4 effort=35 velocity=1000000
- joint 10: origin xyz=0.2225 -0.062 0 -> xyz=0.2225 -0.061999999999999986 0
- joint 11: origin xyz=-0.2225 -0.062 0 -> xyz=-0.2225 -0.061999999999999986 0; parent body -> body2
- joint 8: origin xyz=0.2225 0.062 0 -> xyz=0.2225 0.061999999999999986 0
- joint 9: origin xyz=-0.2225 0.062 0 -> xyz=-0.2225 0.061999999999999986 0; parent body -> body2
