Commit message: ylo2 robot integration

File: quad_simulator/ylo2_description/xacro/const.xacro (robot description, xacro)
@@ -3,58 +3,59 @@
     <!-- Constants for robot dimensions -->
     <xacro:property name="PI" value="3.1415926535897931"/>
-    <!-- simplified collision value for ylo2 -->
-    <!-- body -->
+    <xacro:property name="stick_mass" value="0.00001"/>
+    <xacro:property name="body_center_x" value="0.0"/>
+    <xacro:property name="body_center_y" value="0.0"/>
+    <xacro:property name="body_center_z" value="0.0"/>
+    <!-- simplified collision value -->
     <xacro:property name="trunk_width" value="0.350"/>
-    <xacro:property name="trunk_length" value="0.569125"/>
-    <xacro:property name="trunk_height" value="0.148521"/>
-    <!-- adjust center of robot -->
-    <xacro:property name="trunk_offset_x" value="0.0"/>
-    <xacro:property name="trunk_offset_y" value="0.0"/>
-    <xacro:property name="abab_motors_offset_z" value="0.0"/>
-    <!-- leg params. -->
+    <xacro:property name="trunk_length" value="0.57"/>
+    <xacro:property name="trunk_height" value="0.149"/>
     <xacro:property name="hip_radius" value="0.050"/>
-    <xacro:property name="hip_length" value="0.418"/>
-    <xacro:property name="upperleg_shoulder_radius" value="0.044"/>
-    <xacro:property name="upperleg_shoulder_length" value="0.08"/>
-    <xacro:property name="upperleg_width" value="0.0374"/>
-    <xacro:property name="upperleg_height" value="0.043"/>
-    <xacro:property name="lowerleg_width" value="0.0208"/>
-    <xacro:property name="lowerleg_height" value="0.016"/>
+    <xacro:property name="hip_length" value="0.06"/>
+    <xacro:property name="thigh_shoulder_radius" value="0.044"/>
+    <xacro:property name="thigh_shoulder_length" value="0.08"/>
+    <xacro:property name="thigh_width" value="0.0374"/>
+    <xacro:property name="thigh_height" value="0.043"/>
+    <xacro:property name="calf_width" value="0.0208"/>
+    <xacro:property name="calf_height" value="0.016"/>
     <xacro:property name="foot_radius" value="0.0265"/>
     <xacro:property name="stick_radius" value="0.01"/>
     <xacro:property name="stick_length" value="0.2"/>
+    <xacro:property name="toe_friction" value="0.2"/>
+    <xacro:property name="toe_lateral_friction" value="0.2"/>
+    <xacro:property name="toe_stiffness" value="30000.0"/>
+    <xacro:property name="toe_damping" value="1000.0"/>
     <!-- kinematic value -->
-    <xacro:property name="upperleg_offset" value="0.092"/> <!-- decalage lateral HIP -> upper_leg - lateral difference between HIP and upper_leg -->
-    <xacro:property name="upperleg_length" value="0.215427"/> <!-- upper leg size, from HIP axis, to lower leg axis-->
-    <xacro:property name="lowerleg_length" value="0.229819"/> <!-- lower leg size, from lower leg axis to end foot -->
+    <xacro:property name="thigh_offset" value="0.02"/><!-- decalage lateral HIP -> upper_leg - lateral difference between HIP and upper_leg -->
+    <xacro:property name="thigh_length" value="0.201"/><!-- upper leg size, from HIP axis, to lower leg axis-->
+    <xacro:property name="calf_length" value="0.230"/><!-- lower leg size, from lower leg axis to end foot -->
     <!-- leg offset from trunk center value -->
-    <xacro:property name="leg_offset_x" value="${0.387/2}"/> <!-- ecart centres HIP avant/arriere - HIP distance front/back -->
-    <xacro:property name="leg_offset_y" value="${0.1144/2}"/> <!-- ecart centres HIP gauche/droite - HIP distance left/right-->
-    <xacro:property name="leg_offset_z" value="-0.023"/> <!-- decalage hauteur axes pattes/abad - vertical difference HIP -> ABAD -->
-    <xacro:property name="trunk_offset_z" value="0.01675"/>
+    <xacro:property name="leg_offset_x" value="${0.135}"/><!-- ecart centres HIP avant/arriere - HIP distance front/back -->
+    <xacro:property name="leg_offset_y" value="${0.057}"/><!-- ecart centres HIP gauche/droite - HIP distance left/right-->
+    <xacro:property name="leg_offset_z" value="${0.024}"/>
+    <xacro:property name="trunk_offset_z" value="0.01675"/><!-- decalage hauteur axes pattes/abad - vertical difference HIP -> ABAD -->
     <xacro:property name="hip_offset" value="0.083"/>
     <!-- joint limits -->
     <xacro:property name="damping" value="0"/>
     <xacro:property name="friction" value="0"/>
-    <xacro:property name="hip_position_max" value="${70*PI/180.0}"/>
-    <xacro:property name="hip_position_min" value="${-70*PI/180.0}"/>
-    <xacro:property name="hip_velocity_max" value="20"/>
-    <xacro:property name="hip_torque_max" value="14"/>
-    <xacro:property name="upperleg_velocity_max" value="20"/>
-    <xacro:property name="upperleg_torque_max" value="14"/>
-    <xacro:property name="lowerleg_position_max" value="${-37*PI/180.0}"/>
-    <xacro:property name="lowerleg_position_min" value="${-159*PI/180.0}"/>
-    <xacro:property name="lowerleg_velocity_max" value="15"/>
-    <xacro:property name="lowerleg_torque_max" value="14"/>
-    <!-- dynamics inertial value
-            | ixx ixy ixz |
-            | ixy iyy iyz |
-            | ixz iyz izz | -->
+    <xacro:property name="hip_max" value="46"/>
+    <xacro:property name="hip_min" value="-46"/>
+    <xacro:property name="hip_velocity_max" value="21"/>
+    <xacro:property name="hip_torque_max" value="33.5"/>
+    <xacro:property name="thigh_max" value="360"/>
+    <xacro:property name="thigh_min" value="-360"/>
+    <xacro:property name="thigh_velocity_max" value="21"/>
+    <xacro:property name="thigh_torque_max" value="33.5"/>
+    <xacro:property name="calf_max" value="360"/>
+    <xacro:property name="calf_min" value="-360"/>
+    <xacro:property name="calf_velocity_max" value="21"/>
+    <xacro:property name="calf_torque_max" value="33.5"/>
+    <!-- dynamics inertial value -->
     <!-- trunk -->
-    <xacro:property name="trunk_mass" value="4.950"/> <!-- 3.128 kg-->
-    <xacro:property name="trunk_com_x" value="0.02"/> <!-- 0.000252 -->
-    <xacro:property name="trunk_com_y" value="0.00194"/> <!-- 0.000194 -->
-    <xacro:property name="trunk_com_z" value="0.0"/> <!-- 0.000194 -->
-    <xacro:property name="trunk_ixx" value="0.01585"/>
+    <xacro:property name="trunk_mass" value="6.0"/>
+    <xacro:property name="trunk_com_x" value="0.02"/>
+    <xacro:property name="trunk_com_y" value="0.00194"/>
+    <xacro:property name="trunk_com_z" value="0.0"/>
+    <xacro:property name="trunk_ixx" value="0.0158533"/>
     <xacro:property name="trunk_ixy" value="-0.0001332"/>
     <xacro:property name="trunk_ixz" value="-0.0002403"/>
@@ -73,26 +74,26 @@
     <xacro:property name="hip_iyz" value="0.000000215"/>
     <xacro:property name="hip_izz" value="0.0004707"/>
-    <!-- upperleg -->
-    <xacro:property name="upperleg_mass" value="1.080"/>
-    <xacro:property name="upperleg_com_x" value="-0.000684"/>
-    <xacro:property name="upperleg_com_y" value="-0.010999"/>
-    <xacro:property name="upperleg_com_z" value="-0.035487"/>
-    <xacro:property name="upperleg_ixx" value="0.005666803"/>
-    <xacro:property name="upperleg_ixy" value="0.000003597"/>
-    <xacro:property name="upperleg_ixz" value="0.000491446"/>
-    <xacro:property name="upperleg_iyy" value="0.005847229"/>
-    <xacro:property name="upperleg_iyz" value="0.000010086"/>
-    <xacro:property name="upperleg_izz" value="0.000369811"/>
-    <!-- lowerleg -->
-    <xacro:property name="lowerleg_mass" value="0.265"/>
-    <xacro:property name="lowerleg_com_x" value="0.000252"/>
-    <xacro:property name="lowerleg_com_y" value="0.000194"/>
-    <xacro:property name="lowerleg_com_z" value="-0.05192"/>
-    <xacro:property name="lowerleg_ixx" value="0.0004583"/>
-    <xacro:property name="lowerleg_ixy" value="-0.000000095"/>
-    <xacro:property name="lowerleg_ixz" value="0.000026512"/>
-    <xacro:property name="lowerleg_iyy" value="0.0004675"/>
-    <xacro:property name="lowerleg_iyz" value="0.000000277"/>
-    <xacro:property name="lowerleg_izz" value="0.000029145"/>
+    <!-- thigh / upperleg -->
+    <xacro:property name="thigh_mass" value="1.080"/>
+    <xacro:property name="thigh_com_x" value="-0.000684"/>
+    <xacro:property name="thigh_com_y" value="-0.010999"/>
+    <xacro:property name="thigh_com_z" value="-0.035487"/>
+    <xacro:property name="thigh_ixx" value="0.005666803"/>
+    <xacro:property name="thigh_ixy" value="0.000003597"/>
+    <xacro:property name="thigh_ixz" value="0.000491446"/>
+    <xacro:property name="thigh_iyy" value="0.005847229"/>
+    <xacro:property name="thigh_iyz" value="0.000010086"/>
+    <xacro:property name="thigh_izz" value="0.000369811"/>
+    <!-- calf / lowerleg -->
+    <xacro:property name="calf_mass" value="0.265"/>
+    <xacro:property name="calf_com_x" value="0.000252"/>
+    <xacro:property name="calf_com_y" value="0.000194"/>
+    <xacro:property name="calf_com_z" value="-0.05192"/>
+    <xacro:property name="calf_ixx" value="0.0004583"/>
+    <xacro:property name="calf_ixy" value="-0.000000095"/>
+    <xacro:property name="calf_ixz" value="0.000026512"/>
+    <xacro:property name="calf_iyy" value="0.0004675"/>
+    <xacro:property name="calf_iyz" value="0.000000277"/>
+    <xacro:property name="calf_izz" value="0.000029145"/>
     <!-- foot -->
     <xacro:property name="foot_mass" value="0.078"/>

File: quad_simulator/ylo2_description/xacro/gazebo.xacro (robot description, xacro)
@@ -4,5 +4,5 @@
     <gazebo>
         <plugin name="gazebo_ros_control" filename="libgazebo_ros_control.so">
-            <robotNamespace>/a1</robotNamespace>
+            <robotNamespace>/ylo2</robotNamespace>
             <robotSimType>gazebo_ros_control/DefaultRobotHWSim</robotSimType>
         </plugin>
