Commit message: Working commit of quad_pybullet. Ignore the testbot description.

File: quad_simulator/testbot_description/from18/test.urdf (robot description, URDF)
Before this commit: robot spirit, 19 links, 18 joints
Links:
- removed link body2
- link body: geometry collision box size=0.335 0.24 0.1; visual box size=0.335 0.24 0.1
Joints:
- removed joint spine
- joint 10: origin xyz=0.2225 -0.061999999999999986 0 -> xyz=0.2225 -0.062 0
- joint 11: origin xyz=-0.2225 -0.061999999999999986 0 -> xyz=-0.2225 -0.062 0; parent body2 -> body
- joint 8: origin xyz=0.2225 0.061999999999999986 0 -> xyz=0.2225 0.062 0
- joint 9: origin xyz=-0.2225 0.061999999999999986 0 -> xyz=-0.2225 0.062 0; parent body2 -> body

File: quad_simulator/testbot_description/urdf/test.urdf (robot description, URDF)
Before this commit: robot spirit, 19 links, 18 joints
Links:
- removed link text_left
- removed link text_right
- added link body2, mass 5.75; collision box size=0.1675 0.24 0.104; visual box size=0.1675 0.24 0.104
- added link imu::link, mass 0.001; visual sphere radius=0.02
- link body: mass 7.388 -> 5.75; geometry collision box size=0.1675 0.24 0.104; visual box size=0.1675 0.24 0.104
- link hip0: geometry collision box size=0.11 0.11 0.08; visual cylinder length=0.08 radius=0.055
- link hip1: geometry collision box size=0.11 0.11 0.08; visual cylinder length=0.08 radius=0.055
- link hip2: geometry collision box size=0.11 0.11 0.08; visual cylinder length=0.08 radius=0.055
- link hip3: geometry collision box size=0.11 0.11 0.08; visual cylinder length=0.08 radius=0.055
- link lower0: mass 0.096 -> 0.075
- link lower1: mass 0.096 -> 0.075
- link lower2: mass 0.096 -> 0.075
- link lower3: mass 0.096 -> 0.075
- link upper0: mass 0.792 -> 0.775
- link upper1: mass 0.792 -> 0.775
- link upper2: mass 0.792 -> 0.775
- link upper3: mass 0.792 -> 0.775
Joints:
- removed joint cmu_text_left
- removed joint cmu_text_right
- added joint imu_joint: type fixed, parent body, child imu::link
- added joint spine: type revolute, parent body, child body2, origin xyz=0 0 0, axis 0 1 0, limit lower=-0.4 upper=0.4 effort=35 velocity=1000000
- joint 0: limit lower=-1.57 upper=3.14 effort=21 velocity=37.7 -> lower=-6.28318530718 upper=6.28318530718 effort=40 velocity=30
- joint 1: limit lower=-6.28 upper=6.28 effort=32 velocity=25.1 -> lower=0 upper=3.14159265359 effort=40 velocity=30
- joint 10: limit lower=-0.707 upper=0.707 effort=21 velocity=37.7 -> lower=-0.707 upper=0.707 effort=40 velocity=30; origin xyz=0.2263 -0.07 0 -> xyz=0.2225 -0.061999999999999986 0
- joint 11: limit lower=-0.707 upper=0.707 effort=21 velocity=37.7 -> lower=-0.707 upper=0.707 effort=40 velocity=30; origin xyz=-0.2263 -0.07 0 -> xyz=-0.2225 -0.061999999999999986 0; parent body -> body2
- joint 2: limit lower=-3.14 upper=1.57 effort=21 velocity=37.7 -> lower=-6.28318530718 upper=6.28318530718 effort=40 velocity=30
- joint 3: limit lower=-6.28 upper=6.28 effort=32 velocity=25.1 -> lower=0 upper=3.14159265359 effort=40 velocity=30
- joint 4: limit lower=-1.57 upper=3.14 effort=21 velocity=37.7 -> lower=-6.28318530718 upper=6.28318530718 effort=40 velocity=30
- joint 5: limit lower=-6.28 upper=6.28 effort=32 velocity=25.1 -> lower=0 upper=3.14159265359 effort=40 velocity=30
- joint 6: limit lower=-3.14 upper=1.57 effort=21 velocity=37.7 -> lower=-6.28318530718 upper=6.28318530718 effort=40 velocity=30
- joint 7: limit lower=-6.28 upper=6.28 effort=32 velocity=25.1 -> lower=0 upper=3.14159265359 effort=40 velocity=30
- joint 8: limit lower=-0.707 upper=0.707 effort=21 velocity=37.7 -> lower=-0.707 upper=0.707 effort=40 velocity=30; origin xyz=0.2263 0.07 0 -> xyz=0.2225 0.061999999999999986 0
- joint 9: limit lower=-0.707 upper=0.707 effort=21 velocity=37.7 -> lower=-0.707 upper=0.707 effort=40 velocity=30; origin xyz=-0.2263 0.07 0 -> xyz=-0.2225 0.061999999999999986 0; parent body -> body2
