Commit message: fix urdf/sdf

File: quad_simulator/cyberdog_description/urdf/cyberdog.urdf (robot description, URDF)
Before this commit: robot cyberdog_description, 19 links, 18 joints
Joints:
- removed joint floating_body
- added joint floating_base: type fixed, parent body, child trunk, origin xyz=0 0 0 rpy=0 0 0

Commit message: modify cyberdog

File: quad_simulator/cyberdog_description/urdf/cyberdog.urdf (robot description, URDF)
Before this commit: robot cyberdog_description, 19 links, 18 joints
Links:
- link toe0: mass 0.00 -> 0.06
- link toe2: mass 0.00 -> 0.06
- link toe3: mass 0.00 -> 0.06

Commit message: change foot mass to 0.026

File: quad_simulator/cyberdog_description/urdf/cyberdog.urdf (robot description, URDF)
Before this commit: robot cyberdog_description, 19 links, 18 joints
Links:
- link toe0: mass 0.06 -> 0.026
- link toe1: mass 0.06 -> 0.026
- link toe2: mass 0.06 -> 0.026
- link toe3: mass 0.06 -> 0.026
