Commit message: urdf and sim updates

File: quad_simulator/testbot_description/urdf/pitch.urdf (robot description, URDF)
Before this commit: robot spirit, 19 links, 18 joints
Joints:
- joint spine: axis 0 0 1 -> 0 1 0; limit lower=-0.0 upper=-0.0 effort=35 velocity=1000000 -> lower=-0.4 upper=0.4 effort=35 velocity=1000000

File: quad_simulator/testbot_description/urdf/roll.urdf (robot description, URDF)
Before this commit: robot spirit, 19 links, 18 joints
Links:
- link body: mass 5.75 -> 2.875; geometry collision box size=0.1675 0.24 0.104; visual box size=0.335 0.12 0.104
- link body2: mass 5.75 -> 2.875; geometry collision box size=0.1675 0.24 0.104; visual box size=0.335 0.12 0.104
Joints:
- joint 10: parent body -> body2
- joint 9: parent body2 -> body
- joint spine: axis 0 0 1 -> 1 0 0; limit lower=-0.0 upper=-0.0 effort=35 velocity=1000000 -> lower=-1 upper=1 effort=35 velocity=1000000
