Commit message: a1 is working

File: quad_simulator/a1_description/urdf/a1.urdf (robot description, URDF)
Before this commit: robot a1_description, 23 links, 22 joints
Links:
- removed link FL_calf
- removed link FL_foot
- removed link FL_hip
- removed link FL_thigh
- removed link FL_thigh_shoulder
- removed link FR_calf
- removed link FR_foot
- removed link FR_hip
- removed link FR_thigh
- removed link FR_thigh_shoulder
- removed link RL_calf
- removed link RL_foot
- removed link RL_hip
- removed link RL_thigh
- removed link RL_thigh_shoulder
- removed link RR_calf
- removed link RR_foot
- removed link RR_hip
- removed link RR_thigh
- removed link RR_thigh_shoulder
- removed link base
- added link body; visual box size=0.001 0.001 0.001
- added link hip0, mass 0.696; collision cylinder length=0.04 radius=0.046; visual mesh filename=package://a1_description/meshes/hip.dae scale=1 1 1
- added link hip1, mass 0.696; collision cylinder length=0.04 radius=0.046; visual mesh filename=package://a1_description/meshes/hip.dae scale=1 1 1
- added link hip2, mass 0.696; collision cylinder length=0.04 radius=0.046; visual mesh filename=package://a1_description/meshes/hip.dae scale=1 1 1
- added link hip3, mass 0.696; collision cylinder length=0.04 radius=0.046; visual mesh filename=package://a1_description/meshes/hip.dae scale=1 1 1
- added link lower0, mass 0.166; collision box size=0.2 0.016 0.016; visual mesh filename=package://a1_description/meshes/calf.dae scale=1 1 1
- added link lower1, mass 0.166; collision box size=0.2 0.016 0.016; visual mesh filename=package://a1_description/meshes/calf.dae scale=1 1 1
- added link lower2, mass 0.166; collision box size=0.2 0.016 0.016; visual mesh filename=package://a1_description/meshes/calf.dae scale=1 1 1
- added link lower3, mass 0.166; collision box size=0.2 0.016 0.016; visual mesh filename=package://a1_description/meshes/calf.dae scale=1 1 1
- added link thigh_shoulder0; collision cylinder length=0.032 radius=0.041
- added link thigh_shoulder1; collision cylinder length=0.032 radius=0.041
- added link thigh_shoulder2; collision cylinder length=0.032 radius=0.041
- added link thigh_shoulder3; collision cylinder length=0.032 radius=0.041
- added link toe0, mass 0.06; collision sphere radius=0.02; visual sphere radius=0.01
- added link toe1, mass 0.06; collision sphere radius=0.02; visual sphere radius=0.01
- added link toe2, mass 0.06; collision sphere radius=0.02; visual sphere radius=0.01
- added link toe3, mass 0.06; collision sphere radius=0.02; visual sphere radius=0.01
- added link upper0, mass 1.013; collision box size=0.2 0.0245 0.034; visual mesh filename=package://a1_description/meshes/thigh.dae scale=1 1 1
- added link upper1, mass 1.013; collision box size=0.2 0.0245 0.034; visual mesh filename=package://a1_description/meshes/thigh.dae scale=1 1 1
- added link upper2, mass 1.013; collision box size=0.2 0.0245 0.034; visual mesh filename=package://a1_description/meshes/thigh_mirror.dae scale=1 1 1
- added link upper3, mass 1.013; collision box size=0.2 0.0245 0.034; visual mesh filename=package://a1_description/meshes/thigh_mirror.dae scale=1 1 1
Joints:
- removed joint FL_calf_joint
- removed joint FL_foot_fixed
- removed joint FL_hip_fixed
- removed joint FL_hip_joint
- removed joint FL_thigh_joint
- removed joint FR_calf_joint
- removed joint FR_foot_fixed
- removed joint FR_hip_fixed
- removed joint FR_hip_joint
- removed joint FR_thigh_joint
- removed joint RL_calf_joint
- removed joint RL_foot_fixed
- removed joint RL_hip_fixed
- removed joint RL_hip_joint
- removed joint RL_thigh_joint
- removed joint RR_calf_joint
- removed joint RR_foot_fixed
- removed joint RR_hip_fixed
- removed joint RR_hip_joint
- removed joint RR_thigh_joint
- added joint 0: type revolute, parent hip0, child upper0, origin xyz=0 0.0838 0 rpy=0 1.57079632679 0, axis 0 -1 0, limit lower=-6.28318530718 upper=6.28318530718 effort=33.5 velocity=21
- added joint 1: type revolute, parent upper0, child lower0, origin xyz=0 0 -0.2 rpy=0 -3.14159265359 0, axis 0 1 0, limit lower=-6.28318530718 upper=6.28318530718 effort=33.5 velocity=21
- added joint 10: type revolute, parent trunk, child hip2, origin xyz=0.1805 -0.047 0 rpy=0 0 0, axis 1 0 0, limit lower=-0.802851455917 upper=0.802851455917 effort=33.5 velocity=21
- added joint 11: type revolute, parent trunk, child hip3, origin xyz=-0.1805 -0.047 0 rpy=0 0 0, axis 1 0 0, limit lower=-0.802851455917 upper=0.802851455917 effort=33.5 velocity=21
- added joint 2: type revolute, parent hip1, child upper1, origin xyz=0 0.0838 0 rpy=0 1.57079632679 0, axis 0 -1 0, limit lower=-6.28318530718 upper=6.28318530718 effort=33.5 velocity=21
- added joint 3: type revolute, parent upper1, child lower1, origin xyz=0 0 -0.2 rpy=0 -3.14159265359 0, axis 0 1 0, limit lower=-6.28318530718 upper=6.28318530718 effort=33.5 velocity=21
- added joint 4: type revolute, parent hip2, child upper2, origin xyz=0 -0.0838 0 rpy=0 1.57079632679 0, axis 0 -1 0, limit lower=-6.28318530718 upper=6.28318530718 effort=33.5 velocity=21
- added joint 5: type revolute, parent upper2, child lower2, origin xyz=0 0 -0.2 rpy=0 -3.14159265359 0, axis 0 1 0, limit lower=-6.28318530718 upper=6.28318530718 effort=33.5 velocity=21
- added joint 6: type revolute, parent hip3, child upper3, origin xyz=0 -0.0838 0 rpy=0 1.57079632679 0, axis 0 -1 0, limit lower=-6.28318530718 upper=6.28318530718 effort=33.5 velocity=21
- added joint 7: type revolute, parent upper3, child lower3, origin xyz=0 0 -0.2 rpy=0 -3.14159265359 0, axis 0 1 0, limit lower=-6.28318530718 upper=6.28318530718 effort=33.5 velocity=21
- added joint 8: type revolute, parent trunk, child hip0, origin xyz=0.1805 0.047 0 rpy=0 0 0, axis 1 0 0, limit lower=-0.802851455917 upper=0.802851455917 effort=33.5 velocity=21
- added joint 9: type revolute, parent trunk, child hip1, origin xyz=-0.1805 0.047 0 rpy=0 0 0, axis 1 0 0, limit lower=-0.802851455917 upper=0.802851455917 effort=33.5 velocity=21
- added joint hip0_fixed: type fixed, parent hip0, child thigh_shoulder0, origin xyz=0 0.081 0 rpy=0 0 0
- added joint hip1_fixed: type fixed, parent hip1, child thigh_shoulder1, origin xyz=0 0.081 0 rpy=0 0 0
- added joint hip2_fixed: type fixed, parent hip2, child thigh_shoulder2, origin xyz=0 -0.081 0 rpy=0 0 0
- added joint hip3_fixed: type fixed, parent hip3, child thigh_shoulder3, origin xyz=0 -0.081 0 rpy=0 0 0
- added joint jtoe0: type fixed, parent lower0, child toe0, origin xyz=0 0 -0.2 rpy=0 0 0
- added joint jtoe1: type fixed, parent lower1, child toe1, origin xyz=0 0 -0.2 rpy=0 0 0
- added joint jtoe2: type fixed, parent lower2, child toe2, origin xyz=0 0 -0.2 rpy=0 0 0
- added joint jtoe3: type fixed, parent lower3, child toe3, origin xyz=0 0 -0.2 rpy=0 0 0
- joint floating_base: parent base -> body

Commit message: Rebase with Devel

File: quad_simulator/a1_description/urdf/a1.urdf (robot description, URDF)
Before this commit: robot a1_description, 23 links, 22 joints
Joints:
- joint 0: limit lower=-2.6179938779914944 upper=2.6179938779914944 effort=33.5 velocity=21 -> lower=-6.28318530718 upper=6.28318530718 effort=33.5 velocity=21
- joint 1: limit lower=0.445058959258554 upper=2.2252947962927703 effort=33.5 velocity=21 -> lower=-6.28318530718 upper=6.28318530718 effort=33.5 velocity=21
- joint 2: limit lower=-2.6179938779914944 upper=2.6179938779914944 effort=33.5 velocity=21 -> lower=-6.28318530718 upper=6.28318530718 effort=33.5 velocity=21
- joint 3: limit lower=0.445058959258554 upper=2.2252947962927703 effort=33.5 velocity=21 -> lower=-6.28318530718 upper=6.28318530718 effort=33.5 velocity=21
- joint 4: limit lower=-2.6179938779914944 upper=2.6179938779914944 effort=33.5 velocity=21 -> lower=-6.28318530718 upper=6.28318530718 effort=33.5 velocity=21
- joint 5: limit lower=0.445058959258554 upper=2.2252947962927703 effort=33.5 velocity=21 -> lower=-6.28318530718 upper=6.28318530718 effort=33.5 velocity=21
- joint 6: limit lower=-2.6179938779914944 upper=2.6179938779914944 effort=33.5 velocity=21 -> lower=-6.28318530718 upper=6.28318530718 effort=33.5 velocity=21
- joint 7: limit lower=0.445058959258554 upper=2.2252947962927703 effort=33.5 velocity=21 -> lower=-6.28318530718 upper=6.28318530718 effort=33.5 velocity=21
