Commit message: noetic_ekf_clean_real_ylo2

File: quad_simulator/ylo2_description/urdf/ylo2.urdf (robot description, URDF)
Before this commit: robot ylo2_description, 29 links, 28 joints
Links:
- removed link D435
- removed link T265
- added link d435; visual mesh filename=package://ylo2_description/meshes/body/textured/ylo2_d435_t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 scale=1 1 1
- added link t265; visual mesh filename=package://ylo2_description/meshes/body/textured/ylo2_t265_t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 scale=1 1.06 1.04
- link hip0: mass 0.599 -> 0.552; geometry collision cylinder length=0.0099 radius=0.05; visual mesh filename=package://ylo2_description/meshes/leg/textured/ylo2textured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 scale=1 1 1
- link hip1: mass 0.599 -> 0.552; geometry collision cylinder length=0.0099 radius=0.05; visual mesh filename=package://ylo2_description/meshes/leg/textured/ylo2textured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 scale=1 1 1
- link hip2: mass 0.599 -> 0.552; geometry collision cylinder length=0.0099 radius=0.05; visual mesh filename=package://ylo2_description/meshes/leg/textured/ylo2textured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 scale=1 1 1
- link hip3: mass 0.599 -> 0.552; geometry collision cylinder length=0.0099 radius=0.05; visual mesh filename=package://ylo2_description/meshes/leg/textured/ylo2textured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 scale=1 1 1
- link lower0: mass 0.265 -> 0.235; geometry collision box size=0.19 0.02 0.02; visual mesh filename=package://ylo2_description/meshes/leg/textured/lower_leg.dae scale=1 1 1
- link lower1: mass 0.265 -> 0.235; geometry collision box size=0.19 0.02 0.02; visual mesh filename=package://ylo2_description/meshes/leg/textured/lower_leg.dae scale=1 1 1
- link lower2: mass 0.265 -> 0.235; geometry collision box size=0.19 0.02 0.02; visual mesh filename=package://ylo2_description/meshes/leg/textured/lower_leg.dae scale=1 1 1
- link lower3: mass 0.265 -> 0.235; geometry collision box size=0.19 0.02 0.02; visual mesh filename=package://ylo2_description/meshes/leg/textured/lower_leg.dae scale=1 1 1
- link thigh_shoulder0: geometry collision cylinder length=0.0553 radius=0.05
- link thigh_shoulder1: geometry collision cylinder length=0.0553 radius=0.05
- link thigh_shoulder2: geometry collision cylinder length=0.0553 radius=0.05
- link thigh_shoulder3: geometry collision cylinder length=0.0553 radius=0.05
- link toe0: mass 0.078 -> 0.035; geometry collision sphere radius=0.022; visual mesh filename=package://ylo2_description/meshes/leg/fl_foot.dae scale=1.0 1.0 1.0
- link toe1: mass 0.078 -> 0.035; geometry collision sphere radius=0.022; visual mesh filename=package://ylo2_description/meshes/leg/fl_foot.dae scale=1.0 1.0 1.0
- link toe2: mass 0.078 -> 0.035; geometry collision sphere radius=0.022; visual mesh filename=package://ylo2_description/meshes/leg/fl_foot.dae scale=1.0 1.0 1.0
- link toe3: mass 0.078 -> 0.035; geometry collision sphere radius=0.022; visual mesh filename=package://ylo2_description/meshes/leg/fl_foot.dae scale=1.0 1.0 1.0
- link trunk: mass 6.0 -> 4.076; geometry collision box size=0.26 0.18 0.14; visual mesh filename=package://ylo2_description/meshes/body/textured/ylo2_textur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 scale=1 1 1
- link upper0: mass 1.08 -> 1.009; geometry collision box size=0.201 0.0374 0.03; visual mesh filename=package://ylo2_description/meshes/leg/textured/ylo2_texture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 scale=1 1 1
- link upper1: mass 1.08 -> 1.009; geometry collision box size=0.201 0.0374 0.03; visual mesh filename=package://ylo2_description/meshes/leg/textured/ylo2_texture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 scale=1 1 1
- link upper2: mass 1.08 -> 1.009; geometry collision box size=0.201 0.0374 0.03; visual mesh filename=package://ylo2_description/meshes/leg/textured/ylo2_texture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 scale=1 -1 1
- link upper3: mass 1.08 -> 1.009; geometry collision box size=0.201 0.0374 0.03; visual mesh filename=package://ylo2_description/meshes/leg/textured/ylo2_texture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 scale=1 -1 1
Joints:
- removed joint D435_joint
- removed joint T265_joint
- added joint d435_joint: type fixed, parent trunk, child d435, origin xyz=0 0 0 rpy=0 0 0
- added joint t265_joint: type fixed, parent trunk, child t265, origin xyz=0 0 0 rpy=0 0 0
- joint 0: limit lower=-6.283185307179586 upper=6.283185307179586 effort=33.5 velocity=21 -> lower=-6.283185307179586 upper=6.283185307179586 effort=15 velocity=40
- joint 1: limit lower=-6.283185307179586 upper=6.283185307179586 effort=33.5 velocity=21 -> lower=-6.283185307179586 upper=6.283185307179586 effort=45 velocity=13.33; origin xyz=-0.001 0.075 -0.201 rpy=0 -3.141592653589793 0 -> xyz=-0.001 0.075 -0.215 rpy=0 -3.141592653589793 0
- joint 10: limit lower=-0.8028514559173915 upper=0.8028514559173915 effort=33.5 velocity=21 -> lower=-0.013962634015954637 upper=0.013962634015954637 effort=15 velocity=40
- joint 11: limit lower=-0.8028514559173915 upper=0.8028514559173915 effort=33.5 velocity=21 -> lower=-0.013962634015954637 upper=0.013962634015954637 effort=15 velocity=40
- joint 2: limit lower=-6.283185307179586 upper=6.283185307179586 effort=33.5 velocity=21 -> lower=-6.283185307179586 upper=6.283185307179586 effort=15 velocity=40
- joint 3: limit lower=-6.283185307179586 upper=6.283185307179586 effort=33.5 velocity=21 -> lower=-6.283185307179586 upper=6.283185307179586 effort=45 velocity=13.33; origin xyz=-0.001 0.075 -0.201 rpy=0 -3.141592653589793 0 -> xyz=-0.001 0.075 -0.215 rpy=0 -3.141592653589793 0
- joint 4: limit lower=-6.283185307179586 upper=6.283185307179586 effort=33.5 velocity=21 -> lower=-6.283185307179586 upper=6.283185307179586 effort=15 velocity=40
- joint 5: limit lower=-6.283185307179586 upper=6.283185307179586 effort=33.5 velocity=21 -> lower=-6.283185307179586 upper=6.283185307179586 effort=45 velocity=13.33; origin xyz=-0.001 -0.075 -0.201 rpy=0 -3.141592653589793 0 -> xyz=-0.001 -0.075 -0.215 rpy=0 -3.141592653589793 0
- joint 6: limit lower=-6.283185307179586 upper=6.283185307179586 effort=33.5 velocity=21 -> lower=-6.283185307179586 upper=6.283185307179586 effort=15 velocity=40
- joint 7: limit lower=-6.283185307179586 upper=6.283185307179586 effort=33.5 velocity=21 -> lower=-6.283185307179586 upper=6.283185307179586 effort=45 velocity=13.33; origin xyz=-0.001 -0.075 -0.201 rpy=0 -3.141592653589793 0 -> xyz=-0.001 -0.075 -0.215 rpy=0 -3.141592653589793 0
- joint 8: limit lower=-0.8028514559173915 upper=0.8028514559173915 effort=33.5 velocity=21 -> lower=-0.013962634015954637 upper=0.013962634015954637 effort=15 velocity=40
- joint 9: limit lower=-0.8028514559173915 upper=0.8028514559173915 effort=33.5 velocity=21 -> lower=-0.013962634015954637 upper=0.013962634015954637 effort=15 velocity=40

File: quad_simulator/ylo2_description/xacro/const.xacro (robot description, xacro)
@@ -8,24 +8,23 @@
     <xacro:property name="body_center_z" value="0.0"/>
     <!-- simplified collision value -->
-    <xacro:property name="trunk_width" value="0.350"/>
-    <xacro:property name="trunk_length" value="0.57"/>
-    <xacro:property name="trunk_height" value="0.149"/>
-    <xacro:property name="hip_radius" value="0.050"/>
-    <xacro:property name="hip_length" value="0.06"/>
-    <xacro:property name="thigh_shoulder_radius" value="0.044"/>
-    <xacro:property name="thigh_shoulder_length" value="0.08"/>
+    <xacro:property name="trunk_width" value="0.247"/>
+    <xacro:property name="trunk_length" value="0.2687"/> <!-- à jour aout 2023 -->
+    <xacro:property name="trunk_height" value="0.150"/>
+    <xacro:property name="hip_radius" value="0.050"/> <!-- hanche -->
+    <xacro:property name="hip_length" value="0.0099"/> <!-- à jour juillet 2023 -->
+    <xacro:property name="thigh_shoulder_radius" value="0.050"/> <!-- moteur épaule -->
+    <xacro:property name="thigh_shoulder_length" value="0.0553"/>
     <xacro:property name="thigh_width" value="0.0374"/>
     <xacro:property name="thigh_height" value="0.043"/>
-    <xacro:property name="calf_width" value="0.0208"/>
+    <xacro:property name="calf_width" value="0.0208"/> <!-- mollet -->
     <xacro:property name="calf_height" value="0.016"/>
     <xacro:property name="foot_radius" value="0.0265"/>
-    <xacro:property name="stick_radius" value="0.01"/>
-    <xacro:property name="stick_length" value="0.2"/>
-    <xacro:property name="toe_friction" value="0.2"/>
+    <xacro:property name="toe_friction" value="0.2"/> <!-- bout / pied -->
     <xacro:property name="toe_lateral_friction" value="0.2"/>
     <xacro:property name="toe_stiffness" value="30000.0"/>
     <xacro:property name="toe_damping" value="1000.0"/>
     <!-- kinematic value -->
-    <xacro:property name="thigh_offset" value="0.02"/><!-- decalage lateral HIP -> upper_leg - lateral difference between HIP and upper_leg -->
+    <xacro:property name="hip_offset" value="0.083"/><!-- decalage lateral HIP -> upper_leg - lateral difference between HIP and upper_leg -->
+    <xacro:property name="thigh_offset" value="0.02"/>
     <xacro:property name="thigh_length" value="0.201"/><!-- upper leg size, from HIP axis, to lower leg axis-->
     <xacro:property name="calf_length" value="0.230"/><!-- lower leg size, from lower leg axis to end foot -->
@@ -35,75 +34,75 @@
     <xacro:property name="leg_offset_z" value="${0.024}"/>
     <xacro:property name="trunk_offset_z" value="0.01675"/><!-- decalage hauteur axes pattes/abad - vertical difference HIP -> ABAD -->
-    <xacro:property name="hip_offset" value="0.083"/>
     <!-- joint limits -->
     <xacro:property name="damping" value="0"/>
     <xacro:property name="friction" value="0"/>
-    <xacro:property name="hip_max" value="46"/>
-    <xacro:property name="hip_min" value="-46"/>
-    <xacro:property name="hip_velocity_max" value="21"/>
-    <xacro:property name="hip_torque_max" value="33.5"/>
+    <xacro:property name="hip_max" value="0.80"/>
+    <xacro:property name="hip_min" value="-0.80"/>
+    <xacro:property name="hip_velocity_max" value="40"/>
+    <xacro:property name="hip_torque_max" value="15
+    "/>
     <xacro:property name="thigh_max" value="360"/>
     <xacro:property name="thigh_min" value="-360"/>
-    <xacro:property name="thigh_velocity_max" value="21"/>
-    <xacro:property name="thigh_torque_max" value="33.5"/>
+    <xacro:property name="thigh_velocity_max" value="40"/>
+    <xacro:property name="thigh_torque_max" value="15"/>
     <xacro:property name="calf_max" value="360"/>
     <xacro:property name="calf_min" value="-360"/>
-    <xacro:property name="calf_velocity_max" value="21"/>
-    <xacro:property name="calf_torque_max" value="33.5"/>
+    <xacro:property name="calf_velocity_max" value="13.33"/>
+    <xacro:property name="calf_torque_max" value="45"/>
     <!-- dynamics inertial value -->
     <!-- trunk -->
-    <xacro:property name="trunk_mass" value="6.0"/>
-    <xacro:property name="trunk_com_x" value="0.02"/>
-    <xacro:property name="trunk_com_y" value="0.00194"/>
-    <xacro:property name="trunk_com_z" value="0.0"/>
-    <xacro:property name="trunk_ixx" value="0.0158533"/>
-    <xacro:property name="trunk_ixy" value="-0.0001332"/>
-    <xacro:property name="trunk_ixz" value="-0.0002403"/>
-    <xacro:property name="trunk_iyy" value="0.04168"/>
-    <xacro:property name="trunk_iyz" value="0.000015299"/>
-    <xacro:property name="trunk_izz" value="0.04742"/>
+    <xacro:property name="trunk_mass" value="4.076"/> <!-- corps complet, sans moteurs, sans rplidar / à jour aout 2023 -->
+    <xacro:property name="trunk_com_x" value="0.03250797"/>
+    <xacro:property name="trunk_com_y" value="0.00737083"/>
+    <xacro:property name="trunk_com_z" value="0.03316464"/>
+    <xacro:property name="trunk_ixx" value="0.01982157"/>
+    <xacro:property name="trunk_ixy" value="-0.00002989"/>
+    <xacro:property name="trunk_ixz" value="-0.00037560"/>
+    <xacro:property name="trunk_iyy" value="0.07819480"/>
+    <xacro:property name="trunk_iyz" value="-0.00001253"/>
+    <xacro:property name="trunk_izz" value="0.08412247"/>
     <!-- hip (left front) -->
-    <xacro:property name="hip_mass" value="0.599"/>
-    <xacro:property name="hip_com_x" value="-0.011957"/>
-    <xacro:property name="hip_com_y" value="0.000306"/>
-    <xacro:property name="hip_com_z" value="0.000366"/>
-    <xacro:property name="hip_ixx" value="0.0004159"/>
-    <xacro:property name="hip_ixy" value="0.000004253"/>
-    <xacro:property name="hip_ixz" value="0.000000368"/>
-    <xacro:property name="hip_iyy" value="0.0007108"/>
-    <xacro:property name="hip_iyz" value="0.000000215"/>
-    <xacro:property name="hip_izz" value="0.0004707"/>
+    <xacro:property name="hip_mass" value="0.552"/> <!-- motor+fix+passe-cable+cable / à jour aout 2023 -->
+    <xacro:property name="hip_com_x" value="-0.01857801"/>
+    <xacro:property name="hip_com_y" value="-0.01030756"/>
+    <xacro:property name="hip_com_z" value="0.00689884"/>
+    <xacro:property name="hip_ixx" value="0.00043998"/>
+    <xacro:property name="hip_ixy" value="-0.00000463"/>
+    <xacro:property name="hip_ixz" value="-0.00002717"/>
+    <xacro:property name="hip_iyy" value="0.00070180"/>
+    <xacro:property name="hip_iyz" value="-0.00000463"/>
+    <xacro:property name="hip_izz" value="0.00043986"/>
     <!-- thigh / upperleg -->
-    <xacro:property name="thigh_mass" value="1.080"/>
-    <xacro:property name="thigh_com_x" value="-0.000684"/>
-    <xacro:property name="thigh_com_y" value="-0.010999"/>
-    <xacro:property name="thigh_com_z" value="-0.035487"/>
-    <xacro:property name="thigh_ixx" value="0.005666803"/>
-    <xacro:property name="thigh_ixy" value="0.000003597"/>
-    <xacro:property name="thigh_ixz" value="0.000491446"/>
-    <xacro:property name="thigh_iyy" value="0.005847229"/>
-    <xacro:property name="thigh_iyz" value="0.000010086"/>
-    <xacro:property name="thigh_izz" value="0.000369811"/>
+    <xacro:property name="thigh_mass" value="1.009"/>  <!-- moteur+coques+pignon+axe+fixation hip+poulie nylon+passe-cable+cables / à jour aout 2023 -->
+    <xacro:property name="thigh_com_x" value="0.01454697"/>
+    <xacro:property name="thigh_com_y" value="0.06694306"/>
+    <xacro:property name="thigh_com_z" value="-0.04580968"/>
+    <xacro:property name="thigh_ixx" value="0.00573610"/>
+    <xacro:property name="thigh_ixy" value="0.00001510"/>
+    <xacro:property name="thigh_ixz" value="0.00039092"/>
+    <xacro:property name="thigh_iyy" value="0.00562867"/>
+    <xacro:property name="thigh_iyz" value="-0.00003266"/>
+    <xacro:property name="thigh_izz" value="0.00096304"/>
     <!-- calf / lowerleg -->
-    <xacro:property name="calf_mass" value="0.265"/>
-    <xacro:property name="calf_com_x" value="0.000252"/>
-    <xacro:property name="calf_com_y" value="0.000194"/>
-    <xacro:property name="calf_com_z" value="-0.05192"/>
-    <xacro:property name="calf_ixx" value="0.0004583"/>
-    <xacro:property name="calf_ixy" value="-0.000000095"/>
-    <xacro:property name="calf_ixz" value="0.000026512"/>
-    <xacro:property name="calf_iyy" value="0.0004675"/>
-    <xacro:property name="calf_iyz" value="0.000000277"/>
-    <xacro:property name="calf_izz" value="0.000029145"/>
+    <xacro:property name="calf_mass" value="0.235"/> <!-- à jour juillet 2023 -->
+    <xacro:property name="calf_com_x" value="0.00198597"/>
+    <xacro:property name="calf_com_y" value="0.00042353"/>
+    <xacro:property name="calf_com_z" value="-0.05849061"/>
+    <xacro:property name="calf_ixx" value="0.00065666"/>
+    <xacro:property name="calf_ixy" value="0.00000000"/>
+    <xacro:property name="calf_ixz" value="0.00003548"/>
+    <xacro:property name="calf_iyy" value="0.00067446"/>
+    <xacro:property name="calf_iyz" value="-0.00000000"/>
+    <xacro:property name="calf_izz" value="0.00004729"/>
     <!-- foot -->
-    <xacro:property name="foot_mass" value="0.078"/>
-    <xacro:property name="foot_com_x" value="-0.007246"/>
-    <xacro:property name="foot_com_y" value="0.000092"/>
-    <xacro:property name="foot_com_z" value="-0.038267"/>
-    <xacro:property name="foot_ixx" value="0.000029902"/>
-    <xacro:property name="foot_ixy" value="-0.000000022"/>
-    <xacro:property name="foot_ixz" value="-0.000004427"/>
-    <xacro:property name="foot_iyy" value="0.000030583"/>
-    <xacro:property name="foot_iyz" value="-0.000000099"/>
-    <xacro:property name="foot_izz" value="0.000014025"/>
+    <xacro:property name="foot_mass" value="0.035"/> <!-- à jour aout 2023 -->
+    <xacro:property name="foot_com_x" value="-0.00929514"/>
+    <xacro:property name="foot_com_y" value="0.00292672"/>
+    <xacro:property name="foot_com_z" value="-0.19787919"/>
+    <xacro:property name="foot_ixx" value="0.00001399"/>
+    <xacro:property name="foot_ixy" value="-0.00000001"/>
+    <xacro:property name="foot_ixz" value="-0.00000011"/>
+    <xacro:property name="foot_iyy" value="0.00001374"/>
+    <xacro:property name="foot_iyz" value="-0.00000192"/>
+    <xacro:property name="foot_izz" value="0.00000643"/>
 </robot>

File: quad_simulator/ylo2_description/xacro/leg.xacro (robot description, xacro)
@@ -32,5 +32,10 @@
                 <origin rpy="0 0 0" xyz="${hip_com_x*front_hind} ${hip_com_y*mirror} ${hip_com_z}"/>
                 <mass value="${hip_mass}"/>
-                <inertia ixx="${hip_ixx}" ixy="${hip_ixy*mirror*front_hind}" ixz="${hip_ixz*front_hind}" iyy="${hip_iyy}" iyz="${hip_iyz*mirror}" izz="${hip_izz}"/>
+                <inertia    ixx="${hip_ixx}"
+                            ixy="${hip_ixy*mirror*front_hind}"
+                            ixz="${hip_ixz*front_hind}"
+                            iyy="${hip_iyy}"
+                            iyz="${hip_iyz*mirror}"
+                            izz="${hip_izz}"/>
             </inertial>
         </link>
@@ -75,8 +80,8 @@
                 <material name="orange"/>
             </visual>
-            <collision name="upper${suffix}_collision">
-                <origin rpy="0 ${PI/2.0} 0" xyz="0 0 ${-thigh_length/2.0}"/>
+            <collision>
+                <origin rpy="0 ${pi/2.0+0.05} 0" xyz="0 ${0.074*mirror} -0.07"/>
                 <geometry>
-                    <box size="${thigh_length} ${thigh_width} ${thigh_height}"/>
+                    <box size="0.201 0.0374 0.03"/>
                 </geometry>
             </collision>
@@ -84,5 +89,10 @@
                 <origin rpy="0 0 0" xyz="${thigh_com_x} ${thigh_com_y*mirror} ${thigh_com_z}"/>
                 <mass value="${thigh_mass}"/>
-                <inertia ixx="${thigh_ixx}" ixy="${thigh_ixy*mirror}" ixz="${thigh_ixz}" iyy="${thigh_iyy}" iyz="${thigh_iyz*mirror}" izz="${thigh_izz}"/>
+                <inertia    ixx="${thigh_ixx}"
+                            ixy="${thigh_ixy*mirror}"
+                            ixz="${thigh_ixz}"
+                            iyy="${thigh_iyy}"
+                            iyz="${thigh_iyz*mirror}"
+                            izz="${thigh_izz}"/>
             </inertial>
         </link>
@@ -103,8 +113,8 @@
                 <material name="orange"/>
             </visual>
-            <collision name="lower${suffix}_collision">
-                <origin rpy="0 ${PI/2.0} 0" xyz="0 0 ${-calf_length/2.0}"/>
+            <collision>
+                <origin rpy="0 ${(pi/2.0-0.1)} 0" xyz="0 0 -0.08"/>
                 <geometry>
-                    <mesh filename="package://ylo2_description/meshes/leg/fl_lower_leg_collision.stl" scale="1 -1 1"/>-->
+                    <box size="0.19 0.02 0.02"/>
                 </geometry>
             </collision>
@@ -112,5 +122,10 @@
                 <origin rpy="0 0 0" xyz="${calf_com_x} ${calf_com_y} ${calf_com_z}"/>
                 <mass value="${calf_mass}"/>
-                <inertia ixx="${calf_ixx}" ixy="${calf_ixy}" ixz="${calf_ixz}" iyy="${calf_iyy}" iyz="${calf_iyz}" izz="${calf_izz}"/>
+                <inertia    ixx="${calf_ixx}"
+                            ixy="${calf_ixy}"
+                            ixz="${calf_ixz}"
+                            iyy="${calf_iyy}"
+                            iyz="${calf_iyz}"
+                            izz="${calf_izz}"/>
             </inertial>
         </link>
@@ -132,7 +147,7 @@
             </visual>
             <collision name="toe${suffix}_collision">
-                <origin rpy="0 0 0" xyz="0.009 ${(0.001*mirror)+0.001} 0.069"/>
+                <origin rpy="0 0 0" xyz="0 0 0.02"/>
                 <geometry>
-                    <mesh filename="package://ylo2_description/meshes/leg/fl_foot.dae" scale="1.0 1.0 1.0"/>-->
+                    <sphere radius="0.022"/>
                 </geometry>
                 <surface>
