Commit message: Added Dockerfile, Modifications to Go2W URDF

File: quad_simulator/go2w_description/models/go2w/urdf/go2w.urdf.xacro (robot description, xacro)
@@ -4,8 +4,7 @@
      Commit Version: 1.6.0-4-g7f85cfe  Build Version: 1.6.7995.38578
      For more information, please see http://wiki.ros.org/sw_urdf_exporter -->
-<robot
-  name="go2w_description">
-  <link
-    name="base">
+<robot name="go2w" xmlns:xacro="http://www.ros.org/wiki/xacro">
+  <link
+    name="body">
     <inertial>
       <origin
@@ -28,5 +27,5 @@
       <geometry>
         <mesh
-          filename="package://go2w_description/dae/base.dae" />
+          filename="package://go2w_description/models/go2w/dae/body.dae" />
       </geometry>
       <material
@@ -75,5 +74,5 @@
       rpy="0 0 0" />
     <parent
-      link="base" />
+      link="body" />
     <child
       link="Head_upper" />
@@ -120,5 +119,5 @@
   </joint>
   <link
-    name="FL_hip">
+    name="hip0">
     <inertial>
       <origin
@@ -141,5 +140,5 @@
       <geometry>
         <mesh
-          filename="package://go2w_description/dae/hip.dae" />
+          filename="package://go2w_description/models/go2w/dae/hip.dae" />
       </geometry>
       <material
@@ -157,5 +156,5 @@
   </link>
   <joint
-    name="FL_hip_joint"
+    name="8"
     type="revolute">
     <origin
@@ -163,7 +162,7 @@
       rpy="0 0 0" />
     <parent
-      link="base" />
-    <child
-      link="FL_hip" />
+      link="body" />
+    <child
+      link="hip0" />
     <axis
       xyz="1 0 0" />
@@ -175,5 +174,5 @@
   </joint>
   <link
-    name="FL_thigh">
+    name="upper0">
     <inertial>
       <origin
@@ -196,5 +195,5 @@
       <geometry>
         <mesh
-          filename="package://go2w_description/dae/thigh.dae" />
+          filename="package://go2w_description/models/go2w/dae/thigh.dae" />
       </geometry>
       <material
@@ -212,23 +211,23 @@
   </link>
   <joint
-    name="FL_thigh_joint"
+    name="0"
     type="revolute">
     <origin
       xyz="0 0.0955 0"
-      rpy="0 0 0" />
-    <parent
-      link="FL_hip" />
-    <child
-      link="FL_thigh" />
-    <axis
-      xyz="0 1 0" />
+      rpy="0 1.57079632679 0" />
+    <parent
+      link="hip0" />
+    <child
+      link="upper0" />
+    <axis
+      xyz="0 -1 0" />
     <limit
-      lower="-1.5707963267948966"
-      upper="3.4907"
+      lower="-2.6179938779914944"
+      upper="2.6179938779914944"
       effort="23.7"
       velocity="30.1" />
   </joint>
   <link
-    name="FL_calf">
+    name="lower0">
     <inertial>
       <origin
@@ -251,5 +250,5 @@
       <geometry>
         <mesh
-          filename="package://go2w_description/dae/calf.stl" />
+          filename="package://go2w_description/models/go2w/dae/calf.stl" />
       </geometry>
       <material
@@ -267,23 +266,23 @@
   </link>
   <joint
-    name="FL_calf_joint"
+    name="1"
     type="revolute">
     <origin
       xyz="0 0 -0.213"
-      rpy="0 0 0" />
-    <parent
-      link="FL_thigh" />
-    <child
-      link="FL_calf" />
+      rpy="0 -3.14159265359 0" />
+    <parent
+      link="upper0" />
+    <child
+      link="lower0" />
     <axis
       xyz="0 1 0" />
     <limit
-      lower="-2.7227"
-      upper="-0.83776"
+      lower="0.445058959258554"
+      upper="2.2252947962927703"
       effort="35.55"
       velocity="20.07" />
   </joint>
   <link
-    name="FL_calflower">
+    name="lower0_lower">
     <collision>
       <origin rpy="0 0 0" xyz="0 0 0" />
@@ -294,5 +293,5 @@
   </link>
   <joint
-    name="FL_calflower_joint"
+    name="lower0_lower_joint"
     type="fixed">
     <origin
@@ -300,12 +299,12 @@
       rpy="0 0.05 0" />
     <parent
-      link="FL_calf" />
-    <child
-      link="FL_calflower" />
+      link="lower0" />
+    <child
+      link="lower0_lower" />
     <axis
       xyz="0 0 0" />
   </joint>
   <link
-    name="FL_calflower1">
+    name="lower0_lower1">
     <collision>
       <origin rpy="0 0 0" xyz="0 0 0" />
@@ -316,5 +315,5 @@
   </link>
   <joint
-    name="FL_calflower1_joint"
+    name="lower0_lower1_joint"
     type="fixed">
     <origin
@@ -322,12 +321,12 @@
       rpy="0 0.48 0" />
     <parent
-      link="FL_calflower" />
-    <child
-      link="FL_calflower1" />
+      link="lower0_lower" />
+    <child
+      link="lower0_lower1" />
     <axis
       xyz="0 0 0" />
   </joint>
   <link
-    name="FL_foot_motor">
+    name="toe0_motor">
     <inertial>
       <origin
@@ -352,5 +351,5 @@
   </link>
   <joint
-    name="FL_foot_motor_joint"
+    name="toe0_motor_joint"
     type="fixed">
     <origin
@@ -358,12 +357,12 @@
       rpy="0 0.0 0" />
     <parent
-      link="FL_calf" />
-    <child
-      link="FL_foot_motor" />
+      link="lower0" />
+    <child
+      link="toe0_motor" />
     <axis
       xyz="0 0 0" />
   </joint>
   <link
-    name="FL_foot">
+    name="toe0">
     <inertial>
       <origin
@@ -385,5 +384,5 @@
         rpy="0 0 0" />
       <geometry>
-        <mesh filename="package://go2w_description/dae/left_wheel.dae" />
+        <mesh filename="package://go2w_description/models/go2w/dae/left_wheel.dae" />
       </geometry>
       <material
@@ -396,5 +395,5 @@
       <origin rpy="1.5707963267948966 0 0" xyz="0 0.0 0" />
       <geometry>
-        <mesh filename="package://go2w_description/dae/left_wheel.dae" />
+        <mesh filename="package://go2w_description/models/go2w/dae/left_wheel.dae" />
         <!-- <cylinder length="0.045" radius="0.086" /> -->
       </geometry>
@@ -402,5 +401,5 @@
   </link>
   <joint
-    name="FL_foot_joint"
+    name="jtoe0"
     type="continuous">
     <origin
@@ -408,7 +407,7 @@
       rpy="0 0 0" />
     <parent
-      link="FL_calf" />
-    <child
-      link="FL_foot" />
+      link="lower0" />
+    <child
+      link="toe0" />
     <axis
       xyz="0 1 0" />
@@ -419,5 +418,5 @@
   </joint>
   <link
-    name="FR_hip">
+    name="hip2">
     <inertial>
       <origin
@@ -440,5 +439,5 @@
       <geometry>
         <mesh
-          filename="package://go2w_description/dae/hip.dae" />
+          filename="package://go2w_description/models/go2w/dae/hip.dae" />
       </geometry>
       <material
@@ -456,5 +455,5 @@
   </link>
   <joint
-    name="FR_hip_joint"
+    name="10"
     type="revolute">
     <origin
@@ -462,7 +461,7 @@
       rpy="0 0 0" />
     <parent
-      link="base" />
-    <child
-      link="FR_hip" />
+      link="body" />
+    <child
+      link="hip2" />
     <axis
       xyz="1 0 0" />
@@ -474,5 +473,5 @@
   </joint>
   <link
-    name="FR_thigh">
+    name="upper2">
     <inertial>
       <origin
@@ -495,5 +494,5 @@
       <geometry>
         <mesh
-          filename="package://go2w_description/dae/thigh_mirror.dae" />
+          filename="package://go2w_description/models/go2w/dae/thigh_mirror.dae" />
       </geometry>
       <material
@@ -511,23 +510,23 @@
   </link>
   <joint
-    name="FR_thigh_joint"
+    name="4"
     type="revolute">
     <origin
       xyz="0 -0.0955 0"
-      rpy="0 0 0" />
-    <parent
-      link="FR_hip" />
-    <child
-      link="FR_thigh" />
-    <axis
-      xyz="0 1 0" />
+      rpy="0 1.57079632679 0" />
+    <parent
+      link="hip2" />
+    <child
+      link="upper2" />
+    <axis
+      xyz="0 -1 0" />
     <limit
-      lower="-1.5707963267948966"
-      upper="3.4907"
+      lower="-2.6179938779914944"
+      upper="2.6179938779914944"
       effort="23.7"
       velocity="30.1" />
   </joint>
   <link
-    name="FR_calf">
+    name="lower2">
     <inertial>
       <origin
@@ -550,5 +549,5 @@
       <geometry>
         <mesh
-          filename="package://go2w_description/dae/calf_mirror.stl" />
+          filename="package://go2w_description/models/go2w/dae/calf_mirror.stl" />
       </geometry>
       <material
@@ -566,23 +565,23 @@
   </link>
   <joint
-    name="FR_calf_joint"
+    name="5"
     type="revolute">
     <origin
       xyz="0 0 -0.213"
-      rpy="0 0 0" />
-    <parent
-      link="FR_thigh" />
-    <child
-      link="FR_calf" />
+      rpy="0 -3.14159265359 0" />
+    <parent
+      link="upper2" />
+    <child
+      link="lower2" />
     <axis
       xyz="0 1 0" />
     <limit
-      lower="-2.7227"
-      upper="-0.83776"
+      lower="0.445058959258554"
+      upper="2.2252947962927703"
       effort="35.55"
       velocity="20.07" />
   </joint>
   <link
-    name="FR_calflower">
+    name="lower2_lower">
     <collision>
       <origin rpy="0 0 0" xyz="0 0 0" />
@@ -593,5 +592,5 @@
   </link>
   <joint
-    name="FR_calflower_joint"
+    name="lower2_lower_joint"
     type="fixed">
     <origin
@@ -599,12 +598,12 @@
       rpy="0 0.05 0" />
     <parent
-      link="FR_calf" />
-    <child
-      link="FR_calflower" />
+      link="lower2" />
+    <child
+      link="lower2_lower" />
     <axis
       xyz="0 0 0" />
   </joint>
   <link
-    name="FR_calflower1">
+    name="lower2_lower1">
     <collision>
       <origin rpy="0 0 0" xyz="0 0 0" />
@@ -615,5 +614,5 @@
   </link>
   <joint
-    name="FR_calflower1_joint"
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