Commit message: Updated B2 Xacros

File: quad_simulator/b2_description/models/b2/b2.sdf.xacro (robot description, xacro)
@@ -1,5 +1,8 @@
-<sdf version='1.11'>
-  <model name='b2_description'>
-    <link name='base_link'>
+<?xml version='1.0'?>
+<sdf version='1.11' xmlns:xacro="http://www.ros.org/wiki/xacro">
+  <xacro:arg name="namespace" default="robot_1" />
+  <xacro:arg name="controller_config_path" default="/path/quad_control.yaml" />
+  <model name='b2'>
+    <link name='body'>
       <inertial>
         <pose>0.023466809815318752 0.0045473199620229363 0.011407653769203359 0 0 0</pose>
@@ -14,5 +17,5 @@
         </inertia>
       </inertial>
-      <collision name='base_link_collision'>
+      <collision name='body_collision'>
         <pose>0 0 0 0 0 0</pose>
         <geometry>
@@ -22,5 +25,5 @@
         </geometry>
       </collision>
-      <collision name='base_link_fixed_joint_lump__FL_hip_rotor_collision_1'>
+      <collision name='body_fixed_joint_lump__FL_hip_rotor_collision_1'>
         <pose>0.20205000000000001 0.071999999999999995 0 0 1.5707963267948966 0</pose>
         <geometry>
@@ -31,5 +34,5 @@
         </geometry>
       </collision>
-      <collision name='base_link_fixed_joint_lump__FR_hip_rotor_collision_2'>
+      <collision name='body_fixed_joint_lump__FR_hip_rotor_collision_2'>
         <pose>0.20205000000000001 -0.071999999999999995 0 0 1.5707963267948966 0</pose>
         <geometry>
@@ -40,5 +43,5 @@
         </geometry>
       </collision>
-      <collision name='base_link_fixed_joint_lump__RL_hip_rotor_collision_3'>
+      <collision name='body_fixed_joint_lump__RL_hip_rotor_collision_3'>
         <pose>-0.20205000000000001 0.071999999999999995 0 0 1.5707963267948966 0</pose>
         <geometry>
@@ -49,5 +52,5 @@
         </geometry>
       </collision>
-      <collision name='base_link_fixed_joint_lump__RR_hip_rotor_collision_4'>
+      <collision name='body_fixed_joint_lump__RR_hip_rotor_collision_4'>
         <pose>-0.20205000000000001 -0.071999999999999995 0 0 1.5707963267948966 0</pose>
         <geometry>
@@ -58,5 +61,5 @@
         </geometry>
       </collision>
-      <collision name='base_link_fixed_joint_lump__head_Link_collision_5'>
+      <collision name='body_fixed_joint_lump__head_Link_collision_5'>
         <pose>0.40999999999999998 0 0.0050000000000000001 0 0 0</pose>
         <geometry>
@@ -66,5 +69,5 @@
         </geometry>
       </collision>
-      <collision name='base_link_fixed_joint_lump__lidar_link_collision_6'>
+      <collision name='body_fixed_joint_lump__lidar_link_collision_6'>
         <pose>0.34217999999999998 0 0.15851000000000001 0 0 0</pose>
         <geometry>
@@ -75,5 +78,5 @@
         </geometry>
       </collision>
-      <collision name='base_link_fixed_joint_lump__tail_link_collision_7'>
+      <collision name='body_fixed_joint_lump__tail_link_collision_7'>
         <pose>-0.40500000000000003 0 0.0050000000000000001 0 0 0</pose>
         <geometry>
@@ -83,10 +86,10 @@
         </geometry>
       </collision>
-      <visual name='base_link_visual'>
+      <visual name='body_visual'>
         <pose>0 0 0 0 0 0</pose>
         <geometry>
           <mesh>
             <scale>1 1 1</scale>
-            <uri>model://b2_description/meshes/base_link.dae</uri>
+            <uri>model://b2/meshes/body.dae</uri>
           </mesh>
         </geometry>
@@ -97,8 +100,8 @@
       </visual>
     </link>
-    <joint name='FL_hip_joint' type='revolute'>
-      <pose relative_to='base_link'>0.32850000000000001 0.071999999999999995 0 0 0 0</pose>
-      <parent>base_link</parent>
-      <child>FL_hip</child>
+    <joint name='8' type='revolute'>
+      <pose relative_to='body'>0.32850000000000001 0.071999999999999995 0 0 0 0</pose>
+      <parent>body</parent>
+      <child>hip0</child>
       <axis>
         <xyz>1 0 0</xyz>
@@ -115,6 +118,6 @@
       </axis>
     </joint>
-    <link name='FL_hip'>
-      <pose relative_to='FL_hip_joint'>0 0 0 0 0 0</pose>
+    <link name='hip0'>
+      <pose relative_to='8'>0 0 0 0 0 0</pose>
       <inertial>
         <pose>-0.0034845889899538418 -0.0089670431713277203 0 0 0 0</pose>
@@ -129,5 +132,5 @@
         </inertia>
       </inertial>
-      <collision name='FL_hip_collision'>
+      <collision name='hip0_collision'>
         <pose>0 0.12 0 1.5707963267948959 0 0</pose>
         <geometry>
@@ -138,5 +141,5 @@
         </geometry>
       </collision>
-      <collision name='FL_hip_fixed_joint_lump__FL_thigh_rotor_collision_1'>
+      <collision name='hip0_fixed_joint_lump__FL_thigh_rotor_collision_1'>
         <pose>0 -0.0079799999999999992 0 1.5707963267948959 0 0</pose>
         <geometry>
@@ -147,10 +150,10 @@
         </geometry>
       </collision>
-      <visual name='FL_hip_visual'>
+      <visual name='hip0_visual'>
         <pose>0 0 0 0 0 0</pose>
         <geometry>
           <mesh>
             <scale>1 1 1</scale>
-            <uri>model://b2_description/meshes/FL_hip.dae</uri>
+            <uri>model://b2/meshes/FL_hip.dae</uri>
           </mesh>
         </geometry>
@@ -161,13 +164,13 @@
       </visual>
     </link>
-    <joint name='FL_thigh_joint' type='revolute'>
-      <pose relative_to='FL_hip'>0 0.11973 0 0 0 0</pose>
-      <parent>FL_hip</parent>
-      <child>FL_thigh</child>
-      <axis>
-        <xyz>0 1 0</xyz>
-        <limit>
-          <lower>-0.93999999999999995</lower>
-          <upper>4.6900000000000004</upper>
+    <joint name='0' type='revolute'>
+      <pose relative_to='hip0'>0 0.11973 0 0 1.5708 0</pose>
+      <parent>hip0</parent>
+      <child>upper0</child>
+      <axis>
+        <xyz>0 -1 0</xyz>
+        <limit>
+          <lower>-2.8012</lower>
+          <upper>2.8012</upper>
           <effort>200</effort>
           <velocity>23</velocity>
@@ -179,6 +182,6 @@
       </axis>
     </joint>
-    <link name='FL_thigh'>
-      <pose relative_to='FL_thigh_joint'>0 0 0 0 0 0</pose>
+    <link name='upper0'>
+      <pose relative_to='0'>0 0 0 0 0 0</pose>
       <inertial>
         <pose>-0.0059220576371272924 -0.033517415062169917 -0.054547253295629393 0 0 0</pose>
@@ -193,5 +196,5 @@
         </inertia>
       </inertial>
-      <collision name='FL_thigh_collision'>
+      <collision name='upper0_collision'>
         <pose>-0.025000000000000001 0 -0.16 0 1.5707963267948966 0</pose>
         <geometry>
@@ -201,5 +204,5 @@
         </geometry>
       </collision>
-      <collision name='FL_thigh_fixed_joint_lump__FL_calf_rotor_collision_1'>
+      <collision name='upper0_fixed_joint_lump__FL_calf_rotor_collision_1'>
         <pose>0 -0.057880000000000001 0 1.5707963267948959 0 0</pose>
         <geometry>
@@ -210,10 +213,10 @@
         </geometry>
       </collision>
-      <visual name='FL_thigh_visual'>
+      <visual name='upper0_visual'>
         <pose>0 0 0 0 0 0</pose>
         <geometry>
           <mesh>
             <scale>1 1 1</scale>
-            <uri>model://b2_description/meshes/FL_thigh.dae</uri>
+            <uri>model://b2/meshes/FL_thigh.dae</uri>
           </mesh>
         </geometry>
@@ -224,13 +227,13 @@
       </visual>
     </link>
-    <joint name='FL_calf_joint' type='revolute'>
-      <pose relative_to='FL_thigh'>0 -8.6984000000000006e-05 -0.34999999999999998 0 0 0</pose>
-      <parent>FL_thigh</parent>
-      <child>FL_calf</child>
+    <joint name='1' type='revolute'>
+      <pose relative_to='upper0'>0 -8.6984000000000006e-05 -0.34999999999999998 -3.14159 0 -3.14159</pose>
+      <parent>upper0</parent>
+      <child>lower0</child>
       <axis>
         <xyz>0 1 0</xyz>
         <limit>
-          <lower>-2.8199999999999998</lower>
-          <upper>-0.42999999999999999</upper>
+          <lower>0.32159265359</lower>
+          <upper>2.71159265359</upper>
           <effort>320</effort>
           <velocity>14</velocity>
@@ -242,6 +245,6 @@
       </axis>
     </joint>
-    <link name='FL_calf'>
-      <pose relative_to='FL_calf_joint'>0 0 0 0 0 0</pose>
+    <link name='lower0'>
+      <pose relative_to='1'>0 0 0 0 0 0</pose>
       <inertial>
         <pose>0.0079209471698113206 0 -0.1808945358490566 0 0 0</pose>
@@ -256,5 +259,5 @@
         </inertia>
       </inertial>
-      <collision name='FL_calf_collision'>
+      <collision name='lower0_collision'>
         <pose>-0.002 0 -0.029999999999999999 0 1.2000000000000002 0</pose>
         <geometry>
@@ -264,5 +267,5 @@
         </geometry>
       </collision>
-      <collision name='FL_calf_collision_1'>
+      <collision name='lower0_collision_1'>
         <pose>0.021999999999999999 0 -0.10000000000000001 0 1.3500000000000001 0</pose>
         <geometry>
@@ -272,5 +275,5 @@
         </geometry>
       </collision>
-      <collision name='FL_calf_collision_2'>
+      <collision name='lower0_collision_2'>
         <pose>0.035999999999999997 0 -0.22500000000000001 0 1.530000000000008 0</pose>
         <geometry>
@@ -280,5 +283,5 @@
         </geometry>
       </collision>
-      <collision name='FL_calf_collision_3'>
+      <collision name='lower0_collision_3'>
         <pose>0.023 0 -0.31 3.1415926535897931 1.1415926535897938 3.1415926535897931</pose>
         <geometry>
@@ -288,5 +291,5 @@
         </geometry>
       </collision>
-      <collision name='FL_calf_fixed_joint_lump__FL_foot_collision_4'>
+      <collision name='lower0_fixed_joint_lump__FL_foot_collision_4'>
         <pose>0 0 -0.34999999999999998 1.5700000000000001 0 0</pose>
         <geometry>
@@ -296,10 +299,10 @@
         </geometry>
       </collision>
-      <visual name='FL_calf_visual'>
+      <visual name='lower0_visual'>
         <pose>0 0 0 0 0 0</pose>
         <geometry>
           <mesh>
             <scale>1 1 1</scale>
-            <uri>model://b2_description/meshes/FL_calf.dae</uri>
+            <uri>model://b2/meshes/FL_calf.dae</uri>
           </mesh>
         </geometry>
@@ -310,8 +313,93 @@
       </visual>
     </link>
-    <joint name='FR_hip_joint' type='revolute'>
-      <pose relative_to='base_link'>0.32850000000000001 -0.071999999999999995 0 0 0 0</pose>
-      <parent>base_link</parent>
-      <child>FR_hip</child>
+    <joint name='jtoe0' type='fixed'>
+      <pose relative_to='lower0'>0 0 -0.35 0 0 0</pose>
+      <parent>lower0</parent>
+      <child>toe0</child>
+      <axis>
+        <xyz>0 0 1</xyz>
+        <limit>
+          <lower>-1e+16</lower>
+          <upper>1e+16</upper>
+        </limit>
+        <dynamics>
+          <spring_reference>0</spring_reference>
+          <spring_stiffness>0</spring_stiffness>
+        </dynamics>
+      </axis>
+      <physics>
+        <ode>
+          <limit>
+            <cfm>0</cfm>
+            <erp>0.2</erp>
+          </limit>
+        </ode>
+      </physics>
+    </joint>
+    <link name="toe0">
+      <pose relative_to='jtoe0'>0 0 0 0 0 0</pose>
+      <inertial>
+        <pose xyz="-0.006511 0 -0.010144" rpy="0 0 0" />
+        <mass>0.126</mass>
+        <inertia
+          ixx="3.8E-05"
+          ixy="0"
+          ixz="1.1E-05"
+          iyy="4.1E-05"
+          iyz="0"
+          izz="4.2E-05" />
+      </inertial>
+      <visual name="toe0_visual">
+        <pose>0 0 0 0 0 0</pose>
+        <geometry>
+          <sphere>
+            <radius>0.032</radius>
+          </sphere>
+        </geometry>
+        <material>
+          <ambient>1 1 1 1</ambient>
+          <diffuse>1 1 1 1</diffuse>
+        </material>
+      </visual>
+      <collision name="toe0_collision">
+        <pose>0 0 0 0 0 0</pose>
+        <geometry>
+          <sphere>
+            <radius>0.032</radius>
+          </sphere>
+        </geometry>
+        <surface>
+          <contact>
+            <ode>
+              <kp>1e+06</kp>
+              <kd>1</kd>
+            </ode>
+          </contact>
+          <friction>
+            <ode>
+              <mu>0.6</mu>
+              <mu2>0.6</mu2>
+            </ode>
+          </friction>
+        </surface>
+      </collision>
+      <sensor name="toe0_contact" type="contact">
+        <alwaysOn>true</alwaysOn>
+        <updateRate>500</updateRate>
+        <topic>/gazebo/toe0_contact_state</topic>
+        <frameName>world</frameName>
+        <contact>
+          <collision>toe0_collision</collision>
+        </contact>
+        <plugin filename="libgz-sim8-contact-system.so" name="gz::sim::systems::Contact"> </plugin>
+      </sensor>
+      <gravity>1</gravity>
+      <velocity_decay/>
+      <self_collide>0</self_collide>
+    </link>
+    <joint name='10' type='revolute'>
+      <pose relative_to='body'>0.32850000000000001 -0.071999999999999995 0 0 0 0</pose>
+      <parent>body</parent>
+      <child>hip2</child>
       <axis>
         <xyz>1 0 0</xyz>
@@ -328,6 +416,6 @@
       </axis>
     </joint>
-    <link name='FR_hip'>
-      <pose relative_to='FR_hip_joint'>0 0 0 0 0 0</pose>
+    <link name='hip2'>
+      <pose relative_to='10'>0 0 0 0 0 0</pose>
       <inertial>
         <pose>-0.0084415778577246799 0.010019405376052131 0.00023950312245452079 0 0 0</pose>
@@ -342,5 +430,5 @@
         </inertia>
       </inertial>
-      <collision name='FR_hip_collision'>
+      <collision name='hip2_collision'>
         <pose>0 -0.12 0 1.5707963267948959 0 0</pose>
         <geometry>
@@ -351,5 +439,5 @@
         </geometry>
       </collision>
-      <collision name='FR_hip_fixed_joint_lump__FR_thigh_rotor_collision_1'>
+      <collision name='hip2_fixed_joint_lump__FR_thigh_rotor_collision_1'>
         <pose>0 0.0079799999999999992 0 1.5707963267948959 0 0</pose>
         <geometry>
@@ -360,10 +448,10 @@
         </geometry>
       </collision>
-      <visual name='FR_hip_visual'>
+      <visual name='hip2_visual'>
         <pose>0 0 0 0 0 0</pose>
         <geometry>
           <mesh>
             <scale>1 1 1</scale>
-            <uri>model://b2_description/meshes/FR_hip.dae</uri>
+            <uri>model://b2/meshes/FR_hip.dae</uri>
           </mesh>
         </geometry>
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