Commit message: Updated B2 Xacros

File: quad_simulator/b2_description/models/b2/urdf/b2.urdf.xacro (robot description, xacro)
@@ -4,7 +4,7 @@
      For more information, please see http://wiki.ros.org/sw_urdf_exporter -->
 <robot
-  name="b2_description">
-  <link
-    name="base_link">
+  name="b2">
+  <link
+    name="body">
     <inertial>
       <origin
@@ -27,5 +27,5 @@
       <geometry>
         <mesh
-          filename="package://b2_description/meshes/base_link.dae" />
+          filename="package://b2_description/models/b2/meshes/body.dae" />
       </geometry>
       <material
@@ -67,5 +67,5 @@
         <cylinder length="0.16" radius="0.076" />
         <!-- <mesh
-          filename="package://b2_description/meshes/lidar_link.STL" /> -->
+          filename="package://b2_description/models/b2/meshes/lidar_link.STL" /> -->
       </geometry>
     </collision>
@@ -78,5 +78,5 @@
       rpy="0 0 0" />
     <parent
-      link="base_link" />
+      link="body" />
     <child
       link="lidar_link" />
@@ -108,5 +108,5 @@
       rpy="-2.3562 0 -1.5708" />
     <parent
-      link="base_link" />
+      link="body" />
     <child
       link="f_dc_link" />
@@ -138,5 +138,5 @@
       rpy="-2.3557 0 1.5708" />
     <parent
-      link="base_link" />
+      link="body" />
     <child
       link="r_dc_link" />
@@ -168,5 +168,5 @@
       rpy="0 0 0" />
     <parent
-      link="base_link" />
+      link="body" />
     <child
       link="imu_link" />
@@ -206,5 +206,5 @@
       rpy="0 0 0" />
     <parent
-      link="base_link" />
+      link="body" />
     <child
       link="head_Link" />
@@ -244,5 +244,5 @@
       rpy="0 0 0" />
     <parent
-      link="base_link" />
+      link="body" />
     <child
       link="tail_link" />
@@ -251,5 +251,5 @@
   </joint>
   <link
-    name="FL_hip">
+    name="hip0">
     <inertial>
       <origin
@@ -272,5 +272,5 @@
       <geometry>
         <mesh
-          filename="package://b2_description/meshes/FL_hip.dae" />
+          filename="package://b2_description/models/b2/meshes/FL_hip.dae" />
       </geometry>
       <material
@@ -290,5 +290,5 @@
   </link>
   <joint
-    name="FL_hip_joint"
+    name="8"
     type="revolute">
     <origin
@@ -296,7 +296,7 @@
       rpy="0 0 0" />
     <parent
-      link="base_link" />
-    <child
-      link="FL_hip" />
+      link="body" />
+    <child
+      link="hip0" />
     <axis
       xyz="1 0 0" />
@@ -307,5 +307,5 @@
       velocity="23" />
   </joint>
-  <link name="FL_hip_rotor">
+  <link name="hip0_rotor">
     <!-- <visual>
       <origin rpy="0 1.5707963267948966 0" xyz="0 0 0"/>
@@ -326,11 +326,11 @@
     </inertial>
   </link>
-  <joint name="FL_hip_rotor_joint" type="fixed">
+  <joint name="hip0_rotor_joint" type="fixed">
     <origin rpy="0 0 0" xyz="0.20205 0.072 0"/>
-    <parent link="base_link"/>
-    <child link="FL_hip_rotor"/>
-  </joint>
-  <link
-    name="FL_thigh">
+    <parent link="body"/>
+    <child link="hip0_rotor"/>
+  </joint>
+  <link
+    name="upper0">
     <inertial>
       <origin
@@ -353,5 +353,5 @@
       <geometry>
         <mesh
-          filename="package://b2_description/meshes/FL_thigh.dae" />
+          filename="package://b2_description/models/b2/meshes/FL_thigh.dae" />
       </geometry>
       <material
@@ -371,22 +371,22 @@
   </link>
   <joint
-    name="FL_thigh_joint"
+    name="0"
     type="revolute">
     <origin
       xyz="0 0.11973 0"
-      rpy="0 0 0" />
-    <parent
-      link="FL_hip" />
-    <child
-      link="FL_thigh" />
-    <axis
-      xyz="0 1 0" />
+      rpy="0 1.57079632679 0" />
+    <parent
+      link="hip0" />
+    <child
+      link="upper0" />
+    <axis
+      xyz="0 -1 0" />
     <limit
-      lower="-0.94"
-      upper="4.69"
+      lower="-2.8012"
+      upper="2.8012"
       effort="200"
       velocity="23" />
   </joint>
-  <link name="FL_thigh_rotor">
+  <link name="upper0_rotor">
     <!-- <visual>
       <origin rpy="1.5707963267948966 0 0" xyz="0 0 0"/>
@@ -407,11 +407,11 @@
     </inertial>
   </link>
-  <joint name="FL_thigh_rotor_joint" type="fixed">
+  <joint name="upper0_rotor_joint" type="fixed">
     <origin rpy="0 0 0" xyz="0 -0.00798 0"/>
-    <parent link="FL_hip"/>
-    <child link="FL_thigh_rotor"/>
-  </joint>
-  <link
-    name="FL_calf">
+    <parent link="hip0"/>
+    <child link="upper0_rotor"/>
+  </joint>
+  <link
+    name="lower0">
     <inertial>
       <origin
@@ -434,5 +434,5 @@
       <geometry>
         <mesh
-          filename="package://b2_description/meshes/FL_calf.dae" />
+          filename="package://b2_description/models/b2/meshes/FL_calf.dae" />
       </geometry>
       <material
@@ -468,22 +468,22 @@
   </link>
   <joint
-    name="FL_calf_joint"
+    name="1"
     type="revolute">
     <origin
       xyz="0 -8.6984E-05 -0.35"
-      rpy="0 0 0" />
-    <parent
-      link="FL_thigh" />
-    <child
-      link="FL_calf" />
+      rpy="0 -3.14159265359 0" />
+    <parent
+      link="upper0" />
+    <child
+      link="lower0" />
     <axis
       xyz="0 1 0" />
     <limit
-      lower="-2.82"
-      upper="-0.43"
+      lower="0.32159265359"
+      upper="2.71159265359"
       effort="320"
       velocity="14" />
   </joint>
-  <link name="FL_calf_rotor">
+  <link name="lower0_rotor">
     <!-- <visual>
       <origin rpy="1.5707963267948966 0 0" xyz="0 0 0"/>
@@ -504,11 +504,11 @@
     </inertial>
   </link>
-  <joint name="FL_calf_rotor_joint" type="fixed">
+  <joint name="lower0_rotor_joint" type="fixed">
     <origin rpy="0 0 0" xyz="0 -0.05788 0"/>
-    <parent link="FL_thigh"/>
-    <child link="FL_calf_rotor"/>
-  </joint>
-  <link
-    name="FL_foot">
+    <parent link="upper0"/>
+    <child link="lower0_rotor"/>
+  </joint>
+  <link
+    name="toe0">
     <inertial>
       <origin
@@ -535,5 +535,5 @@
   </link>
   <joint
-    name="FL_foot_joint"
+    name="jtoe0"
     type="fixed">
     <origin
@@ -541,10 +541,10 @@
       rpy="0 0 0" />
     <parent
-      link="FL_calf" />
-    <child
-      link="FL_foot" />
-  </joint>
-  <link
-    name="FR_hip">
+      link="lower0" />
+    <child
+      link="toe0" />
+  </joint>
+  <link
+    name="hip2">
     <inertial>
       <origin
@@ -567,5 +567,5 @@
       <geometry>
         <mesh
-          filename="package://b2_description/meshes/FR_hip.dae" />
+          filename="package://b2_description/models/b2/meshes/FR_hip.dae" />
       </geometry>
       <material
@@ -585,5 +585,5 @@
   </link>
   <joint
-    name="FR_hip_joint"
+    name="10"
     type="revolute">
     <origin
@@ -591,7 +591,7 @@
       rpy="0 0 0" />
     <parent
-      link="base_link" />
-    <child
-      link="FR_hip" />
+      link="body" />
+    <child
+      link="hip2" />
     <axis
       xyz="1 0 0" />
@@ -602,5 +602,5 @@
       velocity="23" />
   </joint>
-  <link name="FR_hip_rotor">
+  <link name="hip2_rotor">
     <!-- <visual>
       <origin rpy="0 1.5707963267948966 0" xyz="0 0 0"/>
@@ -621,11 +621,11 @@
     </inertial>
   </link>
-  <joint name="FR_hip_rotor_joint" type="fixed">
+  <joint name="hip2_rotor_joint" type="fixed">
     <origin rpy="0 0 0" xyz="0.20205 -0.072 0"/>
-    <parent link="base_link"/>
-    <child link="FR_hip_rotor"/>
-  </joint>
-  <link
-    name="FR_thigh">
+    <parent link="body"/>
+    <child link="hip2_rotor"/>
+  </joint>
+  <link
+    name="upper2">
     <inertial>
       <origin
@@ -648,5 +648,5 @@
       <geometry>
         <mesh
-          filename="package://b2_description/meshes/FR_thigh.dae" />
+          filename="package://b2_description/models/b2/meshes/FR_thigh.dae" />
       </geometry>
       <material
@@ -664,22 +664,22 @@
   </link>
   <joint
-    name="FR_thigh_joint"
+    name="4"
     type="revolute">
     <origin
       xyz="0 -0.11973 0"
-      rpy="0 0 0" />
-    <parent
-      link="FR_hip" />
-    <child
-      link="FR_thigh" />
-    <axis
-      xyz="0 1 0" />
+      rpy="0 1.57079632679 0" />
+    <parent
+      link="hip2" />
+    <child
+      link="upper2" />
+    <axis
+      xyz="0 -1 0" />
     <limit
-      lower="-0.94"
-      upper="4.69"
+      lower="-2.8012"
+      upper="2.8012"
       effort="200"
       velocity="23" />
   </joint>
-  <link name="FR_thigh_rotor">
+  <link name="upper2_rotor">
     <!-- <visual>
       <origin rpy="1.5707963267948966 0 0" xyz="0 0 0"/>
@@ -700,11 +700,11 @@
     </inertial>
   </link>
-  <joint name="FR_thigh_rotor_joint" type="fixed">
+  <joint name="upper2_rotor_joint" type="fixed">
     <origin rpy="0 0 0" xyz="0 0.00798 0"/>
-    <parent link="FR_hip"/>
-    <child link="FR_thigh_rotor"/>
-  </joint>
-  <link
-    name="FR_calf">
+    <parent link="hip2"/>
+    <child link="upper2_rotor"/>
+  </joint>
+  <link
+    name="lower2">
     <inertial>
       <origin
@@ -727,5 +727,5 @@
       <geometry>
         <mesh
-          filename="package://b2_description/meshes/FR_calf.dae" />
+          filename="package://b2_description/models/b2/meshes/FR_calf.dae" />
       </geometry>
       <material
@@ -761,22 +761,22 @@
   </link>
   <joint
-    name="FR_calf_joint"
+    name="5"
     type="revolute">
     <origin
       xyz="0 8.6986E-05 -0.35"
-      rpy="0 0 0" />
-    <parent
-      link="FR_thigh" />
-    <child
-      link="FR_calf" />
+      rpy="0 -3.14159265359 0" />
+    <parent
+      link="upper2" />
+    <child
+      link="lower2" />
     <axis
       xyz="0 1 0" />
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
Commit message: Global Planner Updates

File: quad_simulator/b2_description/models/b2/b2.sdf.xacro (robot description, xacro)
@@ -173,6 +173,6 @@
           <lower>-2.8012</lower>
           <upper>2.8012</upper>
-          <effort>200</effort>
-          <velocity>23</velocity>
+          <effort>200.0</effort>
+          <velocity>23.0</velocity>
         </limit>
         <dynamics>
@@ -340,13 +340,14 @@
       <pose relative_to='jtoe0'>0 0 0 0 0 0</pose>
       <inertial>
-        <pose xyz="-0.006511 0 -0.010144" rpy="0 0 0" />
+        <pose> -0.006511 0 -0.010144 0 0 0</pose>
         <mass>0.126</mass>
-        <inertia
-          ixx="3.8E-05"
-          ixy="0"
-          ixz="1.1E-05"
-          iyy="4.1E-05"
-          iyz="0"
-          izz="4.2E-05" />
+        <inertia>
+          <ixx>3.8e-05</ixx>
+          <ixy>1e-6</ixy>
+          <ixz>1.1e-05</ixz>
+          <iyy>4.1e-05</iyy>
+          <iyz>1e-6</iyz>
+          <izz>4.2e-05</izz>
+        </inertia>
       </inertial>
       <visual name="toe0_visual">
@@ -471,6 +472,6 @@
           <lower>-2.8012</lower>
           <upper>2.8012</upper>
-          <effort>200</effort>
-          <velocity>23</velocity>
+          <effort>200.0</effort>
+          <velocity>23.0</velocity>
         </limit>
         <dynamics>
@@ -638,13 +639,14 @@
       <pose relative_to='jtoe2'>0 0 0 0 0 0</pose>
       <inertial>
-        <pose xyz="-0.006511 0 -0.010144" rpy="0 0 0" />
+        <pose> -0.006511 0 -0.010144 0 0 0</pose>
         <mass>0.126</mass>
-        <inertia
-          ixx="3.8E-05"
-          ixy="0"
-          ixz="1.1E-05"
-          iyy="4.1E-05"
-          iyz="0"
-          izz="4.2E-05" />
+        <inertia>
+          <ixx>3.8e-05</ixx>
+          <ixy>1e-6</ixy>
+          <ixz>1.1e-05</ixz>
+          <iyy>4.1e-05</iyy>
+          <iyz>1e-6</iyz>
+          <izz>4.2e-05</izz>
+        </inertia>
       </inertial>
       <visual name="toe2_visual">
@@ -769,6 +771,6 @@
           <lower>-2.8012</lower>
           <upper>2.8012</upper>
-          <effort>200</effort>
-          <velocity>23</velocity>
+          <effort>200.0</effort>
+          <velocity>23.0</velocity>
         </limit>
         <dynamics>
@@ -936,13 +938,14 @@
       <pose relative_to='jtoe1'>0 0 0 0 0 0</pose>
       <inertial>
-        <pose xyz="-0.006511 0 -0.010144" rpy="0 0 0" />
+        <pose> -0.006511 0 -0.010144 0 0 0</pose>
         <mass>0.126</mass>
-        <inertia
-          ixx="3.8E-05"
-          ixy="0"
-          ixz="1.1E-05"
-          iyy="4.1E-05"
-          iyz="0"
-          izz="4.2E-05" />
+        <inertia>
+          <ixx>3.8e-05</ixx>
+          <ixy>1e-6</ixy>
+          <ixz>1.1e-05</ixz>
+          <iyy>4.1e-05</iyy>
+          <iyz>1e-6</iyz>
+          <izz>4.2e-05</izz>
+        </inertia>
       </inertial>
       <visual name="toe1_visual">
@@ -1067,6 +1070,6 @@
           <lower>-2.8012</lower>
           <upper>2.8012</upper>
-          <effort>200</effort>
-          <velocity>23</velocity>
+          <effort>200.0</effort>
+          <velocity>23.0</velocity>
         </limit>
         <dynamics>
@@ -1234,13 +1237,14 @@
       <pose relative_to='jtoe3'>0 0 0 0 0 0</pose>
       <inertial>
-        <pose xyz="-0.006511 0 -0.010144" rpy="0 0 0" />
+        <pose> -0.006511 0 -0.010144 0 0 0</pose>
         <mass>0.126</mass>
-        <inertia
-          ixx="3.8E-05"
-          ixy="0"
-          ixz="1.1E-05"
-          iyy="4.1E-05"
-          iyz="0"
-          izz="4.2E-05" />
+        <inertia>
+          <ixx>3.8e-05</ixx>
+          <ixy>1e-6</ixy>
+          <ixz>1.1e-05</ixz>
+          <iyy>4.1e-05</iyy>
+          <iyz>1e-6</iyz>
+          <izz>4.2e-05</izz>
+        </inertia>
       </inertial>
       <visual name="toe3_visual">

File: quad_simulator/b2_description/models/b2/urdf/b2.urdf.xacro (robot description, xacro)
@@ -385,6 +385,6 @@
       lower="-2.8012"
       upper="2.8012"
-      effort="200"
-      velocity="23" />
+      effort="200.0"
+      velocity="23.0" />
   </joint>
   <link name="upper0_rotor">
@@ -678,6 +678,6 @@
       lower="-2.8012"
       upper="2.8012"
-      effort="200"
-      velocity="23" />
+      effort="200.0"
+      velocity="23.0" />
   </joint>
   <link name="upper2_rotor">
@@ -972,6 +972,6 @@
       lower="-2.8012"
       upper="2.8012"
-      effort="200"
-      velocity="23" />
+      effort="200.0"
+      velocity="23.0" />
   </joint>
   <link name="upper1_rotor">
@@ -1265,6 +1265,6 @@
       lower="-2.8012"
       upper="2.8012"
-      effort="200"
-      velocity="23" />
+      effort="200.0"
+      velocity="23.0" />
   </joint>
   <link name="upper3_rotor">

Commit message: Working B2 Robot, Stand Joint Angles Need Work, Maybe Up the Kp on the hip joint

File: quad_simulator/b2_description/models/b2/b2.sdf.xacro (robot description, xacro)
@@ -165,12 +165,12 @@
     </link>
     <joint name='0' type='revolute'>
-      <pose relative_to='hip0'>0 0.11973 0 0 1.5708 0</pose>
+      <pose relative_to='hip0'>0 0.11973 0 0 0 0</pose>
       <parent>hip0</parent>
       <child>upper0</child>
       <axis>
-        <xyz>0 -1 0</xyz>
-        <limit>
-          <lower>-2.8012</lower>
-          <upper>2.8012</upper>
+        <xyz>0 1 0</xyz>
+        <limit>
+          <lower>-0.94</lower>
+          <upper>4.69</upper>
           <effort>200.0</effort>
           <velocity>23.0</velocity>
@@ -228,5 +228,5 @@
     </link>
     <joint name='1' type='revolute'>
-      <pose relative_to='upper0'>0 -8.6984000000000006e-05 -0.34999999999999998 -3.14159 0 -3.14159</pose>
+      <pose relative_to='upper0'>0 -8.6984000000000006e-05 -0.34999999999999998 0 0 0</pose>
       <parent>upper0</parent>
       <child>lower0</child>
@@ -234,6 +234,6 @@
         <xyz>0 1 0</xyz>
         <limit>
-          <lower>0.32159265359</lower>
-          <upper>2.71159265359</upper>
+          <lower>-2.82</lower>
+          <upper>-0.43</upper>
           <effort>320</effort>
           <velocity>14</velocity>
@@ -464,12 +464,12 @@
     </link>
     <joint name='4' type='revolute'>
-      <pose relative_to='hip2'>0 -0.11973 0 0 1.5708 0</pose>
+      <pose relative_to='hip2'>0 -0.11973 0 0 0 0</pose>
       <parent>hip2</parent>
       <child>upper2</child>
       <axis>
-        <xyz>0 -1 0</xyz>
-        <limit>
-          <lower>-2.8012</lower>
-          <upper>2.8012</upper>
+        <xyz>0 1 0</xyz>
+        <limit>
+          <lower>-0.94</lower>
+          <upper>4.69</upper>
           <effort>200.0</effort>
           <velocity>23.0</velocity>
@@ -527,5 +527,5 @@
     </link>
     <joint name='5' type='revolute'>
-      <pose relative_to='upper2'>0 8.6985999999999997e-05 -0.34999999999999998 -3.14159 0 -3.14159</pose>
+      <pose relative_to='upper2'>0 8.6985999999999997e-05 -0.34999999999999998 0 0 0</pose>
       <parent>upper2</parent>
       <child>lower2</child>
@@ -533,6 +533,6 @@
         <xyz>0 1 0</xyz>
         <limit>
-          <lower>0.32159265359</lower>
-          <upper>2.71159265359</upper>
+          <lower>-2.82</lower>
+          <upper>-0.43</upper>
           <effort>320</effort>
           <velocity>14</velocity>
@@ -763,12 +763,12 @@
     </link>
     <joint name='2' type='revolute'>
-      <pose relative_to='hip1'>0 0.11973 0 0 1.5708 0</pose>
+      <pose relative_to='hip1'>0 0.11973 0 0 0 0</pose>
       <parent>hip1</parent>
       <child>upper1</child>
       <axis>
-        <xyz>0 -1 0</xyz>
-        <limit>
-          <lower>-2.8012</lower>
-          <upper>2.8012</upper>
+        <xyz>0 1 0</xyz>
+        <limit>
+          <lower>-0.94</lower>
+          <upper>4.69</upper>
           <effort>200.0</effort>
           <velocity>23.0</velocity>
@@ -826,5 +826,5 @@
     </link>
     <joint name='3' type='revolute'>
-      <pose relative_to='upper1'>0 -8.6984000000000006e-05 -0.34999999999999998 -3.14159 0 -3.14159</pose>
+      <pose relative_to='upper1'>0 -8.6984000000000006e-05 -0.34999999999999998 0 0 0</pose>
       <parent>upper1</parent>
       <child>lower1</child>
@@ -832,6 +832,6 @@
         <xyz>0 1 0</xyz>
         <limit>
-          <lower>0.32159265359</lower>
-          <upper>2.71159265359</upper>
+          <lower>-2.82</lower>
+          <upper>-0.43</upper>
           <effort>320</effort>
           <velocity>14</velocity>
@@ -1062,12 +1062,12 @@
     </link>
     <joint name='6' type='revolute'>
-      <pose relative_to='hip3'>0 -0.11973 0 0 1.5708 0</pose>
+      <pose relative_to='hip3'>0 -0.11973 0 0 0 0</pose>
       <parent>hip3</parent>
       <child>upper3</child>
       <axis>
-        <xyz>0 -1 0</xyz>
-        <limit>
-          <lower>-2.8012</lower>
-          <upper>2.8012</upper>
+        <xyz>0 1 0</xyz>
+        <limit>
+          <lower>-0.94</lower>
+          <upper>4.69</upper>
           <effort>200.0</effort>
           <velocity>23.0</velocity>
@@ -1125,5 +1125,5 @@
     </link>
     <joint name='7' type='revolute'>
-      <pose relative_to='upper3'>0 8.6985999999999997e-05 -0.34999999999999998 -3.14159 0 -3.14159</pose>
+      <pose relative_to='upper3'>0 8.6985999999999997e-05 -0.34999999999999998 0 0 0</pose>
       <parent>upper3</parent>
       <child>lower3</child>
@@ -1131,6 +1131,6 @@
         <xyz>0 1 0</xyz>
         <limit>
-          <lower>0.32159265359</lower>
-          <upper>2.71159265359</upper>
+          <lower>-2.82</lower>
+          <upper>-0.43</upper>
           <effort>320</effort>
           <velocity>14</velocity>

File: quad_simulator/b2_description/models/b2/urdf/b2.urdf.xacro (robot description, xacro)
@@ -375,5 +375,5 @@
     <origin
       xyz="0 0.11973 0"
-      rpy="0 1.57079632679 0" />
+      rpy="0 0 0" />
     <parent
       link="hip0" />
@@ -381,8 +381,8 @@
       link="upper0" />
     <axis
-      xyz="0 -1 0" />
+      xyz="0 1 0" />
     <limit
-      lower="-2.8012"
-      upper="2.8012"
+      lower="-0.94"
+      upper="4.69"
       effort="200.0"
       velocity="23.0" />
@@ -472,5 +472,5 @@
     <origin
       xyz="0 -8.6984E-05 -0.35"
-      rpy="0 -3.14159265359 0" />
+      rpy="0 0 0" />
     <parent
       link="upper0" />
@@ -480,6 +480,6 @@
       xyz="0 1 0" />
     <limit
-      lower="0.32159265359"
-      upper="2.71159265359"
+      lower="-2.82"
+      upper="-0.43"
       effort="320"
       velocity="14" />
@@ -668,5 +668,5 @@
     <origin
       xyz="0 -0.11973 0"
-      rpy="0 1.57079632679 0" />
+      rpy="0 0 0" />
     <parent
       link="hip2" />
@@ -674,8 +674,8 @@
       link="upper2" />
     <axis
-      xyz="0 -1 0" />
+      xyz="0 1 0" />
     <limit
-      lower="-2.8012"
-      upper="2.8012"
+      lower="-0.94"
+      upper="4.69"
       effort="200.0"
       velocity="23.0" />
@@ -765,5 +765,5 @@
     <origin
       xyz="0 8.6986E-05 -0.35"
-      rpy="0 -3.14159265359 0" />
+      rpy="0 0 0" />
     <parent
       link="upper2" />
@@ -773,6 +773,6 @@
       xyz="0 1 0" />
     <limit
-      lower="0.32159265359"
-      upper="2.71159265359"
+      lower="-2.82"
+      upper="-0.43"
       effort="320"
       velocity="14" />
@@ -962,5 +962,5 @@
     <origin
       xyz="0 0.11973 0"
-      rpy="0 1.57079632679 0" />
+      rpy="0 0 0" />
     <parent
       link="hip1" />
@@ -968,8 +968,8 @@
       link="upper1" />
     <axis
-      xyz="0 -1 0" />
+      xyz="0 1 0" />
     <limit
-      lower="-2.8012"
-      upper="2.8012"
+      lower="-0.94"
+      upper="4.69"
       effort="200.0"
       velocity="23.0" />
@@ -1059,5 +1059,5 @@
     <origin
       xyz="0 -8.6984E-05 -0.35"
-      rpy="0 -3.14159265359 0" />
+      rpy="0 0 0" />
     <parent
       link="upper1" />
@@ -1067,6 +1067,6 @@
       xyz="0 1 0" />
     <limit
-      lower="0.32159265359"
-      upper="2.71159265359"
+      lower="-2.82"
+      upper="-0.43"
       effort="320"
       velocity="14" />
@@ -1255,5 +1255,5 @@
     <origin
       xyz="0 -0.11973 0"
-      rpy="0 1.57079632679 0" />
+      rpy="0 0 0" />
     <parent
       link="hip3" />
@@ -1261,8 +1261,8 @@
       link="upper3" />
     <axis
-      xyz="0 -1 0" />
+      xyz="0 1 0" />
     <limit
-      lower="-2.8012"
-      upper="2.8012"
+      lower="-0.94"
+      upper="4.69"
       effort="200.0"
       velocity="23.0" />
@@ -1352,5 +1352,5 @@
     <origin
       xyz="0 8.6986E-05 -0.35"
-      rpy="0 -3.14159265359 0" />
+      rpy="0 0 0" />
     <parent
       link="upper3" />
@@ -1360,6 +1360,6 @@
       xyz="0 1 0" />
     <limit
-      lower="0.32159265359"
-      upper="2.71159265359"
+      lower="-2.82"
+      upper="-0.43"
       effort="320"
       velocity="14" />
