Commit message: Working Joint State Broadcaster, Joint Controller

File: quad_simulator/go2_description/models/go2/urdf/go2.urdf.xacro (robot description, xacro)
@@ -4,8 +4,7 @@
      Commit Version: 1.6.0-4-g7f85cfe  Build Version: 1.6.7995.38578
      For more information, please see http://wiki.ros.org/sw_urdf_exporter -->
-<robot
-  name="go2_description">
-  <link
-    name="base">
+<robot name="go2" xmlns:xacro="http://www.ros.org/wiki/xacro">
+  <link
+    name="body">
     <inertial>
       <origin
@@ -28,5 +27,5 @@
       <geometry>
         <mesh
-          filename="package://go2_description/dae/base.dae" />
+          filename="package://go2_description/models/go2/dae/body.dae" />
       </geometry>
       <material
@@ -75,5 +74,5 @@
       rpy="0 0 0" />
     <parent
-      link="base" />
+      link="body" />
     <child
       link="Head_upper" />
@@ -120,5 +119,5 @@
   </joint>
   <link
-    name="FL_hip">
+    name="hip0">
     <inertial>
       <origin
@@ -141,5 +140,5 @@
       <geometry>
         <mesh
-          filename="package://go2_description/dae/hip.dae" />
+          filename="package://go2_description/models/go2/dae/hip.dae" />
       </geometry>
       <material
@@ -157,5 +156,5 @@
   </link>
   <joint
-    name="FL_hip_joint"
+    name="8"
     type="revolute">
     <origin
@@ -163,7 +162,7 @@
       rpy="0 0 0" />
     <parent
-      link="base" />
-    <child
-      link="FL_hip" />
+      link="body" />
+    <child
+      link="hip0" />
     <axis
       xyz="1 0 0" />
@@ -174,5 +173,5 @@
       velocity="30.1" />
   </joint>
-  <link name="FL_hip_rotor">
+  <link name="hip0_rotor">
     <inertial>
       <origin rpy="0 0 0" xyz="0.0 0.0 0.0"/>
@@ -181,11 +180,11 @@
     </inertial>
   </link>
-  <joint name="FL_hip_rotor_joint" type="fixed">
+  <joint name="hip0_rotor_joint" type="fixed">
     <origin rpy="0 0 0" xyz="0.11215 0.04675 0"/>
-    <parent link="base"/>
-    <child link="FL_hip_rotor"/>
-  </joint>
-  <link
-    name="FL_thigh">
+    <parent link="body"/>
+    <child link="hip0_rotor"/>
+  </joint>
+  <link
+    name="upper0">
     <inertial>
       <origin
@@ -208,5 +207,5 @@
       <geometry>
         <mesh
-          filename="package://go2_description/dae/thigh.dae" />
+          filename="package://go2_description/models/go2/dae/thigh.dae" />
       </geometry>
       <material
@@ -224,5 +223,5 @@
   </link>
   <joint
-    name="FL_thigh_joint"
+    name="0"
     type="revolute">
     <origin
@@ -230,7 +229,7 @@
       rpy="0 0 0" />
     <parent
-      link="FL_hip" />
-    <child
-      link="FL_thigh" />
+      link="hip0" />
+    <child
+      link="upper0" />
     <axis
       xyz="0 1 0" />
@@ -241,5 +240,5 @@
       velocity="30.1" />
   </joint>
-  <link name="FL_thigh_rotor">
+  <link name="upper0_rotor">
     <inertial>
       <origin rpy="0 0 0" xyz="0.0 0.0 0.0"/>
@@ -248,11 +247,11 @@
     </inertial>
   </link>
-  <joint name="FL_thigh_rotor_joint" type="fixed">
+  <joint name="upper0_rotor_joint" type="fixed">
     <origin rpy="0 0 0" xyz="0 -0.00015 0"/>
-    <parent link="FL_hip"/>
-    <child link="FL_thigh_rotor"/>
-  </joint>
-  <link
-    name="FL_calf">
+    <parent link="hip0"/>
+    <child link="upper0_rotor"/>
+  </joint>
+  <link
+    name="lower0">
     <inertial>
       <origin
@@ -275,5 +274,5 @@
       <geometry>
         <mesh
-          filename="package://go2_description/dae/calf.dae" />
+          filename="package://go2_description/models/go2/dae/calf.dae" />
       </geometry>
       <material
@@ -291,5 +290,5 @@
   </link>
   <joint
-    name="FL_calf_joint"
+    name="1"
     type="revolute">
     <origin
@@ -297,7 +296,7 @@
       rpy="0 0 0" />
     <parent
-      link="FL_thigh" />
-    <child
-      link="FL_calf" />
+      link="upper0" />
+    <child
+      link="lower0" />
     <axis
       xyz="0 1 0" />
@@ -309,5 +308,5 @@
   </joint>
   <link
-    name="FL_calflower">
+    name="lower0_lower">
     <collision>
       <origin rpy="0 0 0" xyz="0 0 0" />
@@ -318,5 +317,5 @@
   </link>
   <joint
-    name="FL_calflower_joint"
+    name="lower0_lower_joint"
     type="fixed">
     <origin
@@ -324,12 +323,12 @@
       rpy="0 0.05 0" />
     <parent
-      link="FL_calf" />
-    <child
-      link="FL_calflower" />
-    <axis
-      xyz="0 0 0" />
-  </joint>
-  <link
-    name="FL_calflower1">
+      link="lower0" />
+    <child
+      link="lower0_lower" />
+    <axis
+      xyz="0 0 0" />
+  </joint>
+  <link
+    name="lower0_lower1">
     <collision>
       <origin rpy="0 0 0" xyz="0 0 0" />
@@ -340,5 +339,5 @@
   </link>
   <joint
-    name="FL_calflower1_joint"
+    name="lower0_lower1_joint"
     type="fixed">
     <origin
@@ -346,11 +345,11 @@
       rpy="0 0.48 0" />
     <parent
-      link="FL_calflower" />
-    <child
-      link="FL_calflower1" />
-    <axis
-      xyz="0 0 0" />
-  </joint>
-  <link name="FL_calf_rotor">
+      link="lower0_lower" />
+    <child
+      link="lower0_lower1" />
+    <axis
+      xyz="0 0 0" />
+  </joint>
+  <link name="lower0_rotor">
     <inertial>
       <origin rpy="0 0 0" xyz="0.0 0.0 0.0"/>
@@ -359,11 +358,11 @@
     </inertial>
   </link>
-  <joint name="FL_calf_rotor_joint" type="fixed">
+  <joint name="lower0_rotor_joint" type="fixed">
     <origin rpy="0 0 0" xyz="0 -0.03235 0"/>
-    <parent link="FL_thigh"/>
-    <child link="FL_calf_rotor"/>
-  </joint>
-  <link
-    name="FL_foot">
+    <parent link="upper0"/>
+    <child link="lower0_rotor"/>
+  </joint>
+  <link
+    name="toe0">
     <inertial>
       <origin
@@ -386,5 +385,5 @@
       <geometry>
         <mesh
-          filename="package://go2_description/dae/foot.dae" />
+          filename="package://go2_description/models/go2/dae/foot.dae" />
       </geometry>
       <material
@@ -402,5 +401,5 @@
   </link>
   <joint
-    name="FL_foot_joint"
+    name="jtoe0"
     type="fixed" dont_collapse="true">
     <origin
@@ -408,12 +407,12 @@
       rpy="0 0 0" />
     <parent
-      link="FL_calf" />
-    <child
-      link="FL_foot" />
-    <axis
-      xyz="0 0 0" />
-  </joint>
-  <link
-    name="FR_hip">
+      link="lower0" />
+    <child
+      link="toe0" />
+    <axis
+      xyz="0 0 0" />
+  </joint>
+  <link
+    name="hip2">
     <inertial>
       <origin
@@ -436,5 +435,5 @@
       <geometry>
         <mesh
-          filename="package://go2_description/dae/hip.dae" />
+          filename="package://go2_description/models/go2/dae/hip.dae" />
       </geometry>
       <material
@@ -452,5 +451,5 @@
   </link>
   <joint
-    name="FR_hip_joint"
+    name="10"
     type="revolute">
     <origin
@@ -458,7 +457,7 @@
       rpy="0 0 0" />
     <parent
-      link="base" />
-    <child
-      link="FR_hip" />
+      link="body" />
+    <child
+      link="hip2" />
     <axis
       xyz="1 0 0" />
@@ -469,5 +468,5 @@
       velocity="30.1" />
   </joint>
-  <link name="FR_hip_rotor">
+  <link name="hip2_rotor">
     <inertial>
       <origin rpy="0 0 0" xyz="0.0 0.0 0.0"/>
@@ -476,11 +475,11 @@
     </inertial>
   </link>
-  <joint name="FR_hip_rotor_joint" type="fixed">
+  <joint name="hip2_rotor_joint" type="fixed">
     <origin rpy="0 0 0" xyz="0.11215 -0.04675 0"/>
-    <parent link="base"/>
-    <child link="FR_hip_rotor"/>
-  </joint>
-  <link
-    name="FR_thigh">
+    <parent link="body"/>
+    <child link="hip2_rotor"/>
+  </joint>
+  <link
+    name="upper2">
     <inertial>
       <origin
@@ -503,5 +502,5 @@
       <geometry>
         <mesh
-          filename="package://go2_description/dae/thigh_mirror.dae" />
+          filename="package://go2_description/models/go2/dae/thigh_mirror.dae" />
       </geometry>
       <material
@@ -519,5 +518,5 @@
   </link>
   <joint
-    name="FR_thigh_joint"
+    name="4"
     type="revolute">
     <origin
@@ -525,7 +524,7 @@
       rpy="0 0 0" />
     <parent
-      link="FR_hip" />
-    <child
-      link="FR_thigh" />
+      link="hip2" />
+    <child
+      link="upper2" />
     <axis
       xyz="0 1 0" />
@@ -536,5 +535,5 @@
       velocity="30.1" />
   </joint>
-  <link name="FR_thigh_rotor">
+  <link name="upper2_rotor">
     <inertial>
       <origin rpy="0 0 0" xyz="0.0 0.0 0.0"/>
@@ -543,11 +542,11 @@
     </inertial>
   </link>
-  <joint name="FR_thigh_rotor_joint" type="fixed">
+  <joint name="upper2_rotor_joint" type="fixed">
     <origin rpy="0 0 0" xyz="0 0.00015 0"/>
-    <parent link="FR_hip"/>
-    <child link="FR_thigh_rotor"/>
-  </joint>
-  <link
-    name="FR_calf">
+    <parent link="hip2"/>
+    <child link="upper2_rotor"/>
+  </joint>
+  <link
+    name="lower2">
     <inertial>
       <origin
@@ -570,5 +569,5 @@
       <geometry>
         <mesh
-          filename="package://go2_description/dae/calf_mirror.dae" />
+          filename="package://go2_description/models/go2/dae/calf_mirror.dae" />
       </geometry>
       <material
@@ -586,5 +585,5 @@
   </link>
   <joint
-    name="FR_calf_joint"
+    name="5"
     type="revolute">
     <origin
@@ -592,7 +591,7 @@
       rpy="0 0 0" />
     <parent
-      link="FR_thigh" />
-    <child
-      link="FR_calf" />
+      link="upper2" />
+    <child
+      link="lower2" />
     <axis
       xyz="0 1 0" />
@@ -604,5 +603,5 @@
   </joint>
   <link
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
File: quad_simulator/go2_description/models/go2/xacro/leg.xacro (robot description, xacro)
@@ -1,5 +1,5 @@
 <?xml version="1.0"?>
 <robot xmlns:xacro="http://www.ros.org/wiki/xacro">
-    <xacro:include filename="$(find go2_description)/xacro/transmission.xacro"/>
+    <xacro:include filename="$(find go2_description)/models/go2/xacro/transmission.xacro"/>
     <xacro:macro name="leg" params="name mirror mirror_dae front_hind front_hind_dae">
         <joint name="${name}_hip_joint" type="revolute">

File: quad_simulator/go2_description/models/go2/xacro/robot.xacro (robot description, xacro)
@@ -2,9 +2,9 @@
 <robot name="go2" xmlns:xacro="http://www.ros.org/wiki/xacro">
     <xacro:arg name="DEBUG" default="false"/>
-    <xacro:include filename="$(find go2_description)/xacro/const.xacro"/>
-    <xacro:include filename="$(find go2_description)/xacro/materials.xacro"/>
-    <xacro:include filename="$(find go2_description)/xacro/leg.xacro"/>
+    <xacro:include filename="$(find go2_description)/models/go2/xacro/const.xacro"/>
+    <xacro:include filename="$(find go2_description)/models/go2/xacro/materials.xacro"/>
+    <xacro:include filename="$(find go2_description)/models/go2/xacro/leg.xacro"/>
     <!-- <xacro:include filename="$(find go2_description)/xacro/stairs.xacro"/> -->
-    <xacro:include filename="$(find go2_description)/xacro/gazebo.xacro"/>
+    <xacro:include filename="$(find go2_description)/models/go2/xacro/gazebo.xacro"/>
     <!-- <xacro:include filename="$(find go2_gazebo)/launch/stairs.urdf.xacro"/> -->
     <!-- <xacro:stairs stairs="15" xpos="0" ypos="0" zpos="0" /> -->
