Commit message: Working Joint State Broadcaster, Joint Controller

File: quad_simulator/spirit_description/models/spirit/urdf/spirit.urdf.xacro (robot description, xacro)
@@ -1,9 +1,6 @@
-<?xml version="1.0"?>
+<?xml version="1.0" encoding="utf-8"?>
 <!--
 MIT License (modified)
-Copyright (c) 2020 Ghost Robotics
-Authors:
-Avik De <avik@ghostrobotics.io>
-Tom Jacobs <tom.jacobs@ghostrobotics.io>
+Copyright (c) 2022 Ghost Robotics
 Permission is hereby granted, free of charge, to any person obtaining a copy
 of this **file** (the "Software"), to deal
@@ -22,208 +19,1021 @@
 SOFTWARE.
 -->
-<robot xmlns:xacro="http://www.ros.org/wiki/xacro" name="ngr">
-	<!-- Define parameters -->
-	<!-- bodyLength + hipdx should be equal to front to back hip distance -->
-	<!-- dy +  dPodAxisToEdge + upperLegWidth should be equal to the center to toe distance along y axis-->
-	<xacro:property name="pi" value="3.14159265359"/>
-	<xacro:property name="bodyLength" value="0.335"/>
-	<xacro:property name="bodyWidth" value="0.24"/>
-	<xacro:property name="bodyHeight" value="0.104"/>
-	<xacro:property name="bodyMass" value="5.75"/>
-	<xacro:property name="podMass" value="0.575"/>
-	<xacro:property name="upperLegMass" value="0.775"/>
-	<xacro:property name="upperLegIxx" value="0.00005"/> <!-- guess -->
-	<xacro:property name="upperLegIyy" value="0.001"/> <!-- guess -->
-	<xacro:property name="upperLegIzz" value="0.001"/> <!-- guess -->
-	<xacro:property name="lowerLegMass" value="0.075"/>
-	<xacro:property name="lowerLegIxx" value="0.000005"/> <!-- guess -->
-	<xacro:property name="lowerLegIyy" value="0.0001"/> <!-- guess -->
-	<xacro:property name="lowerLegIzz" value="0.0001"/> <!-- guess -->
-	<xacro:property name="toeMass" value="0.015"/>
-	<xacro:property name="upperLegLength" value="0.206"/>
-	<xacro:property name="upperLegWidth" value="0.022"/>
-	<xacro:property name="upperLegHeight" value="0.055"/>
-	<xacro:property name="lowerLegLength" value="0.206"/>
-	<xacro:property name="lowerLegRadius" value="0.013"/> <!--visual only-->
-	<xacro:property name="podLength" value="0.08"/>
-	<xacro:property name="podRadius" value="0.055"/>
-	<xacro:property name="dPodAxisToEdge" value="0.028"/> <!--center of pod cylinder to the ab axis-->
-	<xacro:property name="abOffs" value="0.10098"/>
-	<xacro:property name="dx" value="0.2263"/>
-	<xacro:property name="dy" value="0.07"/>
-	<xacro:property name="toeRadius" value="0.02"/>
-	<xacro:property name="toeOffset" value="0.0"/>
-	<xacro:property name="toeStiffness" value="30000.0"/>
-	<xacro:property name="toeDamping" value="1000.0"/>
-	<xacro:property name="toeSpinningFriction" value="0.3"/>
-	<xacro:property name="toeLateralFriction" value="3.0"/>
-	<xacro:property name="abKinLimit" value="0.707"/>
-	<xacro:property name="abSpeedLimit" value="30"/>
-	<xacro:property name="abEffortLimit" value="40"/>
-	<xacro:property name="jointSpeedLimit" value="30"/>
-	<xacro:property name="jointEffortLimit" value="40"/>
-	<!-- Define materials -->
-	<material name="darkgray">
-		<color rgba="0.1 0.1 0.1 1.0"/>
-	</material>
-	<material name="silver">
-		<color rgba="0.3 0.3 0.3 1.0"/>
-	</material>
-	<material name="red">
-		<color rgba="0.8 0.0 0.2 1.0"/>
-	</material>
-	<!-- Body -->
-	<link name="body">
-		<visual>
-			<origin rpy="0 0 0" xyz="0 0 0"/>
-			<geometry>
-				<box size="${bodyLength} ${bodyWidth} ${bodyHeight}"/>
-			</geometry>
-			<material name="darkgray"/>
-		</visual>
-		<inertial>
-			<mass value="${bodyMass}"/>
-			<!-- Uniform box -->
-			<!-- <inertia ixx="1/12*${bodyMass}*(${bodyWidth}*${bodyWidth} + ${bodyHeight}*${bodyHeight})"  ixy="0"  ixz="0" iyy="1/12*${bodyMass}*(${bodyLength}*${bodyLength} + ${bodyHeight}*${bodyHeight})" iyz="0" izz="1/12*${bodyMass}*(${bodyLength}*${bodyLength} + ${bodyWidth}*${bodyWidth})"/> -->
-			<inertia ixx="0.05"  ixy="0"  ixz="0" iyy="0.1" iyz="0" izz="0.1" />
-		</inertial>
-		<!-- Just copy geometry for collision -->
-		<collision>
-		<origin rpy="0 0 0" xyz="0 0 0"/>
-			<geometry>
-				<box size="${bodyLength} ${bodyWidth} ${bodyHeight}"/>
-			</geometry>
-		</collision>
-	</link>
-	<!-- Define our leg macro -->
-	<xacro:macro name="leg" params="suffix left front hipJointName kneeJointName abductionJointName hipJointLowerLimit hipJointUpperLimit color">
-		<!-- Hip motor -->
-		<link name="hip${suffix}">
-			<visual>
-				<origin rpy="${pi/2} 0 0" xyz="${front * 0} ${left * (dPodAxisToEdge)} 0"/>
-				<geometry>
-					<cylinder length="${podLength}" radius="${podRadius}"/>
-				</geometry>
-				<material name="${color}"/>
-			</visual>
-			<collision>
-				<origin rpy="${pi/2} 0 0" xyz="0 ${left * (dPodAxisToEdge)} 0"/>
-				<geometry>
-					<cylinder length="${podLength}" radius="${podRadius}"/>
-				</geometry>
-			</collision>
-			<inertial>
-				<mass value="${podMass}"/>
-				<!-- <inertia ixx="1/12*${podMass}*${podLength}*${podLength} + 1/4*${podMass}*${podRadius}*${podRadius}"  ixy="0"  ixz="0" iyy="1/12*${podMass}*${podLength}*${podLength} + 1/4*${podMass}*${podRadius}*${podRadius}" iyz="0" izz="1/2*${podMass}*${podRadius}*$
+<robot name="spirit" xmlns:xacro="http://www.ros.org/wiki/xacro">
+  <xacro:arg name="prefix" default=""/>
+  <xacro:property name="prefix" value="$(arg prefix)"/>
+  <!-- Define materials -->
+  <material name="gray">
+    <color rgba="0.2 0.2 0.2 1.0"/>
+  </material>
+  <material name="darkgray">
+    <color rgba="0.1 0.1 0.1 1.0"/>
+  </material>
+  <material name="silver">
+    <color rgba="0.3 0.3 0.3 1.0"/>
+  </material>
+  <material name="red">
+    <color rgba="0.8 0.0 0.2 1.0"/>
+  </material>
+  <material name="scots-rose">
+    <color rgba="0.937 0.2 0.251 1.0"/>
+  </material>
+  <!-- Body -->
+  <link name="${prefix}body">
+    <visual>
+      <origin rpy="0 0 0" xyz="0 0 0"/>
+      <geometry>
+        <box size="0.335 0.24 0.104"/>
+      </geometry>
+      <material name="darkgray"/>
+    </visual>
+    <inertial>
+      <mass value="7.388"/>
+      <!-- Uniform box -->
+      <!-- <inertia ixx="1/12*${bodyMass}*(${bodyWidth}*${bodyWidth} + ${bodyHeight}*${bodyHeight})"  ixy="0"  ixz="0" iyy="1/12*${bodyMass}*(${bodyLength}*${bodyLength} + ${bodyHeight}*${bodyHeight})" iyz="0" izz="1/12*${bodyMass}*(${bodyLength}*${bodyLength} + ${bodyWidth}*${bodyWidth})"/> -->
+      <inertia ixx="0.0642434782" ixy="0" ixz="0" iyy="0.1284869565" iyz="0" izz="0.1284869565"/>
+    </inertial>
+    <!-- Just copy geometry for collision -->
+    <collision>
+      <origin rpy="0 0 0" xyz="0 0 0"/>
+      <geometry>
+        <box size="0.335 0.24 0.104"/>
+      </geometry>
+    </collision>
+  </link>
+  <gazebo reference="${prefix}body">
+    <gravity>true</gravity>
+    <sensor name="imu_sensor" type="imu">
+      <always_on>true</always_on>
+      <visualize>true</visualize>
+      <topic>__default_topic_</topic>
+      <plugin filename="libgazebo_ros_imu_sensor.so" name="imu_plugin">
+        <topicName>imu</topicName>
+        <bodyName>${prefix}body</bodyName>
+        <updateRateHZ>500.0</updateRateHZ>
+        <gaussianNoise>0.0</gaussianNoise>
+        <xyzOffset>0 0 0</xyzOffset>
+        <rpyOffset>0 0 0</rpyOffset>
+        <frameName>${prefix}body</frameName>
+        <initialOrientationAsReference>true</initialOrientationAsReference>
+      </plugin>
+      <pose>0 0 0 0 0 0</pose>
+    </sensor>
+  </gazebo>
+  <!-- Hip motor -->
+  <link name="${prefix}hip0">
+    <visual>
+      <origin rpy="1.5707963268 0 0" xyz="0.0 0.028 0"/>
+      <geometry>
+        <cylinder length="0.08" radius="0.055"/>
+      </geometry>
+      <material name="darkgray"/>
+    </visual>
+    <collision>
+      <origin rpy="1.5707963268 0 0" xyz="0 0.028 0"/>
+      <geometry>
+        <cylinder length="0.08" radius="0.055"/>
+      </geometry>
+    </collision>
+    <inertial>
+      <mass value="0.575"/>
+      <!-- <inertia ixx="1/12*${podMass}*${podLength}*${podLength} + 1/4*${podMass}*${podRadius}*${podRadius}"  ixy="0"  ixz="0" iyy="1/12*${podMass}*${podLength}*${podLength} + 1/4*${podMass}*${podRadius}*${podRadius}" iyz="0" izz="1/2*${podMass}*${podRadius}*$
 				{podRadius}" /> -->
-				<inertia ixx="0.00066963541"  ixy="0"  ixz="0" iyy="0.00066963541" iyz="0" izz="0.0008696875" />
-			</inertial>
-		</link>
-		<!-- Abduction joint. Joint names are: 8 9 10 11 -->
-		<joint name="${abductionJointName}" type="revolute">
-			<parent link="body"/>
-			<child link="hip${suffix}"/>
-			<axis xyz="1 0 0"/>
-			<origin xyz="${front * dx} ${left * dy} 0"/>
-			<limit effort="${abEffortLimit}" velocity="${abSpeedLimit}" lower="${-abKinLimit}" upper="${abKinLimit}"/>
-			<dynamics damping="0.0" friction="0.0"/>
-		</joint>
-		<!-- Upper leg -->
-		<link name="upper${suffix}">
-			<visual>
-				<origin rpy="0 0 0" xyz="-${upperLegLength/2} ${-left*upperLegWidth} 0"/>
-				<geometry>
-					<box size="${upperLegLength} ${upperLegWidth} ${upperLegHeight}"/>
-				</geometry>
-				<material name="silver"/>
-			</visual>
-			<collision>
-				<origin rpy="0 0 0" xyz="-${upperLegLength/2} ${-left*upperLegWidth} 0"/>
-				<geometry>
-					<box size="${upperLegLength} ${upperLegWidth} ${upperLegHeight}"/>
-				</geometry>
-			</collision>
-			<inertial>
-				<mass value="${upperLegMass}"/>
-				<inertia ixx="${upperLegIxx}"  ixy="0" ixz="0" iyy="${upperLegIyy}" iyz="0" izz="${upperLegIzz}"/>
-			</inertial>
-		</link>
-		<!-- Hip joint. (Motor to upper leg). Joint names are: 0 2 4 6 -->
-		<joint name="${hipJointName}" type="revolute">
-			<parent link="hip${suffix}"/>
-			<child link="upper${suffix}"/>
-			<axis xyz="0 -1 0"/>
-			<origin xyz="${front * 0} ${left * abOffs} 0"/> <!--  rpy="0 -0.3 0" -->
-			<limit effort="${jointEffortLimit}" velocity="${jointSpeedLimit}" lower="${hipJointLowerLimit}" upper="${hipJointUpperLimit}"/>
-			<dynamics damping="0.0" friction="0.0"/>
-		</joint>
-		<!-- Lower leg -->
-		<link name="lower${suffix}">
-			<visual>
-				<origin rpy="0 ${pi/2} 0" xyz="${lowerLegLength/2} 0 0"/>
-				<geometry>
-					<cylinder length="${lowerLegLength}" radius="${lowerLegRadius}"/>
-				</geometry>
-				<material name="darkgray"/>
-			</visual>
-			<collision>
-				<origin rpy="0 ${pi/2} 0" xyz="${lowerLegLength/2} 0 0"/>
-				<geometry>
-					<cylinder length="${lowerLegLength}" radius="${lowerLegRadius}"/>
-				</geometry>
-			</collision>
-			<inertial>
-				<mass value="${lowerLegMass}"/>
-				<inertia ixx="${lowerLegIxx}"  ixy="0" ixz="0" iyy="${lowerLegIyy}" iyz="0" izz="${lowerLegIzz}"/>
-			</inertial>
-		</link>
-		<!-- Knee joint. Joint names are: 1 3 5 7 -->
-		<joint name="${kneeJointName}" type="revolute">
-			<parent link="upper${suffix}"/>
-			<child link="lower${suffix}"/>
-			<axis xyz="0 1 0"/>
-			<origin xyz="-${upperLegLength} 0 0"/> <!--rpy="0 0.5 0"-->
-			<limit effort="${jointEffortLimit}" velocity="${jointSpeedLimit}" lower="0" upper="${pi}"/>
-			<dynamics damping="0.0" friction="0.0"/>
-		</joint>
-		<!-- Toe -->
-		<link name="toe${suffix}">
-			<contact>
-				<friction_anchor/>
-				<stiffness value="${toeStiffness}"/>
-				<damping value="${toeDamping}"/>
-				<spinning_friction value="${toeSpinningFriction}"/>
-				<lateral_friction value="${toeLateralFriction}"/>
-			</contact>
-			<visual>
-				<origin rpy="0 0 0" xyz="0 0 0"/>
-				<geometry>
-					<sphere radius="${toeRadius}"/>
-				</geometry>
-				<material name="darkgray"/>
-			</visual>
-			<collision>
-				<origin rpy="0 0 0" xyz="0 0 0"/>
-				<geometry>
-					<sphere radius="${toeRadius}"/>
-				</geometry>
-			</collision>
-			<inertial>
-				<mass value="${toeMass}"/>
-				<inertia ixx="0.000025"  ixy="0"  ixz="0" iyy="0.000025" iyz="0" izz="0.000025" />
-				<!-- <inertia ixx="2/5*${toeMass}*${toeRadius}*${toeRadius}"  ixy="0"  ixz="0" iyy="2/5*${toeMass}*${toeRadius}*${toeRadius}" iyz="0" izz="2/5*${toeMass}*${toeRadius}*${toeRadius}" /> -->
-			</inertial>
-		</link>
-		<joint name="jtoe${suffix}" type="fixed">
-			<parent link="lower${suffix}"/>
-			<child link="toe${suffix}"/>
-			<origin xyz="${lowerLegLength} 0 -${toeOffset}"/>
-			<dynamics damping="0.0" friction="0.0"/>
-		</joint>
-	</xacro:macro>
-	<!-- Our four legs -->
-	<xacro:leg suffix="0" hipJointName="0" kneeJointName="1" abductionJointName="8" front="1" left="1" hipJointLowerLimit="${-2*pi}" hipJointUpperLimit="${2*pi}" color="darkgray"/>
- 	<xacro:leg suffix="1" hipJointName="2" kneeJointName="3" abductionJointName="9" front="-1" left="1" hipJointLowerLimit="${-2*pi}" hipJointUpperLimit="${2*pi}" color="darkgray"/>
- 	<xacro:leg suffix="2" hipJointName="4" kneeJointName="5" abductionJointName="10" front="1" left="-1" hipJointLowerLimit="${-2*pi}" hipJointUpperLimit="${2*pi}" color="red"/>
- 	<xacro:leg suffix="3" hipJointName="6" kneeJointName="7" abductionJointName="11" front="-1" left="-1" hipJointLowerLimit="${-2*pi}" hipJointUpperLimit="${2*pi}" color="darkgray"/>
+      <inertia ixx="0.00066963541" ixy="0" ixz="0" iyy="0.00066963541" iyz="0" izz="0.0008696875"/>
+    </inertial>
+  </link>
+  <gazebo reference="${prefix}hip0">
+    <material>Gazebo/Gray</material>
+  </gazebo>
+  <!-- Abduction joint. Joint names are: 8 9 10 11 -->
+  <joint name="8" type="revolute">
+    <parent link="${prefix}body"/>
+    <child link="${prefix}hip0"/>
+    <axis xyz="1 0 0"/>
+    <origin xyz="0.2263 0.07 0"/>
+    <limit effort="21" lower="-0.707" upper="0.707" velocity="37.7"/>
+    <dynamics damping="0.0" friction="0.0"/>
+  </joint>
+  <!-- Transmission elements required for Gazebo -->
+  <transmission name="${prefix}transmission_8">
+    <type>transmission_interface/SimpleTransmission</type>
+    <joint name="8">
+      <hardwareInterface>hardware_interface/EffortJointInterface</hardwareInterface>
+    </joint>
+    <actuator name="motor_8">
+      <hardwareInterface>EffortJointInterface</hardwareInterface>
+      <mechanicalReduction>1</mechanicalReduction>
+    </actuator>
+  </transmission>
+  <!-- Upper leg -->
+  <link name="${prefix}upper0">
+    <visual>
+      <origin rpy="0 0 0" xyz="-0.103 -0.022 0"/>
+      <geometry>
+        <box size="0.206 0.022 0.055"/>
+      </geometry>
+      <material name="silver"/>
+    </visual>
+    <collision>
+      <origin rpy="0 0 0" xyz="-0.103 -0.022 0"/>
+      <geometry>
+        <box size="0.206 0.022 0.055"/>
+      </geometry>
+    </collision>
+    <inertial>
+      <origin rpy="0 0 0" xyz="-0.040 -0.041 0"/>
+      <mass value="0.792"/>
+      <inertia ixx="5e-03" ixy="0" ixz="0" iyy="0.0070" iyz="0" izz="0.0070"/>
+    </inertial>
+  </link>
+  <gazebo reference="${prefix}upper0">
+    <material>Gazebo/Gray</material>
+  </gazebo>
+  <!-- Hip joint. (Motor to upper leg). Joint names are: 0 2 4 6 -->
+  <joint name="0" type="revolute">
+    <parent link="${prefix}hip0"/>
+    <child link="${prefix}upper0"/>
+    <axis xyz="0 -1 0"/>
+    <origin xyz="0 0.10098 0"/>
+    <!--  rpy="0 -0.3 0" -->
+    <limit effort="21" lower="-1.57" upper="3.14" velocity="37.7"/>
+    <dynamics damping="0.0" friction="0.0"/>
+  </joint>
+  <!-- Transmission elements required for Gazebo -->
+  <transmission name="${prefix}transmission_0">
+    <type>transmission_interface/SimpleTransmission</type>
+    <joint name="0">
+      <hardwareInterface>hardware_interface/EffortJointInterface</hardwareInterface>
+    </joint>
+    <actuator name="motor_0">
+      <hardwareInterface>EffortJointInterface</hardwareInterface>
+      <mechanicalReduction>1</mechanicalReduction>
+    </actuator>
+  </transmission>
+  <!-- Lower leg -->
+  <link name="${prefix}lower0">
+    <visual>
+      <origin rpy="0 1.5707963268 0" xyz="0.103 0 0"/>
+      <geometry>
+        <cylinder length="0.206" radius="0.013"/>
+      </geometry>
+      <material name="darkgray"/>
+    </visual>
+    <collision>
+      <origin rpy="0 1.5707963268 0" xyz="0.103 0 0"/>
+      <geometry>
+        <cylinder length="0.206" radius="0.013"/>
+      </geometry>
+    </collision>
+    <inertial>
+      <origin rpy="0 0 0" xyz="0.092 0 0"/>
+      <mass value="0.096"/>
+      <inertia ixx="1.3e-05" ixy="0" ixz="0" iyy="0.00047" iyz="0" izz="0.00047"/>
+    </inertial>
+  </link>
+  <gazebo reference="${prefix}lower0">
+    <material>Gazebo/Black</material>
+  </gazebo>
+  <!-- Knee joint. Joint names are: 1 3 5 7 -->
+  <joint name="1" type="revolute">
+    <parent link="${prefix}upper0"/>
+    <child link="${prefix}lower0"/>
+    <axis xyz="0 1 0"/>
+    <origin xyz="-0.206 0 0"/>
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
Commit message: Quad-SDK Update to Conform to ROS2 Control

File: quad_simulator/go2_description/models/go2/urdf/go2.urdf.xacro (robot description, xacro)
@@ -5,4 +5,10 @@
      For more information, please see http://wiki.ros.org/sw_urdf_exporter -->
 <robot name="go2" xmlns:xacro="http://www.ros.org/wiki/xacro">
+  <!-- Backend selection: use_sim=true -> gz_ros2_control (Gazebo, default);
+       use_sim=false -> quad_hardware/UnitreeSystem (real Go2 via DDS).
+       read_only (hardware only) -> true commands no torque (safe bring-up). -->
+  <xacro:arg name="use_sim" default="true" />
+  <xacro:arg name="read_only" default="true" />
+  <xacro:arg name="network_interface" default="eth0" />
   <link
     name="body">
@@ -1372,4 +1378,5 @@
     name="front_camera">
   </link>
+  <xacro:if value="$(arg use_sim)">
   <ros2_control name="GazeboSimSystem" type="system">
     <hardware>
@@ -1437,4 +1444,54 @@
     </joint>
   </ros2_control>
+  </xacro:if>
+  <xacro:unless value="$(arg use_sim)">
+  <!-- Real Go2 hardware via quad_hardware/UnitreeSystem. Five command
+       interfaces per joint drive the onboard motor PD; effort/pos/vel states
+       come from rt/lowstate. IMU is exposed as a sensor for
+       imu_sensor_broadcaster. -->
+  <xacro:macro name="unitree_hw_joint" params="jname">
+    <joint name="${jname}">
+      <command_interface name="position" />
+      <command_interface name="velocity" />
+      <command_interface name="kp" />
+      <command_interface name="kd" />
+      <command_interface name="effort" />
+      <state_interface name="position" />
+      <state_interface name="velocity" />
+      <state_interface name="effort" />
+    </joint>
+  </xacro:macro>
+  <ros2_control name="UnitreeSystem" type="system">
+    <hardware>
+      <plugin>quad_hardware/UnitreeSystem</plugin>
+      <param name="network_interface">$(arg network_interface)</param>
+      <param name="read_only">$(arg read_only)</param>
+    </hardware>
+    <xacro:unitree_hw_joint jname="0" />
+    <xacro:unitree_hw_joint jname="1" />
+    <xacro:unitree_hw_joint jname="2" />
+    <xacro:unitree_hw_joint jname="3" />
+    <xacro:unitree_hw_joint jname="4" />
+    <xacro:unitree_hw_joint jname="5" />
+    <xacro:unitree_hw_joint jname="6" />
+    <xacro:unitree_hw_joint jname="7" />
+    <xacro:unitree_hw_joint jname="8" />
+    <xacro:unitree_hw_joint jname="9" />
+    <xacro:unitree_hw_joint jname="10" />
+    <xacro:unitree_hw_joint jname="11" />
+    <sensor name="imu">
+      <state_interface name="orientation.x" />
+      <state_interface name="orientation.y" />
+      <state_interface name="orientation.z" />
+      <state_interface name="orientation.w" />
+      <state_interface name="angular_velocity.x" />
+      <state_interface name="angular_velocity.y" />
+      <state_interface name="angular_velocity.z" />
+      <state_interface name="linear_acceleration.x" />
+      <state_interface name="linear_acceleration.y" />
+      <state_interface name="linear_acceleration.z" />
+    </sensor>
+  </ros2_control>
+  </xacro:unless>
   <link name="cmu_text">
     <visual>

File: quad_simulator/spirit_description/models/spirit/urdf/spirit.urdf.xacro (robot description, xacro)
@@ -21,4 +21,9 @@
 <robot name="spirit" xmlns:xacro="http://www.ros.org/wiki/xacro">
   <xacro:arg name="prefix" default=""/>
+  <!-- Backend selection: use_sim=true -> gz_ros2_control (Gazebo, default);
+       use_sim=false -> quad_hardware/SpiritSystem (real Spirit 40 via MBLink).
+       read_only (hardware only) -> true commands no torque (safe bring-up). -->
+  <xacro:arg name="use_sim" default="true"/>
+  <xacro:arg name="read_only" default="true"/>
   <xacro:property name="prefix" value="$(arg prefix)"/>
   <!-- Define materials -->
@@ -972,4 +977,5 @@
     <origin xyz="-0.04 0 -0.005" rpy="0 0 3.14159"/>
   </joint>
+  <xacro:if value="$(arg use_sim)">
   <ros2_control name="GazeboSimSystem" type="system">
     <hardware>
@@ -1037,3 +1043,51 @@
     </joint>
   </ros2_control>
+  </xacro:if>
+  <xacro:unless value="$(arg use_sim)">
+  <!-- Real Spirit 40 hardware via quad_hardware/SpiritSystem (MBLink). Five
+       command interfaces per joint drive the onboard motor PD; effort is
+       derived from joint current. IMU is exposed for imu_sensor_broadcaster. -->
+  <xacro:macro name="spirit_hw_joint" params="jname">
+    <joint name="${jname}">
+      <command_interface name="position" />
+      <command_interface name="velocity" />
+      <command_interface name="kp" />
+      <command_interface name="kd" />
+      <command_interface name="effort" />
+      <state_interface name="position" />
+      <state_interface name="velocity" />
+      <state_interface name="effort" />
+    </joint>
+  </xacro:macro>
+  <ros2_control name="SpiritSystem" type="system">
+    <hardware>
+      <plugin>quad_hardware/SpiritSystem</plugin>
+      <param name="read_only">$(arg read_only)</param>
+    </hardware>
+    <xacro:spirit_hw_joint jname="0" />
+    <xacro:spirit_hw_joint jname="1" />
+    <xacro:spirit_hw_joint jname="2" />
+    <xacro:spirit_hw_joint jname="3" />
+    <xacro:spirit_hw_joint jname="4" />
+    <xacro:spirit_hw_joint jname="5" />
+    <xacro:spirit_hw_joint jname="6" />
+    <xacro:spirit_hw_joint jname="7" />
+    <xacro:spirit_hw_joint jname="8" />
+    <xacro:spirit_hw_joint jname="9" />
+    <xacro:spirit_hw_joint jname="10" />
+    <xacro:spirit_hw_joint jname="11" />
+    <sensor name="imu">
+      <state_interface name="orientation.x" />
+      <state_interface name="orientation.y" />
+      <state_interface name="orientation.z" />
+      <state_interface name="orientation.w" />
+      <state_interface name="angular_velocity.x" />
+      <state_interface name="angular_velocity.y" />
+      <state_interface name="angular_velocity.z" />
+      <state_interface name="linear_acceleration.x" />
+      <state_interface name="linear_acceleration.y" />
+      <state_interface name="linear_acceleration.z" />
+    </sensor>
+  </ros2_control>
+  </xacro:unless>
 </robot>
