Commit message: Networking refinements

File: quad_simulator/go2_description/models/go2/urdf/go2_isaac_clean.urdf (robot description, URDF)
Before this commit: robot go2, 43 links, 42 joints
Links:
- removed link cmu_text
Joints:
- removed joint cmu_text_joint

File: quad_simulator/go2w_description/models/go2w/urdf/go2w.urdf.xacro (robot description, xacro)
@@ -1462,20 +1462,3 @@
     </joint>
   </ros2_control>
-  <link name="cmu_text">
-    <visual>
-      <origin xyz="0 0 0" rpy="0 0 0" />
-      <geometry>
-        <mesh filename="package://objects_description/models/cmu_text/meshes/Spirit40_CMU_Text_transformed.stl" scale="1.3 1 1.3" />
-      </geometry>
-    </visual>
-    <inertial>
-      <mass value="0.0001" />
-      <inertia ixx="1e-08" ixy="0" ixz="0" iyy="1e-08" iyz="0" izz="1e-08" />
-    </inertial>
-  </link>
-  <joint name="cmu_text_joint" type="fixed">
-    <parent link="body" />
-    <child link="cmu_text" />
-    <origin xyz="0 0 -0.005" rpy="0 0 0" />
-  </joint>
 </robot>
