Commit message: vision60 working

File: quad_simulator/spot_description/models/spot/spot.sdf.xacro (robot description, xacro)
@@ -7,13 +7,13 @@
       <pose>0 0 0 0 -0 0</pose>
       <inertial>
-        <pose>0 0 -0.004962 0 -0 0</pose>
-        <mass>16.7077</mass>
-        <inertia>
-          <ixx>0.0815438</ixx>
+        <pose>0 0 -0.00496172 0 -0 0</pose>
+        <mass>16.70765207</mass>
+        <inertia>
+          <ixx>0.081543792</ixx>
           <ixy>0</ixy>
           <ixz>0</ixz>
-          <iyy>0.549231</iyy>
+          <iyy>0.549231154</iyy>
           <iyz>0</iyz>
-          <izz>0.569454</izz>
+          <izz>0.569454373</izz>
         </inertia>
       </inertial>
@@ -49,12 +49,12 @@
       <pose>0.29785 0.055 0 0 -0 0</pose>
       <inertial>
-        <pose>-0.015867 0.008558 9e-06 0 -0 0</pose>
-        <mass>1.13688</mass>
+        <pose>-0.01586739 0.00855842 0.00000903 0 -0 0</pose>
+        <mass>1.13688339</mass>
         <inertia>
           <ixx>0.00122166</ixx>
           <ixy>-0.00017754</ixy>
-          <ixz>4.3e-07</ixz>
+          <ixz>0.00000043</ixz>
           <iyy>0.00158957</iyy>
-          <iyz>-4.9e-07</iyz>
+          <iyz>-0.00000049</iyz>
           <izz>0.00172903</izz>
         </inertia>
@@ -89,6 +89,6 @@
             <lower>-0.7853981633974483</lower>
             <upper>0.7853981633974483</upper>
-            <effort>1000</effort>
-            <velocity>1000.00</velocity>
+            <effort>45</effort>
+            <velocity>100.00</velocity>
         </limit>
         <dynamics>
@@ -104,11 +104,11 @@
       <pose>0.29785 0.165945 0 0 -0 0</pose>
       <inertial>
-        <pose>0.002144 -0.011102 -0.078812 0 -0 0</pose>
-        <mass>2.2562</mass>
-        <inertia>
-          <ixx>0.026925</ixx>
-          <ixy>-8.782e-05</ixy>
+        <pose>0.00214442 -0.01110184 -0.07881204 0 -0 0</pose>
+        <mass>2.25620359</mass>
+        <inertia>
+          <ixx>0.02692501</ixx>
+          <ixy>-0.00008782</ixy>
           <ixz>0.00054873</ixz>
-          <iyy>0.0258391</iyy>
+          <iyy>0.02583907</iyy>
           <iyz>0.00207146</iyz>
           <izz>0.00318737</izz>
@@ -159,8 +159,8 @@
         <xyz>0 1 0</xyz>
         <limit>
-            <lower>-0.8988445647770796</lower>
-            <upper>2.2951079663725436</upper>
-            <effort>1000</effort>
-            <velocity>1000.00</velocity>
+            <lower>-0.89884456477707963539</lower>
+            <upper>2.2951079663725435509</upper>
+            <effort>45</effort>
+            <velocity>100.00</velocity>
         </limit>
         <dynamics>
@@ -176,13 +176,13 @@
       <pose>0.32285 0.165945 -0.3205 0 -0 0</pose>
       <inertial>
-        <pose>0.081455 0 -0.126678 0 -0 0</pose>
-        <mass>0.53</mass>
-        <inertia>
-          <ixx>0.00920778</ixx>
-          <ixy>0</ixy>
-          <ixz>-0.00310153</ixz>
-          <iyy>0.0142761</iyy>
-          <iyz>0</iyz>
-          <izz>0.00530824</izz>
+        <pose>0.00597360 0 -0.17466427 0 -0 0</pose>
+        <mass>0.330</mass>
+        <inertia>
+          <ixx>0.00701356</ixx>
+          <ixy>0.0</ixy>
+          <ixz>0.00006600</ixz>
+          <iyy>0.00709946</iyy>
+          <iyz>0.0</iyz>
+          <izz>0.00014529</izz>
         </inertia>
       </inertial>
@@ -248,6 +248,6 @@
             <lower>-2.7929</lower>
             <upper>-0.254402</upper>
-            <effort>1000</effort>
-            <velocity>1000.00</velocity>
+            <effort>115</effort>
+            <velocity>100.00</velocity>
         </limit>
         <dynamics>
@@ -263,12 +263,12 @@
       <pose>-0.29785 0.055 0 0 -0 0</pose>
       <inertial>
-        <pose>0.015867 0.008558 9e-06 0 -0 0</pose>
-        <mass>1.13688</mass>
+        <pose>0.01586739 0.00855842 0.00000903 0 -0 0</pose>
+        <mass>1.13688339</mass>
         <inertia>
           <ixx>0.00122166</ixx>
           <ixy>0.00017754</ixy>
-          <ixz>-4.3e-07</ixz>
+          <ixz>-0.00000043</ixz>
           <iyy>0.00158957</iyy>
-          <iyz>-4.9e-07</iyz>
+          <iyz>-0.00000049</iyz>
           <izz>0.00172903</izz>
         </inertia>
@@ -303,6 +303,6 @@
             <lower>-0.7853981633974483</lower>
             <upper>0.7853981633974483</upper>
-            <effort>1000</effort>
-            <velocity>1000.00</velocity>
+            <effort>45</effort>
+            <velocity>100.00</velocity>
         </limit>
         <dynamics>
@@ -318,11 +318,11 @@
       <pose>-0.29785 0.165945 0 0 -0 0</pose>
       <inertial>
-        <pose>0.002144 -0.011102 -0.078812 0 -0 0</pose>
-        <mass>2.2562</mass>
-        <inertia>
-          <ixx>0.026925</ixx>
-          <ixy>-8.782e-05</ixy>
+        <pose>0.00214442 -0.01110184 -0.07881204 0 -0 0</pose>
+        <mass>2.25620359</mass>
+        <inertia>
+          <ixx>0.02692501</ixx>
+          <ixy>-0.00008782</ixy>
           <ixz>0.00054873</ixz>
-          <iyy>0.0258391</iyy>
+          <iyy>0.02583907</iyy>
           <iyz>0.00207146</iyz>
           <izz>0.00318737</izz>
@@ -373,8 +373,8 @@
         <xyz>0 1 0</xyz>
         <limit>
-            <lower>-0.898845</lower>
-            <upper>2.24363</upper>
-            <effort>1000</effort>
-            <velocity>1000.00</velocity>
+            <lower>-0.89884456477707963539</lower>
+            <upper>2.2951079663725435509</upper>
+            <effort>45</effort>
+            <velocity>100.00</velocity>
         </limit>
         <dynamics>
@@ -390,13 +390,13 @@
       <pose>-0.27285 0.165945 -0.3205 0 -0 0</pose>
       <inertial>
-        <pose>0.081455 0 -0.126678 0 -0 0</pose>
-        <mass>0.53</mass>
-        <inertia>
-          <ixx>0.00920778</ixx>
-          <ixy>0</ixy>
-          <ixz>-0.00310153</ixz>
-          <iyy>0.0142761</iyy>
-          <iyz>0</iyz>
-          <izz>0.00530824</izz>
+        <pose>0.00597360 0 -0.17466427 0 -0 0</pose>
+        <mass>0.330</mass>
+        <inertia>
+          <ixx>0.00701356</ixx>
+          <ixy>0.0</ixy>
+          <ixz>0.00006600</ixz>
+          <iyy>0.00709946</iyy>
+          <iyz>0.0</iyz>
+          <izz>0.00014529</izz>
         </inertia>
       </inertial>
@@ -465,6 +465,6 @@
             <lower>-2.7929</lower>
             <upper>-0.255648</upper>
-            <effort>1000</effort>
-            <velocity>1000.00</velocity>
+            <effort>115</effort>
+            <velocity>100.00</velocity>
         </limit>
         <dynamics>
@@ -480,12 +480,12 @@
       <pose>0.29785 -0.055 0 0 -0 0</pose>
       <inertial>
-        <pose>-0.015867 -0.008558 9e-06 0 -0 0</pose>
-        <mass>1.13688</mass>
+        <pose>-0.01586739 -0.00855842 0.00000903 0 -0 0</pose>
+        <mass>1.13688339</mass>
         <inertia>
           <ixx>0.00122166</ixx>
           <ixy>0.00017754</ixy>
-          <ixz>4.3e-07</ixz>
+          <ixz>0.00000043</ixz>
           <iyy>0.00158957</iyy>
-          <iyz>4.9e-07</iyz>
+          <iyz>0.00000049</iyz>
           <izz>0.00172903</izz>
         </inertia>
@@ -520,6 +520,6 @@
             <lower>-0.7853981633974483</lower>
             <upper>0.7853981633974483</upper>
-            <effort>1000</effort>
-            <velocity>1000.00</velocity>
+            <effort>45</effort>
+            <velocity>100.00</velocity>
         </limit>
         <dynamics>
@@ -535,11 +535,11 @@
       <pose>0.29785 -0.165945 0 0 -0 0</pose>
       <inertial>
-        <pose>0.002144 0.011102 -0.078812 0 -0 0</pose>
-        <mass>2.2562</mass>
-        <inertia>
-          <ixx>0.026925</ixx>
-          <ixy>8.782e-05</ixy>
+        <pose>0.00214442 0.01110184 -0.07881204 0 -0 0</pose>
+        <mass>2.25620359</mass>
+        <inertia>
+          <ixx>0.02692501</ixx>
+          <ixy>0.00008782</ixy>
           <ixz>0.00054873</ixz>
-          <iyy>0.0258391</iyy>
+          <iyy>0.02583907</iyy>
           <iyz>-0.00207146</iyz>
           <izz>0.00318737</izz>
@@ -590,8 +590,8 @@
         <xyz>0 1 0</xyz>
         <limit>
-            <lower>-0.8988445647770796</lower>
-            <upper>2.2951079663725436</upper>
-            <effort>1000</effort>
-            <velocity>1000.00</velocity>
+            <lower>-0.89884456477707963539</lower>
+            <upper>2.2951079663725435509</upper>
+            <effort>45</effort>
+            <velocity>100.00</velocity>
         </limit>
         <dynamics>
@@ -607,13 +607,13 @@
       <pose>0.32285 -0.165945 -0.3205 0 -0 0</pose>
       <inertial>
-        <pose>0.081455 0 -0.126678 0 -0 0</pose>
-        <mass>0.53</mass>
-        <inertia>
-          <ixx>0.00920778</ixx>
-          <ixy>0</ixy>
-          <ixz>-0.00310153</ixz>
-          <iyy>0.0142761</iyy>
-          <iyz>0</iyz>
-          <izz>0.00530824</izz>
+        <pose>0.00597360 0 -0.17466427 0 -0 0</pose>
+        <mass>0.330</mass>
+        <inertia>
+          <ixx>0.00701356</ixx>
+          <ixy>0.0</ixy>
+          <ixz>0.00006600</ixz>
+          <iyy>0.00709946</iyy>
+          <iyz>0.0</iyz>
+          <izz>0.00014529</izz>
         </inertia>
       </inertial>
@@ -682,6 +682,6 @@
             <lower>-2.7929</lower>
             <upper>-0.247067</upper>
-            <effort>1000</effort>
-            <velocity>1000.00</velocity>
+            <effort>115</effort>
+            <velocity>100.00</velocity>
         </limit>
         <dynamics>
@@ -697,12 +697,12 @@
       <pose>-0.29785 -0.055 0 0 -0 0</pose>
       <inertial>
-        <pose>0.015867 -0.008558 9e-06 0 -0 0</pose>
-        <mass>1.13688</mass>
+        <pose>0.01586739 -0.00855842 0.00000903 0 -0 0</pose>
+        <mass>1.13688339</mass>
         <inertia>
           <ixx>0.00122166</ixx>
           <ixy>-0.00017754</ixy>
-          <ixz>-4.3e-07</ixz>
+          <ixz>-0.00000043</ixz>
           <iyy>0.00158957</iyy>
-          <iyz>4.9e-07</iyz>
+          <iyz>0.00000049</iyz>
           <izz>0.00172903</izz>
         </inertia>
@@ -737,6 +737,6 @@
             <lower>-0.7853981633974483</lower>
             <upper>0.7853981633974483</upper>
-            <effort>1000</effort>
-            <velocity>1000.00</velocity>
+            <effort>45</effort>
+            <velocity>100.00</velocity>
         </limit>
         <dynamics>
@@ -752,11 +752,11 @@
       <pose>-0.29785 -0.165945 0 0 -0 0</pose>
       <inertial>
-        <pose>0.002144 0.011102 -0.078812 0 -0 0</pose>
-        <mass>2.2562</mass>
-        <inertia>
-          <ixx>0.026925</ixx>
-          <ixy>8.782e-05</ixy>
+        <pose>0.00214442 0.01110184 -0.07881204 0 -0 0</pose>
+        <mass>2.25620359</mass>
+        <inertia>
+          <ixx>0.02692501</ixx>
+          <ixy>0.00008782</ixy>
           <ixz>0.00054873</ixz>
-          <iyy>0.0258391</iyy>
+          <iyy>0.02583907</iyy>
           <iyz>-0.00207146</iyz>
           <izz>0.00318737</izz>
@@ -807,8 +807,8 @@
         <xyz>0 1 0</xyz>
         <limit>
-            <lower>-0.8988445647770796</lower>
-            <upper>2.2951079663725436</upper>
-            <effort>1000</effort>
-            <velocity>1000.00</velocity>
+            <lower>-0.89884456477707963539</lower>
+            <upper>2.2951079663725435509</upper>
+            <effort>45</effort>
+            <velocity>100.00</velocity>
         </limit>
         <dynamics>
@@ -824,13 +824,13 @@
       <pose>-0.27285 -0.165945 -0.3205 0 -0 0</pose>
       <inertial>
-        <pose>0.081455 0 -0.126678 0 -0 0</pose>
-        <mass>0.53</mass>
-        <inertia>
-          <ixx>0.00920778</ixx>
-          <ixy>0</ixy>
-          <ixz>-0.00310153</ixz>
-          <iyy>0.0142761</iyy>
-          <iyz>0</iyz>
-          <izz>0.00530824</izz>
+        <pose>0.00597360 0 -0.17466427 0 -0 0</pose>
+        <mass>0.330</mass>
+        <inertia>
+          <ixx>0.00701356</ixx>
+          <ixy>0.0</ixy>
+          <ixz>0.00006600</ixz>
+          <iyy>0.00709946</iyy>
+          <iyz>0.0</iyz>
+          <izz>0.00014529</izz>
         </inertia>
       </inertial>
@@ -899,6 +899,6 @@
             <lower>-2.7929</lower>
             <upper>-0.248282</upper>
-            <effort>1000</effort>
-            <velocity>1000.00</velocity>
+            <effort>115</effort>
+            <velocity>100.00</velocity>
         </limit>
         <dynamics>

File: quad_simulator/spot_description/models/spot/urdf/spot.urdf.xacro (robot description, xacro)
@@ -88,5 +88,5 @@
     <origin xyz="0.29785 0.05500 0.00000" rpy="0 0 0"/>
     <axis xyz="1 0 0"/>
-    <limit effort="1000" velocity="1000.00" lower="-0.78539816339744827899" upper="0.78539816339744827899"/>
+    <limit effort="45" velocity="100.00" lower="-0.78539816339744827899" upper="0.78539816339744827899"/>
     <dynamics damping="0" friction="0"/>
   </joint>
@@ -129,5 +129,5 @@
     <origin xyz="0.0 0.110945 0.0" rpy="0 0 0"/>
     <axis xyz="0 1 0"/>
-    <limit effort="1000" velocity="1000.00" lower="-0.89884456477707963539" upper="2.2951079663725435509"/>
+    <limit effort="45" velocity="100.00" lower="-0.89884456477707963539" upper="2.2951079663725435509"/>
     <dynamics damping="0" friction="0"/>
   </joint>
@@ -176,5 +176,5 @@
     <origin xyz="0.025 0.000 -0.3205" rpy="0 0 0"/>
     <axis xyz="0 1 0"/>
-    <limit effort="1000" velocity="1000.00" lower="-2.7929" upper="-0.254402"/>
+    <limit effort="115" velocity="100.00" lower="-2.7929" upper="-0.254402"/>
     <dynamics damping="0" friction="0"/>
   </joint>
@@ -257,5 +257,5 @@
     <origin xyz="-0.29785 0.05500 0.00000" rpy="0 0 0"/>
     <axis xyz="1 0 0"/>
-    <limit effort="1000" velocity="1000.00" lower="-0.78539816339744827899" upper="0.78539816339744827899"/>
+    <limit effort="45" velocity="100.00" lower="-0.78539816339744827899" upper="0.78539816339744827899"/>
     <dynamics damping="0" friction="0"/>
   </joint>
@@ -298,5 +298,5 @@
     <origin xyz="0.0 0.110945 0.0" rpy="0 0 0"/>
     <axis xyz="0 1 0"/>
-    <limit effort="1000" velocity="1000.00" lower="-0.898845" upper="2.24363"/>
+    <limit effort="45" velocity="100.00" lower="-0.898845" upper="2.24363"/>
     <dynamics damping="0" friction="0"/>
   </joint>
@@ -345,5 +345,5 @@
     <origin xyz="0.025 0.000 -0.3205" rpy="0 0 0"/>
     <axis xyz="0 1 0"/>
-    <limit effort="1000" velocity="1000.00" lower="-2.7929" upper="-0.255648"/>
+    <limit effort="115" velocity="100.00" lower="-2.7929" upper="-0.255648"/>
     <dynamics damping="0" friction="0"/>
   </joint>
@@ -426,5 +426,5 @@
     <origin xyz="0.29785 -0.05500 0.00000" rpy="0 0 0"/>
     <axis xyz="1 0 0"/>
-    <limit effort="1000" velocity="1000.00" lower="-0.78539816339744827899" upper="0.78539816339744827899"/>
+    <limit effort="45" velocity="100.00" lower="-0.78539816339744827899" upper="0.78539816339744827899"/>
     <dynamics damping="0" friction="0"/>
   </joint>
@@ -467,5 +467,5 @@
     <origin xyz="0.0 -0.110945 0.0" rpy="0 0 0"/>
     <axis xyz="0 1 0"/>
-    <limit effort="1000" velocity="1000.00" lower="-0.89884456477707963539" upper="2.2951079663725435509"/>
+    <limit effort="45" velocity="100.00" lower="-0.89884456477707963539" upper="2.2951079663725435509"/>
     <dynamics damping="0" friction="0"/>
   </joint>
@@ -514,5 +514,5 @@
     <origin xyz="0.025 0.000 -0.3205" rpy="0 0 0"/>
     <axis xyz="0 1 0"/>
-    <limit effort="1000" velocity="1000.00" lower="-2.7929" upper="-0.247067"/>
+    <limit effort="115" velocity="100.00" lower="-2.7929" upper="-0.247067"/>
     <dynamics damping="0" friction="0"/>
   </joint>
@@ -595,5 +595,5 @@
     <origin xyz="-0.29785 -0.05500 0.00000" rpy="0 0 0"/>
     <axis xyz="1 0 0"/>
-    <limit effort="1000" velocity="1000.00" lower="-0.78539816339744827899" upper="0.78539816339744827899"/>
+    <limit effort="45" velocity="100.00" lower="-0.78539816339744827899" upper="0.78539816339744827899"/>
     <dynamics damping="0" friction="0"/>
   </joint>
@@ -636,5 +636,5 @@
     <origin xyz="0.0 -0.110945 0.0" rpy="0 0 0"/>
     <axis xyz="0 1 0"/>
-    <limit effort="1000" velocity="1000.00" lower="-0.89884456477707963539" upper="2.2951079663725435509"/>
+    <limit effort="45" velocity="100.00" lower="-0.89884456477707963539" upper="2.2951079663725435509"/>
     <dynamics damping="0" friction="0"/>
   </joint>
@@ -683,5 +683,5 @@
     <origin xyz="0.025 0.000 -0.3205" rpy="0 0 0"/>
     <axis xyz="0 1 0"/>
-    <limit effort="1000" velocity="1000.00" lower="-2.7929" upper="-0.248282"/>
+    <limit effort="115" velocity="100.00" lower="-2.7929" upper="-0.248282"/>
     <dynamics damping="0" friction="0"/>
   </joint>
