Commit message: testing different spot urdf, stil not working

File: quad_simulator/spot_description/models/spot/spot.sdf.xacro (robot description, xacro)
@@ -7,13 +7,13 @@
       <pose>0 0 0 0 -0 0</pose>
       <inertial>
-        <pose>0 0 -0.00496172 0 -0 0</pose>
-        <mass>16.70765207</mass>
-        <inertia>
-          <ixx>0.081543792</ixx>
-          <ixy>0</ixy>
-          <ixz>0</ixz>
-          <iyy>0.549231154</iyy>
-          <iyz>0</iyz>
-          <izz>0.569454373</izz>
+        <pose>0.006394396536052227 -9.812158532440662e-05 0.0009113792330026627 0 -0 0</pose>
+        <mass>32.86</mass>
+        <inertia>
+          <ixx>0.13143999874591827</ixx>
+          <ixy>0</ixy>
+          <ixz>0</ixz>
+          <iyy>0.13143999874591827</iyy>
+          <iyz>0</iyz>
+          <izz>0.13143999874591827</izz>
         </inertia>
       </inertial>
@@ -49,13 +49,13 @@
       <pose>0.29785 0.055 0 0 -0 0</pose>
       <inertial>
-        <pose>-0.01586739 0.00855842 0.00000903 0 -0 0</pose>
-        <mass>1.13688339</mass>
-        <inertia>
-          <ixx>0.00122166</ixx>
-          <ixy>-0.00017754</ixy>
-          <ixz>0.00000043</ixz>
-          <iyy>0.00158957</iyy>
-          <iyz>-0.00000049</iyz>
-          <izz>0.00172903</izz>
+        <pose>-0.005374345928430557 0.012841847725212574 9.875232353806496e-05 0 -0 0</pose>
+        <mass>1.68</mass>
+        <inertia>
+          <ixx>0.0021147398873455382</ixx>
+          <ixy>0</ixy>
+          <ixz>0</ixz>
+          <iyy>0.0018129577956607131</iyy>
+          <iyz>0</iyz>
+          <izz>0.002265435737304666</izz>
         </inertia>
       </inertial>
@@ -104,13 +104,13 @@
       <pose>0.29785 0.165945 0 0 -0 0</pose>
       <inertial>
-        <pose>0.00214442 -0.01110184 -0.07881204 0 -0 0</pose>
-        <mass>2.25620359</mass>
-        <inertia>
-          <ixx>0.02692501</ixx>
-          <ixy>-0.00008782</ixy>
-          <ixz>0.00054873</ixz>
-          <iyy>0.02583907</iyy>
-          <iyz>0.00207146</iyz>
-          <izz>0.00318737</izz>
+        <pose>0.005142373498529196 -0.0024323679972440004 -0.12100915610790253 0 -0 0</pose>
+        <mass>2.34</mass>
+        <inertia>
+          <ixx>0.02755964961185679</ixx>
+          <ixy>0</ixy>
+          <ixz>0</ixz>
+          <iyy>0.027354914287651046</iyy>
+          <iyz>0</iyz>
+          <izz>0.002848145546743553</izz>
         </inertia>
       </inertial>
@@ -176,13 +176,13 @@
       <pose>0.32285 0.165945 -0.3205 0 -0 0</pose>
       <inertial>
-        <pose>0.00597360 0 -0.17466427 0 -0 0</pose>
-        <mass>0.330</mass>
-        <inertia>
-          <ixx>0.00701356</ixx>
-          <ixy>0.0</ixy>
-          <ixz>0.00006600</ixz>
-          <iyy>0.00709946</iyy>
-          <iyz>0.0</iyz>
-          <izz>0.00014529</izz>
+        <pose>0.00225794012658298 4.607596201822162e-05 -0.1800822913646698 0 -0 0</pose>
+        <mass>0.35</mass>
+        <inertia>
+          <ixx>0.003999022654901177</ixx>
+          <ixy>0</ixy>
+          <ixz>0</ixz>
+          <iyy>0.0040503157598010785</iyy>
+          <iyz>0</iyz>
+          <izz>0.0001493402097647426</izz>
         </inertia>
       </inertial>
@@ -263,13 +263,13 @@
       <pose>-0.29785 0.055 0 0 -0 0</pose>
       <inertial>
-        <pose>0.01586739 0.00855842 0.00000903 0 -0 0</pose>
-        <mass>1.13688339</mass>
-        <inertia>
-          <ixx>0.00122166</ixx>
-          <ixy>0.00017754</ixy>
-          <ixz>-0.00000043</ixz>
-          <iyy>0.00158957</iyy>
-          <iyz>-0.00000049</iyz>
-          <izz>0.00172903</izz>
+        <pose>0.005374345928430557 0.012841847725212574 -9.875232353806496e-05 0 -0 0</pose>
+        <mass>1.68</mass>
+        <inertia>
+          <ixx>0.0021147398873455382</ixx>
+          <ixy>0</ixy>
+          <ixz>0</ixz>
+          <iyy>0.0018129577956607131</iyy>
+          <iyz>0</iyz>
+          <izz>0.002265435737304666</izz>
         </inertia>
       </inertial>
@@ -318,13 +318,13 @@
       <pose>-0.29785 0.165945 0 0 -0 0</pose>
       <inertial>
-        <pose>0.00214442 -0.01110184 -0.07881204 0 -0 0</pose>
-        <mass>2.25620359</mass>
-        <inertia>
-          <ixx>0.02692501</ixx>
-          <ixy>-0.00008782</ixy>
-          <ixz>0.00054873</ixz>
-          <iyy>0.02583907</iyy>
-          <iyz>0.00207146</iyz>
-          <izz>0.00318737</izz>
+        <pose>0.005142373498529196 -0.0024323679972440004 -0.12100915610790253 0 -0 0</pose>
+        <mass>2.34</mass>
+        <inertia>
+          <ixx>0.02755964961185679</ixx>
+          <ixy>0</ixy>
+          <ixz>0</ixz>
+          <iyy>0.027354914287651046</iyy>
+          <iyz>0</iyz>
+          <izz>0.002848145546743553</izz>
         </inertia>
       </inertial>
@@ -390,13 +390,13 @@
       <pose>-0.27285 0.165945 -0.3205 0 -0 0</pose>
       <inertial>
-        <pose>0.00597360 0 -0.17466427 0 -0 0</pose>
-        <mass>0.330</mass>
-        <inertia>
-          <ixx>0.00701356</ixx>
-          <ixy>0.0</ixy>
-          <ixz>0.00006600</ixz>
-          <iyy>0.00709946</iyy>
-          <iyz>0.0</iyz>
-          <izz>0.00014529</izz>
+        <pose>0.00225794012658298 4.607596201822162e-05 -0.1800822913646698 0 -0 0</pose>
+        <mass>0.35</mass>
+        <inertia>
+          <ixx>0.003999022654901177</ixx>
+          <ixy>0</ixy>
+          <ixz>0</ixz>
+          <iyy>0.0040503157598010785</iyy>
+          <iyz>0</iyz>
+          <izz>0.0001493402097647426</izz>
         </inertia>
       </inertial>
@@ -464,5 +464,5 @@
         <limit>
             <lower>-2.7929</lower>
-            <upper>-0.255648</upper>
+            <upper>-0.247067</upper>
             <effort>115</effort>
             <velocity>100.00</velocity>
@@ -480,13 +480,13 @@
       <pose>0.29785 -0.055 0 0 -0 0</pose>
       <inertial>
-        <pose>-0.01586739 -0.00855842 0.00000903 0 -0 0</pose>
-        <mass>1.13688339</mass>
-        <inertia>
-          <ixx>0.00122166</ixx>
-          <ixy>0.00017754</ixy>
-          <ixz>0.00000043</ixz>
-          <iyy>0.00158957</iyy>
-          <iyz>0.00000049</iyz>
-          <izz>0.00172903</izz>
+        <pose>-0.005374345928430557 -0.012841847725212574 -9.875232353806496e-05 0 -0 0</pose>
+        <mass>1.68</mass>
+        <inertia>
+          <ixx>0.0021147398873455382</ixx>
+          <ixy>0</ixy>
+          <ixz>0</ixz>
+          <iyy>0.0018129577956607131</iyy>
+          <iyz>0</iyz>
+          <izz>0.002265435737304666</izz>
         </inertia>
       </inertial>
@@ -535,13 +535,13 @@
       <pose>0.29785 -0.165945 0 0 -0 0</pose>
       <inertial>
-        <pose>0.00214442 0.01110184 -0.07881204 0 -0 0</pose>
-        <mass>2.25620359</mass>
-        <inertia>
-          <ixx>0.02692501</ixx>
-          <ixy>0.00008782</ixy>
-          <ixz>0.00054873</ixz>
-          <iyy>0.02583907</iyy>
-          <iyz>-0.00207146</iyz>
-          <izz>0.00318737</izz>
+        <pose>0.005142373498529196 0.0024323677644133568 -0.12100915610790253 0 -0 0</pose>
+        <mass>2.34</mass>
+        <inertia>
+          <ixx>0.02755964678927691</ixx>
+          <ixy>0</ixy>
+          <ixz>0</ixz>
+          <iyy>0.02735491706466737</iyy>
+          <iyz>0</iyz>
+          <izz>0.0028481453594764797</izz>
         </inertia>
       </inertial>
@@ -607,13 +607,13 @@
       <pose>0.32285 -0.165945 -0.3205 0 -0 0</pose>
       <inertial>
-        <pose>0.00597360 0 -0.17466427 0 -0 0</pose>
-        <mass>0.330</mass>
-        <inertia>
-          <ixx>0.00701356</ixx>
-          <ixy>0.0</ixy>
-          <ixz>0.00006600</ixz>
-          <iyy>0.00709946</iyy>
-          <iyz>0.0</iyz>
-          <izz>0.00014529</izz>
+        <pose>0.00225794012658298 4.607596201822162e-05 -0.1800822913646698 0 -0 0</pose>
+        <mass>0.35</mass>
+        <inertia>
+          <ixx>0.003999022654901177</ixx>
+          <ixy>0</ixy>
+          <ixz>0</ixz>
+          <iyy>0.0040503157598010785</iyy>
+          <iyz>0</iyz>
+          <izz>0.0001493402097647426</izz>
         </inertia>
       </inertial>
@@ -681,5 +681,5 @@
         <limit>
             <lower>-2.7929</lower>
-            <upper>-0.247067</upper>
+            <upper>-0.255648</upper>
             <effort>115</effort>
             <velocity>100.00</velocity>
@@ -697,13 +697,13 @@
       <pose>-0.29785 -0.055 0 0 -0 0</pose>
       <inertial>
-        <pose>0.01586739 -0.00855842 0.00000903 0 -0 0</pose>
-        <mass>1.13688339</mass>
-        <inertia>
-          <ixx>0.00122166</ixx>
-          <ixy>-0.00017754</ixy>
-          <ixz>-0.00000043</ixz>
-          <iyy>0.00158957</iyy>
-          <iyz>0.00000049</iyz>
-          <izz>0.00172903</izz>
+        <pose>0.005374345928430557 -0.012841847725212574 9.875232353806496e-05 0 -0 0</pose>
+        <mass>1.68</mass>
+        <inertia>
+          <ixx>0.0021147398873455382</ixx>
+          <ixy>0</ixy>
+          <ixz>0</ixz>
+          <iyy>0.0018129577956607131</iyy>
+          <iyz>0</iyz>
+          <izz>0.002265435737304666</izz>
         </inertia>
       </inertial>
@@ -752,13 +752,13 @@
       <pose>-0.29785 -0.165945 0 0 -0 0</pose>
       <inertial>
-        <pose>0.00214442 0.01110184 -0.07881204 0 -0 0</pose>
-        <mass>2.25620359</mass>
-        <inertia>
-          <ixx>0.02692501</ixx>
-          <ixy>0.00008782</ixy>
-          <ixz>0.00054873</ixz>
-          <iyy>0.02583907</iyy>
-          <iyz>-0.00207146</iyz>
-          <izz>0.00318737</izz>
+        <pose>0.005142373498529196 0.0024323677644133568 -0.12100915610790253 0 -0 0</pose>
+        <mass>2.34</mass>
+        <inertia>
+          <ixx>0.02755964678927691</ixx>
+          <ixy>0</ixy>
+          <ixz>0</ixz>
+          <iyy>0.02735491706466737</iyy>
+          <iyz>0</iyz>
+          <izz>0.0028481453594764797</izz>
         </inertia>
       </inertial>
@@ -824,13 +824,13 @@
       <pose>-0.27285 -0.165945 -0.3205 0 -0 0</pose>
       <inertial>
-        <pose>0.00597360 0 -0.17466427 0 -0 0</pose>
-        <mass>0.330</mass>
-        <inertia>
-          <ixx>0.00701356</ixx>
-          <ixy>0.0</ixy>
-          <ixz>0.00006600</ixz>
-          <iyy>0.00709946</iyy>
-          <iyz>0.0</iyz>
-          <izz>0.00014529</izz>
+        <pose>0.00225794012658298 4.607596201822162e-05 -0.1800822913646698 0 -0 0</pose>
+        <mass>0.35</mass>
+        <inertia>
+          <ixx>0.003999022654901177</ixx>
+          <ixy>0</ixy>
+          <ixz>0</ixz>
+          <iyy>0.0040503157598010785</iyy>
+          <iyz>0</iyz>
+          <izz>0.0001493402097647426</izz>
         </inertia>
       </inertial>

File: quad_simulator/spot_description/models/spot/urdf/spot.urdf.xacro (robot description, xacro)
@@ -41,7 +41,7 @@
     </collision>
     <inertial>
-      <origin xyz="0 0 -0.00496172"/>
-      <mass value="16.70765207"/>
-      <inertia ixx="0.081543792" ixy="0.0" ixz="0.0" iyy="0.549231154" iyz="0.0" izz="0.569454373"/>
+      <origin xyz="0.006394396536052227 -9.812158532440662e-05 0.0009113792330026627"/>
+      <mass value="32.86"/>
+      <inertia ixx="0.13143999874591827" ixy="0.0" ixz="0.0" iyy="0.13143999874591827" iyz="0.0" izz="0.13143999874591827"/>
     </inertial>
   </link>
@@ -74,7 +74,7 @@
     </visual>
     <inertial>
-      <origin xyz="-0.01586739 0.00855842 0.00000903"/>
-      <inertia ixx="0.00122166" ixy="-0.00017754" ixz="0.00000043" iyy="0.00158957" iyz="-0.00000049" izz="0.00172903"/>
-      <mass value="1.13688339"/>
+      <origin xyz="-0.005374345928430557 0.012841847725212574 9.875232353806496e-05"/>
+      <inertia ixx="0.0021147398873455382" ixy="0.0" ixz="0.0" iyy="0.0018129577956607131" iyz="0.0" izz="0.002265435737304666"/>
+      <mass value="1.68"/>
     </inertial>
   </link>
@@ -115,7 +115,7 @@
     </collision>
     <inertial>
-      <origin xyz="0.00214442 -0.01110184 -0.07881204"/>
-      <inertia ixx="0.02692501" ixy="-0.00008782" ixz="0.00054873" iyy="0.02583907" iyz="0.00207146" izz="0.00318737"/>
-      <mass value="2.25620359"/>
+      <origin xyz="0.005142373498529196 -0.0024323679972440004 -0.12100915610790253"/>
+      <inertia ixx="0.02755964961185679" ixy="0.0" ixz="0.0" iyy="0.027354914287651046" iyz="0.0" izz="0.002848145546743553"/>
+      <mass value="2.34"/>
     </inertial>
   </link>
@@ -127,5 +127,5 @@
     <parent link="hip0"/>
     <child link="upper0"/>
-    <origin xyz="0.0 0.110945 0.0" rpy="0 0 0"/>
+    <origin xyz="0.0 0.11080 0.0" rpy="0 0 0"/>
     <axis xyz="0 1 0"/>
     <limit effort="45" velocity="100.00" lower="-0.89884456477707963539" upper="2.2951079663725435509"/>
@@ -162,7 +162,7 @@
     </collision> -->
     <inertial>
-      <origin xyz="0.00597360 0.0 -0.17466427"/>
-      <inertia ixx="0.00701356" ixy="0.0" ixz="0.00006600" iyy="0.00709946" iyz="0.0" izz="0.00014529"/>
-      <mass value="0.330"/>
+      <origin xyz="0.00225794012658298 4.607596201822162e-05 -0.1800822913646698"/>
+      <inertia ixx="0.003999022654901177" ixy="0.0" ixz="0.0" iyy="0.0040503157598010785" iyz="0.0" izz="0.0001493402097647426"/>
+      <mass value="0.35"/>
     </inertial>
   </link>
@@ -174,5 +174,5 @@
     <parent link="upper0"/>
     <child link="lower0"/>
-    <origin xyz="0.025 0.000 -0.3205" rpy="0 0 0"/>
+    <origin xyz="0.025 0.000 -0.3200" rpy="0 0 0"/>
     <axis xyz="0 1 0"/>
     <limit effort="115" velocity="100.00" lower="-2.7929" upper="-0.254402"/>
@@ -243,7 +243,7 @@
     </visual>
     <inertial>
-      <origin xyz="0.01586739 0.00855842 0.00000903"/>
-      <inertia ixx="0.00122166" ixy="0.00017754" ixz="-0.00000043" iyy="0.00158957" iyz="-0.00000049" izz="0.00172903"/>
-      <mass value="1.13688339"/>
+      <origin xyz="0.005374345928430557 0.012841847725212574 -9.875232353806496e-05"/>
+      <inertia ixx="0.0021147398873455382" ixy="0.0" ixz="0.0" iyy="0.0018129577956607131" iyz="0.0" izz="0.002265435737304666"/>
+      <mass value="1.68"/>
     </inertial>
   </link>
@@ -284,7 +284,7 @@
     </collision>
     <inertial>
-      <origin xyz="0.00214442 -0.01110184 -0.07881204"/>
-      <inertia ixx="0.02692501" ixy="-0.00008782" ixz="0.00054873" iyy="0.02583907" iyz="0.00207146" izz="0.00318737"/>
-      <mass value="2.25620359"/>
+      <origin xyz="0.005142373498529196 -0.0024323679972440004 -0.12100915610790253"/>
+      <inertia ixx="0.02755964961185679" ixy="0.0" ixz="0.0" iyy="0.027354914287651046" iyz="0.0" izz="0.002848145546743553"/>
+      <mass value="2.34"/>
     </inertial>
   </link>
@@ -296,7 +296,7 @@
     <parent link="hip1"/>
     <child link="upper1"/>
-    <origin xyz="0.0 0.110945 0.0" rpy="0 0 0"/>
+    <origin xyz="0.0 0.11080 0.0" rpy="0 0 0"/>
     <axis xyz="0 1 0"/>
-    <limit effort="45" velocity="100.00" lower="-0.898845" upper="2.24363"/>
+    <limit effort="45" velocity="100.00" lower="-0.89884456477707963539" upper="2.2951079663725435509"/>
     <dynamics damping="0" friction="0"/>
   </joint>
@@ -331,7 +331,7 @@
     </collision> -->
     <inertial>
-      <origin xyz="0.00597360 0.0 -0.17466427"/>
-      <inertia ixx="0.00701356" ixy="0.0" ixz="0.00006600" iyy="0.00709946" iyz="0.0" izz="0.00014529"/>
-      <mass value="0.330"/>
+      <origin xyz="0.00225794012658298 4.607596201822162e-05 -0.1800822913646698"/>
+      <inertia ixx="0.003999022654901177" ixy="0.0" ixz="0.0" iyy="0.0040503157598010785" iyz="0.0" izz="0.0001493402097647426"/>
+      <mass value="0.35"/>
     </inertial>
   </link>
@@ -343,7 +343,7 @@
     <parent link="upper1"/>
     <child link="lower1"/>
-    <origin xyz="0.025 0.000 -0.3205" rpy="0 0 0"/>
+    <origin xyz="0.025 0.000 -0.3200" rpy="0 0 0"/>
     <axis xyz="0 1 0"/>
-    <limit effort="115" velocity="100.00" lower="-2.7929" upper="-0.255648"/>
+    <limit effort="115" velocity="100.00" lower="-2.7929" upper="-0.247067"/>
     <dynamics damping="0" friction="0"/>
   </joint>
@@ -412,7 +412,7 @@
     </visual>
     <inertial>
-      <origin xyz="-0.01586739 -0.00855842 0.00000903"/>
-      <inertia ixx="0.00122166" ixy="0.00017754" ixz="0.00000043" iyy="0.00158957" iyz="0.00000049" izz="0.00172903"/>
-      <mass value="1.13688339"/>
+      <origin xyz="-0.005374345928430557 -0.012841847725212574 -9.875232353806496e-05"/>
+      <inertia ixx="0.0021147398873455382" ixy="0.0" ixz="0.0" iyy="0.0018129577956607131" iyz="0.0" izz="0.002265435737304666"/>
+      <mass value="1.68"/>
     </inertial>
   </link>
@@ -453,7 +453,7 @@
     </collision>
     <inertial>
-      <origin xyz="0.00214442 0.01110184 -0.07881204"/>
-      <inertia ixx="0.02692501" ixy="0.00008782" ixz="0.00054873" iyy="0.02583907" iyz="-0.00207146" izz="0.00318737"/>
-      <mass value="2.25620359"/>
+      <origin xyz="0.005142373498529196 0.0024323677644133568 -0.12100915610790253"/>
+      <inertia ixx="0.02755964678927691" ixy="0.0" ixz="0.0" iyy="0.02735491706466737" iyz="0.0" izz="0.0028481453594764797"/>
+      <mass value="2.34"/>
     </inertial>
   </link>
@@ -465,5 +465,5 @@
     <parent link="hip2"/>
     <child link="upper2"/>
-    <origin xyz="0.0 -0.110945 0.0" rpy="0 0 0"/>
+    <origin xyz="0.0 -0.11080 0.0" rpy="0 0 0"/>
     <axis xyz="0 1 0"/>
     <limit effort="45" velocity="100.00" lower="-0.89884456477707963539" upper="2.2951079663725435509"/>
@@ -500,7 +500,7 @@
     </collision> -->
     <inertial>
-      <origin xyz="0.00597360 0.0 -0.17466427"/>
-      <inertia ixx="0.00701356" ixy="0.0" ixz="0.00006600" iyy="0.00709946" iyz="0.0" izz="0.00014529"/>
-      <mass value="0.330"/>
+      <origin xyz="0.00225794012658298 4.607596201822162e-05 -0.1800822913646698"/>
+      <inertia ixx="0.003999022654901177" ixy="0.0" ixz="0.0" iyy="0.0040503157598010785" iyz="0.0" izz="0.0001493402097647426"/>
+      <mass value="0.35"/>
     </inertial>
   </link>
@@ -512,7 +512,7 @@
     <parent link="upper2"/>
     <child link="lower2"/>
-    <origin xyz="0.025 0.000 -0.3205" rpy="0 0 0"/>
+    <origin xyz="0.025 0.000 -0.3200" rpy="0 0 0"/>
     <axis xyz="0 1 0"/>
-    <limit effort="115" velocity="100.00" lower="-2.7929" upper="-0.247067"/>
+    <limit effort="115" velocity="100.00" lower="-2.7929" upper="-0.255648"/>
     <dynamics damping="0" friction="0"/>
   </joint>
@@ -581,7 +581,7 @@
     </visual>
     <inertial>
-      <origin xyz="0.01586739 -0.00855842 0.00000903"/>
-      <inertia ixx="0.00122166" ixy="-0.00017754" ixz="-0.00000043" iyy="0.00158957" iyz="0.00000049" izz="0.00172903"/>
-      <mass value="1.13688339"/>
+      <origin xyz="0.005374345928430557 -0.012841847725212574 9.875232353806496e-05"/>
+      <inertia ixx="0.0021147398873455382" ixy="0.0" ixz="0.0" iyy="0.0018129577956607131" iyz="0.0" izz="0.002265435737304666"/>
+      <mass value="1.68"/>
     </inertial>
   </link>
@@ -622,7 +622,7 @@
     </collision>
     <inertial>
-      <origin xyz="0.00214442 0.01110184 -0.07881204"/>
-      <inertia ixx="0.02692501" ixy="0.00008782" ixz="0.00054873" iyy="0.02583907" iyz="-0.00207146" izz="0.00318737"/>
-      <mass value="2.25620359"/>
+      <origin xyz="0.005142373498529196 0.0024323677644133568 -0.12100915610790253"/>
+      <inertia ixx="0.02755964678927691" ixy="0.0" ixz="0.0" iyy="0.02735491706466737" iyz="0.0" izz="0.0028481453594764797"/>
+      <mass value="2.34"/>
     </inertial>
   </link>
@@ -634,5 +634,5 @@
     <parent link="hip3"/>
     <child link="upper3"/>
-    <origin xyz="0.0 -0.110945 0.0" rpy="0 0 0"/>
+    <origin xyz="0.0 -0.11080 0.0" rpy="0 0 0"/>
     <axis xyz="0 1 0"/>
     <limit effort="45" velocity="100.00" lower="-0.89884456477707963539" upper="2.2951079663725435509"/>
@@ -669,7 +669,7 @@
     </collision> -->
     <inertial>
-      <origin xyz="0.00597360 0.0 -0.17466427"/>
-      <inertia ixx="0.00701356" ixy="0.0" ixz="0.00006600" iyy="0.00709946" iyz="0.0" izz="0.00014529"/>
-      <mass value="0.330"/>
+      <origin xyz="0.00225794012658298 4.607596201822162e-05 -0.1800822913646698"/>
+      <inertia ixx="0.003999022654901177" ixy="0.0" ixz="0.0" iyy="0.0040503157598010785" iyz="0.0" izz="0.0001493402097647426"/>
+      <mass value="0.35"/>
     </inertial>
   </link>
@@ -681,7 +681,7 @@
     <parent link="upper3"/>
     <child link="lower3"/>
-    <origin xyz="0.025 0.000 -0.3205" rpy="0 0 0"/>
+    <origin xyz="0.025 0.000 -0.3200" rpy="0 0 0"/>
     <axis xyz="0 1 0"/>
-    <limit effort="115" velocity="100.00" lower="-2.7929" upper="-0.248282"/>
+    <limit effort="115" velocity="100.00" lower="-2.7929" upper="-0.247067"/>
     <dynamics damping="0" friction="0"/>
   </joint>
