Commit message: rviz ground truth fail

File: quad_simulator/go1_description/models/go1/go1.sdf.xacro (robot description, xacro)
@@ -75,108 +75,4 @@
         </geometry>
       </collision>
-      <collision name='trunk_fixed_joint_lump__camera_chin_collision_5'>
-        <pose>0.25219999999999998 0.012500000000000001 -0.0436 3.1415926535897931 1.5707963267948966 0</pose>
-        <geometry>
-          <box>
-            <size>0.001 0.001 0.001</size>
-          </box>
-        </geometry>
-        <surface>
-          <contact>
-            <ode/>
-          </contact>
-          <friction>
-            <ode/>
-          </friction>
-        </surface>
-      </collision>
-      <collision name='trunk_fixed_joint_lump__camera_face_collision_6'>
-        <pose>0.27850000000000003 0.012500000000000001 0.0167 3.1415926535897931 0 0</pose>
-        <geometry>
-          <box>
-            <size>0.001 0.001 0.001</size>
-          </box>
-        </geometry>
-        <surface>
-          <contact>
-            <ode/>
-          </contact>
-          <friction>
-            <ode/>
-          </friction>
-        </surface>
-      </collision>
-      <collision name='trunk_fixed_joint_lump__camera_left_collision_7'>
-        <pose>-0.066000000000000003 0.082000000000000003 -0.017600000000000001 3.1415926535897931 0.26179999999999998 1.5707963267948957</pose>
-        <geometry>
-          <box>
-            <size>0.001 0.001 0.001</size>
-          </box>
-        </geometry>
-        <surface>
-          <contact>
-            <ode/>
-          </contact>
-          <friction>
-            <ode/>
-          </friction>
-        </surface>
-      </collision>
-      <collision name='trunk_fixed_joint_lump__camera_rearDown_collision_8'>
-        <pose>-0.082500000000000004 0.012500000000000001 -0.043650000000000001 3.1415926535897931 1.5707963267948966 0</pose>
-        <geometry>
-          <box>
-            <size>0.001 0.001 0.001</size>
-          </box>
-        </geometry>
-        <surface>
-          <contact>
-            <ode/>
-          </contact>
-          <friction>
-            <ode/>
-          </friction>
-        </surface>
-      </collision>
-      <collision name='trunk_fixed_joint_lump__camera_right_collision_9'>
-        <pose>-0.041000000000000002 -0.082000000000000003 -0.017600000000000001 3.1415926535897931 0.26179999999999998 -1.570796326794897</pose>
-        <geometry>
-          <box>
-            <size>0.001 0.001 0.001</size>
-          </box>
-        </geometry>
-        <surface>
-          <contact>
-            <ode/>
-          </contact>
-          <friction>
-            <ode/>
-          </friction>
-        </surface>
-      </collision>
-      <collision name='trunk_fixed_joint_lump__ultraSound_face_collision_10'>
-        <pose>0.2747 0 -0.0088000000000000005 0 0 0</pose>
-        <geometry>
-          <box>
-            <size>0.001 0.001 0.001</size>
-          </box>
-        </geometry>
-      </collision>
-      <collision name='trunk_fixed_joint_lump__ultraSound_left_collision_11'>
-        <pose>-0.053499999999999999 0.082600000000000007 0.0086800000000000002 0 0.26179999999999998 1.570796326794897</pose>
-        <geometry>
-          <box>
-            <size>0.001 0.001 0.001</size>
-          </box>
-        </geometry>
-      </collision>
-      <collision name='trunk_fixed_joint_lump__ultraSound_right_collision_12'>
-        <pose>-0.053499999999999999 -0.082600000000000007 0.0086800000000000002 0 0.26179999999999998 -1.570796326794897</pose>
-        <geometry>
-          <box>
-            <size>0.001 0.001 0.001</size>
-          </box>
-        </geometry>
-      </collision>
       <visual name='trunk_visual'>
         <pose>0 0 0 0 0 0</pose>
@@ -184,5 +80,5 @@
           <mesh>
             <scale>1 1 1</scale>
-            <uri>model://go1/dae/trunk.dae</uri>
+            <uri>model://go1/meshes/trunk.dae</uri>
           </mesh>
         </geometry>
@@ -244,188 +140,4 @@
         </material>
       </visual>
-      <visual name='trunk_fixed_joint_lump__camera_chin_visual_5'>
-        <pose>0.25219999999999998 0.012500000000000001 -0.0436 3.1415926535897931 1.5707963267948966 0</pose>
-        <geometry>
-          <mesh>
-            <scale>1 1 1</scale>
-            <uri>model://go1/dae/depthCamera.dae</uri>
-          </mesh>
-        </geometry>
-        <material>
-          <diffuse>0.05 0.05 0.05 1</diffuse>
-          <ambient>0.05 0.05 0.05 1</ambient>
-        </material>
-      </visual>
-      <visual name='trunk_fixed_joint_lump__camera_face_visual_6'>
-        <pose>0.27850000000000003 0.012500000000000001 0.0167 3.1415926535897931 0 0</pose>
-        <geometry>
-          <mesh>
-            <scale>1 1 1</scale>
-            <uri>model://go1/dae/depthCamera.dae</uri>
-          </mesh>
-        </geometry>
-        <material>
-          <diffuse>0.05 0.05 0.05 1</diffuse>
-          <ambient>0.05 0.05 0.05 1</ambient>
-        </material>
-      </visual>
-      <visual name='trunk_fixed_joint_lump__camera_left_visual_7'>
-        <pose>-0.066000000000000003 0.082000000000000003 -0.017600000000000001 3.1415926535897931 0.26179999999999998 1.5707963267948957</pose>
-        <geometry>
-          <mesh>
-            <scale>1 1 1</scale>
-            <uri>model://go1/dae/depthCamera.dae</uri>
-          </mesh>
-        </geometry>
-        <material>
-          <diffuse>0.05 0.05 0.05 1</diffuse>
-          <ambient>0.05 0.05 0.05 1</ambient>
-        </material>
-      </visual>
-      <visual name='trunk_fixed_joint_lump__camera_rearDown_visual_8'>
-        <pose>-0.082500000000000004 0.012500000000000001 -0.043650000000000001 3.1415926535897931 1.5707963267948966 0</pose>
-        <geometry>
-          <mesh>
-            <scale>1 1 1</scale>
-            <uri>model://go1/dae/depthCamera.dae</uri>
-          </mesh>
-        </geometry>
-        <material>
-          <diffuse>0.05 0.05 0.05 1</diffuse>
-          <ambient>0.05 0.05 0.05 1</ambient>
-        </material>
-      </visual>
-      <visual name='trunk_fixed_joint_lump__camera_right_visual_9'>
-        <pose>-0.041000000000000002 -0.082000000000000003 -0.017600000000000001 3.1415926535897931 0.26179999999999998 -1.570796326794897</pose>
-        <geometry>
-          <mesh>
-            <scale>1 1 1</scale>
-            <uri>model://go1/dae/depthCamera.dae</uri>
-          </mesh>
-        </geometry>
-        <material>
-          <diffuse>0.05 0.05 0.05 1</diffuse>
-          <ambient>0.05 0.05 0.05 1</ambient>
-        </material>
-      </visual>
-      <visual name='trunk_fixed_joint_lump__ultraSound_face_visual_10'>
-        <pose>0.2747 0 -0.0088000000000000005 0 0 0</pose>
-        <geometry>
-          <mesh>
-            <scale>1 1 1</scale>
-            <uri>model://go1/dae/ultraSound.dae</uri>
-          </mesh>
-        </geometry>
-        <material>
-          <diffuse>0 0 0 1</diffuse>
-          <ambient>0 0 0 1</ambient>
-        </material>
-      </visual>
-      <visual name='trunk_fixed_joint_lump__ultraSound_left_visual_11'>
-        <pose>-0.053499999999999999 0.082600000000000007 0.0086800000000000002 0 0.26179999999999998 1.570796326794897</pose>
-        <geometry>
-          <mesh>
-            <scale>1 1 1</scale>
-            <uri>model://go1/dae/ultraSound.dae</uri>
-          </mesh>
-        </geometry>
-        <material>
-          <diffuse>0 0 0 1</diffuse>
-          <ambient>0 0 0 1</ambient>
-        </material>
-      </visual>
-      <visual name='trunk_fixed_joint_lump__ultraSound_right_visual_12'>
-        <pose>-0.053499999999999999 -0.082600000000000007 0.0086800000000000002 0 0.26179999999999998 -1.570796326794897</pose>
-        <geometry>
-          <mesh>
-            <scale>1 1 1</scale>
-            <uri>model://go1/dae/ultraSound.dae</uri>
-          </mesh>
-        </geometry>
-        <material>
-          <diffuse>0 0 0 1</diffuse>
-          <ambient>0 0 0 1</ambient>
-        </material>
-      </visual>
-      <sensor name='camera_chin_camera' type='depth'>
-        <update_rate>16</update_rate>
-        <camera>
-          <horizontal_fov>2.0939999999999999</horizontal_fov>
-          <image>
-            <width>928</width>
-            <height>800</height>
-            <format>R8G8B8</format>
-          </image>
-          <clip>
-            <near>0.10000000000000001</near>
-            <far>5</far>
-          </clip>
-        </camera>
-        <pose>0.25219999999999998 0.012500000000000001 -0.0436 3.1415926535897931 1.5707926536359933 2.6535897933410511e-06</pose>
-      </sensor>
-      <sensor name='camera_face_camera' type='depth'>
-        <update_rate>16</update_rate>
-        <camera>
-          <horizontal_fov>2.0939999999999999</horizontal_fov>
-          <image>
-            <width>928</width>
-            <height>800</height>
-            <format>R8G8B8</format>
-          </image>
-          <clip>
-            <near>0.10000000000000001</near>
-            <far>5</far>
-          </clip>
-        </camera>
-        <pose>0.27850000000000003 0.012500000000000001 0.0167 3.1415899999999999 0 0</pose>
-      </sensor>
-      <sensor name='camera_left_camera' type='depth'>
-        <update_rate>16</update_rate>
-        <camera>
-          <horizontal_fov>2.0939999999999999</horizontal_fov>
-          <image>
-            <width>928</width>
-            <height>800</height>
-            <format>R8G8B8</format>
-          </image>
-          <clip>
-            <near>0.10000000000000001</near>
-            <far>5</far>
-          </clip>
-        </camera>
-        <pose>-0.066000000000000003 0.082000000000000003 -0.017600000000000001 3.1415899999999999 0.26180000000000009 1.5708</pose>
-      </sensor>
-      <sensor name='camera_rearDown_camera' type='depth'>
-        <update_rate>16</update_rate>
-        <camera>
-          <horizontal_fov>2.0939999999999999</horizontal_fov>
-          <image>
-            <width>928</width>
-            <height>800</height>
-            <format>R8G8B8</format>
-          </image>
-          <clip>
-            <near>0.10000000000000001</near>
-            <far>5</far>
-          </clip>
-        </camera>
-        <pose>-0.082500000000000004 0.012500000000000001 -0.043650000000000001 3.1415926535897931 1.5707926536359933 2.6535897933410511e-06</pose>
-      </sensor>
-      <sensor name='camera_right_camera' type='depth'>
-        <update_rate>16</update_rate>
-        <camera>
-          <horizontal_fov>2.0939999999999999</horizontal_fov>
-          <image>
-            <width>928</width>
-            <height>800</height>
-            <format>R8G8B8</format>
-          </image>
-          <clip>
-            <near>0.10000000000000001</near>
-            <far>5</far>
-          </clip>
-        </camera>
-        <pose>-0.041000000000000002 -0.082000000000000003 -0.017600000000000001 3.1415899999999999 0.26179999999999998 -1.5707999999999998</pose>
-      </sensor>
     </link>
     <joint name='FL_hip_joint' type='revolute'>
@@ -497,5 +209,5 @@
           <mesh>
             <scale>1 1 1</scale>
-            <uri>model://go1/dae/hip.dae</uri>
+            <uri>model://go1/meshes/hip.dae</uri>
           </mesh>
         </geometry>
@@ -589,5 +301,5 @@
           <mesh>
             <scale>1 1 1</scale>
-            <uri>model://go1/dae/thigh.dae</uri>
+            <uri>model://go1/meshes/thigh.dae</uri>
           </mesh>
         </geometry>
@@ -670,5 +382,5 @@
           <mesh>
             <scale>1 1 1</scale>
-            <uri>model://go1/dae/calf.dae</uri>
+            <uri>model://go1/meshes/calf.dae</uri>
           </mesh>
         </geometry>
@@ -829,5 +541,5 @@
           <mesh>
             <scale>1 1 1</scale>
-            <uri>model://go1/dae/hip.dae</uri>
+            <uri>model://go1/meshes/hip.dae</uri>
           </mesh>
         </geometry>
@@ -921,5 +633,5 @@
           <mesh>
             <scale>1 1 1</scale>
-            <uri>model://go1/dae/thigh_mirror.dae</uri>
+            <uri>model://go1/meshes/thigh_mirror.dae</uri>
           </mesh>
         </geometry>
@@ -1002,5 +714,5 @@
           <mesh>
             <scale>1 1 1</scale>
-            <uri>model://go1/dae/calf.dae</uri>
+            <uri>model://go1/meshes/calf.dae</uri>
           </mesh>
         </geometry>
@@ -1161,5 +873,5 @@
           <mesh>
             <scale>1 1 1</scale>
-            <uri>model://go1/dae/hip.dae</uri>
+            <uri>model://go1/meshes/hip.dae</uri>
           </mesh>
         </geometry>
@@ -1253,5 +965,5 @@
           <mesh>
             <scale>1 1 1</scale>
-            <uri>model://go1/dae/thigh.dae</uri>
+            <uri>model://go1/meshes/thigh.dae</uri>
           </mesh>
         </geometry>
@@ -1334,5 +1046,5 @@
           <mesh>
             <scale>1 1 1</scale>
-            <uri>model://go1/dae/calf.dae</uri>
+            <uri>model://go1/meshes/calf.dae</uri>
           </mesh>
         </geometry>
@@ -1493,5 +1205,5 @@
           <mesh>
             <scale>1 1 1</scale>
-            <uri>model://go1/dae/hip.dae</uri>
+            <uri>model://go1/meshes/hip.dae</uri>
           </mesh>
         </geometry>
@@ -1585,5 +1297,5 @@
           <mesh>
             <scale>1 1 1</scale>
-            <uri>model://go1/dae/thigh_mirror.dae</uri>
+            <uri>model://go1/meshes/thigh_mirror.dae</uri>
           </mesh>
         </geometry>
@@ -1666,10 +1378,10 @@
           <mesh>
             <scale>1 1 1</scale>
-            <uri>model://go1/dae/calf.dae</uri>
+            <uri>model://go1/meshes/calf.dae</uri>
           </mesh>
         </geometry>
         <material>
-          <diffuse>0.2 0.2 0.2 1</diffuse>
-          <ambient>0.2 0.2 0.2 1</ambient>
+          <diffuse>1.0 0.4235294117647059 0.0392156862745098 1</diffuse>
+          <ambient>1.0 0.4235294117647059 0.0392156862745098 1</ambient>
         </material>
       </visual>
@@ -1751,6 +1463,6 @@
         </geometry>
         <material>
-          <diffuse>0.2 0.2 0.2 1</diffuse>
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