Commit message: rviz ground truth fail

File: quad_simulator/go1_description/models/go1/urdf/go1.urdf.xacro (robot description, xacro)
@@ -49,7 +49,9 @@
       <origin rpy="0 0 0" xyz="0 0 0"/>
       <geometry>
-        <mesh filename="package://go1_description/models/go1/dae/trunk.dae" scale="1 1 1"/>
-      </geometry>
-      <!-- <material name="orange"/> -->
+        <mesh filename="package://go1_description/models/go1/meshes/trunk.dae" scale="1 1 1"/>
+      </geometry>
+      <material name="">
+        <color rgba="1.0 0.4235294117647059 0.0392156862745098 1.0"/>
+      </material>
     </visual>
     <collision>
@@ -107,7 +109,9 @@
       <origin rpy="3.141592653589793 0 0" xyz="0 0 0"/>
       <geometry>
-        <mesh filename="package://go1_description/models/go1/dae/hip.dae" scale="1 1 1"/>
-      </geometry>
-      <!-- <material name="orange"/> -->
+        <mesh filename="package://go1_description/models/go1/meshes/hip.dae" scale="1 1 1"/>
+      </geometry>
+      <material name="">
+        <color rgba="1.0 0.4235294117647059 0.0392156862745098 1.0"/>
+      </material>
     </visual>
     <collision>
@@ -129,5 +133,7 @@
         <cylinder length="0.02" radius="0.035"/>
       </geometry>
-      <material name="green"/>
+      <material name="">
+        <color rgba="0.0 0.8 0.0 1.0"/>
+      </material>
     </visual>
     <collision>
@@ -160,7 +166,9 @@
       <origin rpy="0 0 0" xyz="0 0 0"/>
       <geometry>
-        <mesh filename="package://go1_description/models/go1/dae/thigh_mirror.dae" scale="1 1 1"/>
-      </geometry>
-      <!-- <material name="orange"/> -->
+        <mesh filename="package://go1_description/models/go1/meshes/thigh_mirror.dae" scale="1 1 1"/>
+      </geometry>
+      <material name="">
+        <color rgba="1.0 0.4235294117647059 0.0392156862745098 1.0"/>
+      </material>
     </visual>
     <collision>
@@ -182,5 +190,7 @@
         <cylinder length="0.02" radius="0.035"/>
       </geometry>
-      <material name="green"/>
+      <material name="">
+        <color rgba="0.0 0.8 0.0 1.0"/>
+      </material>
     </visual>
     <collision>
@@ -213,7 +223,9 @@
       <origin rpy="0 0 0" xyz="0 0 0"/>
       <geometry>
-        <mesh filename="package://go1_description/models/go1/dae/calf.dae" scale="1 1 1"/>
-      </geometry>
-      <!-- <material name="orange"/> -->
+        <mesh filename="package://go1_description/models/go1/meshes/calf.dae" scale="1 1 1"/>
+      </geometry>
+      <material name="">
+        <color rgba="1.0 0.4235294117647059 0.0392156862745098 1.0"/>
+      </material>
     </visual>
     <collision>
@@ -235,5 +247,7 @@
         <cylinder length="0.02" radius="0.035"/>
       </geometry>
-      <material name="green"/>
+      <material name="">
+        <color rgba="0.0 0.8 0.0 1.0"/>
+      </material>
     </visual>
     <collision>
@@ -260,5 +274,7 @@
         <sphere radius="0.01"/>
       </geometry>
-      <!-- <material name="orange"/> -->
+      <material name="">
+        <color rgba="1.0 0.4235294117647059 0.0392156862745098 1.0"/>
+      </material>
     </visual>
     <collision>
@@ -273,34 +289,4 @@
     </inertial>
   </link>
-  <transmission name="FR_hip_tran">
-    <type>transmission_interface/SimpleTransmission</type>
-    <joint name="FR_hip_joint">
-      <hardwareInterface>hardware_interface/EffortJointInterface</hardwareInterface>
-    </joint>
-    <actuator name="FR_hip_motor">
-      <hardwareInterface>hardware_interface/EffortJointInterface</hardwareInterface>
-      <mechanicalReduction>1</mechanicalReduction>
-    </actuator>
-  </transmission>
-  <transmission name="FR_thigh_tran">
-    <type>transmission_interface/SimpleTransmission</type>
-    <joint name="FR_thigh_joint">
-      <hardwareInterface>hardware_interface/EffortJointInterface</hardwareInterface>
-    </joint>
-    <actuator name="FR_thigh_motor">
-      <hardwareInterface>hardware_interface/EffortJointInterface</hardwareInterface>
-      <mechanicalReduction>1</mechanicalReduction>
-    </actuator>
-  </transmission>
-  <transmission name="FR_calf_tran">
-    <type>transmission_interface/SimpleTransmission</type>
-    <joint name="FR_calf_joint">
-      <hardwareInterface>hardware_interface/EffortJointInterface</hardwareInterface>
-    </joint>
-    <actuator name="FR_calf_motor">
-      <hardwareInterface>hardware_interface/EffortJointInterface</hardwareInterface>
-      <mechanicalReduction>1</mechanicalReduction>
-    </actuator>
-  </transmission>
   <joint name="FL_hip_joint" type="revolute">
     <origin rpy="0 0 0" xyz="0.1881 0.04675 0"/>
@@ -320,7 +306,9 @@
       <origin rpy="0 0 0" xyz="0 0 0"/>
       <geometry>
-        <mesh filename="package://go1_description/models/go1/dae/hip.dae" scale="1 1 1"/>
-      </geometry>
-      <!-- <material name="orange"/> -->
+        <mesh filename="package://go1_description/models/go1/meshes/hip.dae" scale="1 1 1"/>
+      </geometry>
+      <material name="">
+        <color rgba="1.0 0.4235294117647059 0.0392156862745098 1.0"/>
+      </material>
     </visual>
     <collision>
@@ -342,5 +330,7 @@
         <cylinder length="0.02" radius="0.035"/>
       </geometry>
-      <material name="green"/>
+      <material name="">
+        <color rgba="0.0 0.8 0.0 1.0"/>
+      </material>
     </visual>
     <collision>
@@ -373,7 +363,9 @@
       <origin rpy="0 0 0" xyz="0 0 0"/>
       <geometry>
-        <mesh filename="package://go1_description/models/go1/dae/thigh.dae" scale="1 1 1"/>
-      </geometry>
-      <!-- <material name="orange"/> -->
+        <mesh filename="package://go1_description/models/go1/meshes/thigh.dae" scale="1 1 1"/>
+      </geometry>
+      <material name="">
+        <color rgba="1.0 0.4235294117647059 0.0392156862745098 1.0"/>
+      </material>
     </visual>
     <collision>
@@ -395,5 +387,7 @@
         <cylinder length="0.02" radius="0.035"/>
       </geometry>
-      <material name="green"/>
+      <material name="">
+        <color rgba="0.0 0.8 0.0 1.0"/>
+      </material>
     </visual>
     <collision>
@@ -426,7 +420,9 @@
       <origin rpy="0 0 0" xyz="0 0 0"/>
       <geometry>
-        <mesh filename="package://go1_description/models/go1/dae/calf.dae" scale="1 1 1"/>
-      </geometry>
-      <!-- <material name="orange"/> -->
+        <mesh filename="package://go1_description/models/go1/meshes/calf.dae" scale="1 1 1"/>
+      </geometry>
+      <material name="">
+        <color rgba="1.0 0.4235294117647059 0.0392156862745098 1.0"/>
+      </material>
     </visual>
     <collision>
@@ -448,5 +444,7 @@
         <cylinder length="0.02" radius="0.035"/>
       </geometry>
-      <material name="green"/>
+      <material name="">
+        <color rgba="0.0 0.8 0.0 1.0"/>
+      </material>
     </visual>
     <collision>
@@ -473,5 +471,7 @@
         <sphere radius="0.01"/>
       </geometry>
-      <!-- <material name="orange"/> -->
+      <material name="">
+        <color rgba="1.0 0.4235294117647059 0.0392156862745098 1.0"/>
+      </material>
     </visual>
     <collision>
@@ -486,34 +486,4 @@
     </inertial>
   </link>
-  <transmission name="FL_hip_tran">
-    <type>transmission_interface/SimpleTransmission</type>
-    <joint name="FL_hip_joint">
-      <hardwareInterface>hardware_interface/EffortJointInterface</hardwareInterface>
-    </joint>
-    <actuator name="FL_hip_motor">
-      <hardwareInterface>hardware_interface/EffortJointInterface</hardwareInterface>
-      <mechanicalReduction>1</mechanicalReduction>
-    </actuator>
-  </transmission>
-  <transmission name="FL_thigh_tran">
-    <type>transmission_interface/SimpleTransmission</type>
-    <joint name="FL_thigh_joint">
-      <hardwareInterface>hardware_interface/EffortJointInterface</hardwareInterface>
-    </joint>
-    <actuator name="FL_thigh_motor">
-      <hardwareInterface>hardware_interface/EffortJointInterface</hardwareInterface>
-      <mechanicalReduction>1</mechanicalReduction>
-    </actuator>
-  </transmission>
-  <transmission name="FL_calf_tran">
-    <type>transmission_interface/SimpleTransmission</type>
-    <joint name="FL_calf_joint">
-      <hardwareInterface>hardware_interface/EffortJointInterface</hardwareInterface>
-    </joint>
-    <actuator name="FL_calf_motor">
-      <hardwareInterface>hardware_interface/EffortJointInterface</hardwareInterface>
-      <mechanicalReduction>1</mechanicalReduction>
-    </actuator>
-  </transmission>
   <joint name="RR_hip_joint" type="revolute">
     <origin rpy="0 0 0" xyz="-0.1881 -0.04675 0"/>
@@ -533,7 +503,9 @@
       <origin rpy="3.141592653589793 3.141592653589793 0" xyz="0 0 0"/>
       <geometry>
-        <mesh filename="package://go1_description/models/go1/dae/hip.dae" scale="1 1 1"/>
-      </geometry>
-      <!-- <material name="orange"/> -->
+        <mesh filename="package://go1_description/models/go1/meshes/hip.dae" scale="1 1 1"/>
+      </geometry>
+      <material name="">
+        <color rgba="1.0 0.4235294117647059 0.0392156862745098 1.0"/>
+      </material>
     </visual>
     <collision>
@@ -555,5 +527,7 @@
         <cylinder length="0.02" radius="0.035"/>
       </geometry>
-      <material name="green"/>
+      <material name="">
+        <color rgba="0.0 0.8 0.0 1.0"/>
+      </material>
     </visual>
     <collision>
@@ -586,7 +560,9 @@
       <origin rpy="0 0 0" xyz="0 0 0"/>
       <geometry>
-        <mesh filename="package://go1_description/models/go1/dae/thigh_mirror.dae" scale="1 1 1"/>
-      </geometry>
-      <!-- <material name="orange"/> -->
+        <mesh filename="package://go1_description/models/go1/meshes/thigh_mirror.dae" scale="1 1 1"/>
+      </geometry>
+      <material name="">
+        <color rgba="1.0 0.4235294117647059 0.0392156862745098 1.0"/>
+      </material>
     </visual>
     <collision>
@@ -608,5 +584,7 @@
         <cylinder length="0.02" radius="0.035"/>
       </geometry>
-      <material name="green"/>
+      <material name="">
+        <color rgba="0.0 0.8 0.0 1.0"/>
+      </material>
     </visual>
     <collision>
@@ -639,7 +617,9 @@
       <origin rpy="0 0 0" xyz="0 0 0"/>
       <geometry>
-        <mesh filename="package://go1_description/models/go1/dae/calf.dae" scale="1 1 1"/>
-      </geometry>
-      <!-- <material name="orange"/> -->
+        <mesh filename="package://go1_description/models/go1/meshes/calf.dae" scale="1 1 1"/>
+      </geometry>
+      <material name="">
+        <color rgba="1.0 0.4235294117647059 0.0392156862745098 1.0"/>
+      </material>
     </visual>
     <collision>
@@ -661,5 +641,7 @@
         <cylinder length="0.02" radius="0.035"/>
       </geometry>
-      <material name="green"/>
+      <material name="">
+        <color rgba="0.0 0.8 0.0 1.0"/>
+      </material>
     </visual>
     <collision>
@@ -686,5 +668,7 @@
         <sphere radius="0.01"/>
       </geometry>
-      <!-- <material name="orange"/> -->
+      <material name="">
+        <color rgba="1.0 0.4235294117647059 0.0392156862745098 1.0"/>
+      </material>
     </visual>
     <collision>
@@ -699,34 +683,4 @@
     </inertial>
   </link>
-  <transmission name="RR_hip_tran">
-    <type>transmission_interface/SimpleTransmission</type>
-    <joint name="RR_hip_joint">
-      <hardwareInterface>hardware_interface/EffortJointInterface</hardwareInterface>
-    </joint>
-    <actuator name="RR_hip_motor">
-      <hardwareInterface>hardware_interface/EffortJointInterface</hardwareInterface>
-      <mechanicalReduction>1</mechanicalReduction>
-    </actuator>
-  </transmission>
-  <transmission name="RR_thigh_tran">
-    <type>transmission_interface/SimpleTransmission</type>
-    <joint name="RR_thigh_joint">
-      <hardwareInterface>hardware_interface/EffortJointInterface</hardwareInterface>
-    </joint>
-    <actuator name="RR_thigh_motor">
-      <hardwareInterface>hardware_interface/EffortJointInterface</hardwareInterface>
-      <mechanicalReduction>1</mechanicalReduction>
-    </actuator>
-  </transmission>
-  <transmission name="RR_calf_tran">
-    <type>transmission_interface/SimpleTransmission</type>
-    <joint name="RR_calf_joint">
-      <hardwareInterface>hardware_interface/EffortJointInterface</hardwareInterface>
-    </joint>
-    <actuator name="RR_calf_motor">
-      <hardwareInterface>hardware_interface/EffortJointInterface</hardwareInterface>
-      <mechanicalReduction>1</mechanicalReduction>
-    </actuator>
-  </transmission>
   <joint name="RL_hip_joint" type="revolute">
     <origin rpy="0 0 0" xyz="-0.1881 0.04675 0"/>
@@ -746,7 +700,9 @@
       <origin rpy="0 3.141592653589793 0" xyz="0 0 0"/>
       <geometry>
-        <mesh filename="package://go1_description/models/go1/dae/hip.dae" scale="1 1 1"/>
-      </geometry>
-      <!-- <material name="orange"/> -->
+        <mesh filename="package://go1_description/models/go1/meshes/hip.dae" scale="1 1 1"/>
+      </geometry>
+      <material name="">
+        <color rgba="1.0 0.4235294117647059 0.0392156862745098 1.0"/>
+      </material>
     </visual>
     <collision>
@@ -768,5 +724,7 @@
         <cylinder length="0.02" radius="0.035"/>
       </geometry>
-      <material name="green"/>
+      <material name="">
+        <color rgba="0.0 0.8 0.0 1.0"/>
+      </material>
     </visual>
     <collision>
@@ -799,7 +757,9 @@
       <origin rpy="0 0 0" xyz="0 0 0"/>
       <geometry>
-        <mesh filename="package://go1_description/models/go1/dae/thigh.dae" scale="1 1 1"/>
-      </geometry>
-      <!-- <material name="orange"/> -->
+        <mesh filename="package://go1_description/models/go1/meshes/thigh.dae" scale="1 1 1"/>
+      </geometry>
+      <material name="">
+        <color rgba="1.0 0.4235294117647059 0.0392156862745098 1.0"/>
+      </material>
     </visual>
     <collision>
@@ -821,5 +781,7 @@
         <cylinder length="0.02" radius="0.035"/>
       </geometry>
-      <material name="green"/>
+      <material name="">
+        <color rgba="0.0 0.8 0.0 1.0"/>
+      </material>
     </visual>
     <collision>
@@ -852,7 +814,9 @@
       <origin rpy="0 0 0" xyz="0 0 0"/>
       <geometry>
-        <mesh filename="package://go1_description/models/go1/dae/calf.dae" scale="1 1 1"/>
-      </geometry>
-      <!-- <material name="orange"/> -->
+        <mesh filename="package://go1_description/models/go1/meshes/calf.dae" scale="1 1 1"/>
+      </geometry>
+      <material name="">
+        <color rgba="1.0 0.4235294117647059 0.0392156862745098 1.0"/>
+      </material>
     </visual>
     <collision>
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