Commit message: Working Multi-Agent Launch Sequence

File: quad_simulator/go2w_description/models/go2w/go2w.sdf.xacro (robot description, xacro)
@@ -1,16 +1,17 @@
 <?xml version='1.0'?>
-<sdf version='1.11'>
-  <model name='go2'>
+<sdf version='1.11' xmlns:xacro="http://www.ros.org/wiki/xacro">
+  <xacro:arg name="namespace" default="robot_1" />
+  <model name='go2w'>
     <link name='body'>
       <inertial>
-        <pose>0.020153063882401429 0 -0.0051089553510097526 0 0 0</pose>
-        <mass>7.2790000000000017</mass>
-        <inertia>
-          <ixx>0.025737618948512481</ixx>
+        <pose>0.021189390726563631 0 -0.0053716721074678611 0 0 0</pose>
+        <mass>6.923</mass>
+        <inertia>
+          <ixx>0.02450242076517968</ixx>
           <ixy>0.00012166</ixy>
-          <ixz>0.001534235398809762</ixz>
-          <iyy>0.1031209538931058</iyy>
+          <ixz>0.0014956963870049491</ixz>
+          <iyy>0.098242939262173756</iyy>
           <iyz>-3.1199999999999999e-05</iyz>
-          <izz>0.1128090234445933</izz>
+          <izz>0.1071627184969941</izz>
         </inertia>
       </inertial>
@@ -28,5 +29,5 @@
           <cylinder>
             <length>0.089999999999999997</length>
-            <radius>0.050000000000000003</radius>
+            <radius>0.059999999999999998</radius>
           </cylinder>
         </geometry>
@@ -36,5 +37,5 @@
         <geometry>
           <sphere>
-            <radius>0.047</radius>
+            <radius>0.059999999999999998</radius>
           </sphere>
         </geometry>
@@ -45,5 +46,5 @@
           <mesh>
             <scale>1 1 1</scale>
-            <uri>model://go2/dae/body.dae</uri>
+            <uri>model://go2w/dae/body.dae</uri>
           </mesh>
         </geometry>
@@ -75,13 +76,13 @@
       <pose relative_to='8'>0 0 0 0 0 0</pose>
       <inertial>
-        <pose>-0.0047734028683181226 0.00169748370273794 -9.2816166883963517e-05 0 0 0</pose>
-        <mass>0.76700000000000002</mass>
-        <inertia>
-          <ixx>0.00053999151781062584</ixx>
-          <ixy>-2.1220993324641449e-06</ixy>
-          <ixz>1.0653925501955671e-06</ixz>
-          <iyy>0.00099813696478559337</iyy>
-          <iyz>-1.4027352647979141e-06</iyz>
-          <izz>0.00065828474786205991</izz>
+        <pose>-0.0054000000000000003 0.0019400000000000001 -0.000105 0 0 0</pose>
+        <mass>0.67800000000000005</mass>
+        <inertia>
+          <ixx>0.00048000000000000001</ixx>
+          <ixy>-3.01e-06</ixy>
+          <ixz>1.11e-06</ixz>
+          <iyy>0.00088400000000000002</iyy>
+          <iyz>-1.42e-06</iyz>
+          <izz>0.00059599999999999996</izz>
         </inertia>
       </inertial>
@@ -100,5 +101,5 @@
           <mesh>
             <scale>1 1 1</scale>
-            <uri>model://go2/dae/hip.dae</uri>
+            <uri>model://go2w/dae/hip.dae</uri>
           </mesh>
         </geometry>
@@ -130,13 +131,13 @@
       <pose relative_to='0'>0 0 0 0 0 0</pose>
       <inertial>
-        <pose>-0.003471780821917808 -0.02302074939564867 -0.03035487510072523 0 0 0</pose>
-        <mass>1.2410000000000001</mass>
-        <inertia>
-          <ixx>0.0059963333412087023</ixx>
-          <ixy>9.0305334356164388e-05</ixy>
-          <ixz>-0.00029910392372602731</ixz>
-          <iyy>0.0060013394099700237</iyy>
-          <iyz>0.00083515091803384382</iyz>
-          <izz>0.0010991471651674461</izz>
+        <pose>-0.0037399999999999998 -0.0223 -0.0327 0 0 0</pose>
+        <mass>1.1519999999999999</mass>
+        <inertia>
+          <ixx>0.0058399999999999997</ixx>
+          <ixy>8.7200000000000005e-05</ixy>
+          <ixz>-0.00028899999999999998</ixz>
+          <iyy>0.0057999999999999996</iyy>
+          <iyz>0.00080800000000000002</iyz>
+          <izz>0.0010300000000000001</izz>
         </inertia>
       </inertial>
@@ -145,5 +146,5 @@
         <geometry>
           <box>
-            <size>0.21299999999999999 0.024500000000000001 0.034000000000000002</size>
+            <size>0.11 0.024500000000000001 0.034000000000000002</size>
           </box>
         </geometry>
@@ -172,6 +173,6 @@
           <lower>0.445059</lower>
           <upper>2.22529</upper>
-          <effort>45.43</effort>
-          <velocity>15.699999999999999</velocity>
+          <effort>35.549999999999997</effort>
+          <velocity>20.07</velocity>
         </limit>
         <dynamics>
@@ -184,13 +185,13 @@
       <pose relative_to='1'>0 0 0 0 0 0</pose>
       <inertial>
-        <pose>0.0043501030927835041 -0.00077396907216494828 -0.13520618556701031 0 0 0</pose>
-        <mass>0.19400000000000001</mass>
-        <inertia>
-          <ixx>0.001394581937371134</ixx>
-          <ixy>5.0965402061855686e-07</ixy>
-          <ixz>1.4759587628868399e-07</ixz>
-          <iyy>0.001415505295175258</iyy>
-          <iyz>1.1313958762886591e-05</iyz>
-          <izz>4.3483727391752568e-05</izz>
+        <pose>0.0010548999999999999 0.0078873125000000002 -0.20495550000000001 0 0 0</pose>
+        <mass>0.80000000000000004</mass>
+        <inertia>
+          <ixx>0.00363821921327187</ixx>
+          <ixy>7.8190827650000003e-06</ixy>
+          <ixz>-5.8715245559999983e-05</ixz>
+          <iyy>0.0042469750061919836</iyy>
+          <iyz>0.0001603182883249997</iyz>
+          <izz>0.001051613067863875</izz>
         </inertia>
       </inertial>
@@ -222,10 +223,11 @@
         </geometry>
       </collision>
-      <collision name='lower0_fixed_joint_lump__FL_foot_collision_3'>
-        <pose>-0.002 0 -0.21299999999999999 0 0 0</pose>
-        <geometry>
-          <sphere>
-            <radius>0.021999999999999999</radius>
-          </sphere>
+      <collision name='lower0_fixed_joint_lump__FL_foot_motor_collision_3'>
+        <pose>0 0.01 -0.22639999999999999 1.5707963267948959 0 0</pose>
+        <geometry>
+          <cylinder>
+            <length>0.050000000000000003</length>
+            <radius>0.050000000000000003</radius>
+          </cylinder>
         </geometry>
       </collision>
@@ -235,97 +237,67 @@
           <mesh>
             <scale>1 1 1</scale>
-            <uri>model://go2/dae/calf.dae</uri>
-          </mesh>
-        </geometry>
-        <material>
-          <diffuse>1 1 1 1</diffuse>
-          <ambient>1 1 1 1</ambient>
-        </material>
-      </visual>
-      <visual name='lower_fixed_joint_lump__FL_foot_visual_1'>
-        <pose>0 0 -0.21299999999999999 0 0 0</pose>
-        <geometry>
-          <mesh>
-            <scale>1 1 1</scale>
-            <uri>model://go2/dae/foot.dae</uri>
-          </mesh>
-        </geometry>
-        <material>
-          <diffuse>1 1 1 1</diffuse>
-          <ambient>1 1 1 1</ambient>
-        </material>
-      </visual>
-    </link>
-    <joint name='jtoe0' type='fixed'>
-      <pose relative_to='lower0'>0 0 -0.213 0 0 0</pose>
+            <uri>model://go2w/dae/calf.stl</uri>
+          </mesh>
+        </geometry>
+        <material>
+          <diffuse>1 1 1 1</diffuse>
+          <ambient>1 1 1 1</ambient>
+        </material>
+      </visual>
+    </link>
+    <joint name='jtoe0' type='revolute'>
+      <pose relative_to='lower0'>0 0 -0.22639999999999999 0 0 0</pose>
       <parent>lower0</parent>
       <child>toe0</child>
       <axis>
-        <xyz>0 0 1</xyz>
-        <limit>
-          <lower>-1e+16</lower>
-          <upper>1e+16</upper>
-        </limit>
-        <dynamics>
-          <spring_reference>0</spring_reference>
-          <spring_stiffness>0</spring_stiffness>
-        </dynamics>
-      </axis>
-      <physics>
-        <ode>
-          <limit>
-            <cfm>0</cfm>
-            <erp>0.2</erp>
-          </limit>
-        </ode>
-      </physics>
-    </joint>
-    <link name="toe0">
+        <xyz>0 1 0</xyz>
+        <limit>
+          <effort>23.699999999999999</effort>
+          <velocity>30.100000000000001</velocity>
+          <lower>-inf</lower>
+          <upper>inf</upper>
+        </limit>
+        <dynamics>
+          <spring_reference>0</spring_reference>
+          <spring_stiffness>0</spring_stiffness>
+        </dynamics>
+      </axis>
+    </joint>
+    <link name='toe0'>
       <pose relative_to='jtoe0'>0 0 0 0 0 0</pose>
       <inertial>
-        <mass>0.04</mass>
-        <inertia>
-          <ixx>9.6e-06</ixx>
+        <pose>0 0.059999999999999998 0 0 0 0</pose>
+        <mass>0.52000000000000002</mass>
+        <inertia>
+          <ixx>0.00069999999999999999</ixx>
           <ixy>0</ixy>
           <ixz>0</ixz>
-          <iyy>9.6e-06</iyy>
+          <iyy>0.0011999999999999999</iyy>
           <iyz>0</iyz>
-          <izz>9.6e-06</izz>
-        </inertia>
-      </inertial>
-      <visual name="toe0_visual">
-        <pose>0 0 0 0 0 0</pose>
-        <geometry>
-          <sphere>
-            <radius>0.022</radius>
-          </sphere>
-        </geometry>
-        <material>
-          <ambient>1 1 1 1</ambient>
-          <diffuse>1 1 1 1</diffuse>
-        </material>
-      </visual>
-      <collision name="toe0_collision">
-        <pose>-0.002 0 0 0 0 0</pose>
-        <geometry>
-          <sphere>
-            <radius>0.022</radius>
-          </sphere>
-        </geometry>
-        <surface>
-          <contact>
-            <ode>
-              <kp>1e+06</kp>
-              <kd>1</kd>
-            </ode>
-          </contact>
-          <friction>
-            <ode>
-              <mu>0.6</mu>
-              <mu2>0.6</mu2>
-            </ode>
-          </friction>
-        </surface>
-      </collision>
+          <izz>0.00069999999999999999</izz>
+        </inertia>
+      </inertial>
+      <collision name='toe0_collision'>
+        <pose>0 0 0 1.5707963267948959 0 0</pose>
+        <geometry>
+          <mesh>
+            <scale>1 1 1</scale>
+            <uri>model://go2w/dae/left_wheel.dae</uri>
+          </mesh>
+        </geometry>
+      </collision>
+      <visual name='toe0_visual'>
+        <pose>0 0 0 0 0 0</pose>
+        <geometry>
+          <mesh>
+            <scale>1 1 1</scale>
+            <uri>model://go2w/dae/left_wheel.dae</uri>
+          </mesh>
+        </geometry>
+        <material>
+          <diffuse>1 1 1 1</diffuse>
+          <ambient>1 1 1 1</ambient>
+        </material>
+      </visual>
       <sensor name="toe0_contact" type="contact">
         <alwaysOn>true</alwaysOn>
@@ -363,13 +335,13 @@
       <pose relative_to='10'>0 0 0 0 0 0</pose>
       <inertial>
-        <pose>-0.0047734028683181226 -0.00169748370273794 -9.2816166883963517e-05 0 0 0</pose>
-        <mass>0.76700000000000002</mass>
-        <inertia>
-          <ixx>0.00053999151781062584</ixx>
-          <ixy>2.1220993324641449e-06</ixy>
-          <ixz>1.0653925501955671e-06</ixz>
-          <iyy>0.00099813696478559337</iyy>
-          <iyz>1.4027352647979141e-06</iyz>
-          <izz>0.00065828474786205991</izz>
+        <pose>-0.0054000000000000003 -0.0019400000000000001 -0.000105 0 0 0</pose>
+        <mass>0.67800000000000005</mass>
+        <inertia>
+          <ixx>0.00048000000000000001</ixx>
+          <ixy>3.01e-06</ixy>
+          <ixz>1.11e-06</ixz>
+          <iyy>0.00088400000000000002</iyy>
+          <iyz>1.42e-06</iyz>
+          <izz>0.00059599999999999996</izz>
         </inertia>
       </inertial>
@@ -388,5 +360,5 @@
           <mesh>
             <scale>1 1 1</scale>
-            <uri>model://go2/dae/hip.dae</uri>
+            <uri>model://go2w/dae/hip.dae</uri>
           </mesh>
         </geometry>
@@ -418,13 +390,13 @@
       <pose relative_to='4'>0 0 0 0 0 0</pose>
       <inertial>
-        <pose>-0.003471780821917808 0.02302074939564867 -0.03035487510072523 0 0 0</pose>
-        <mass>1.2410000000000001</mass>
-        <inertia>
-          <ixx>0.0059963333412087023</ixx>
-          <ixy>-9.0305334356164388e-05</ixy>
-          <ixz>-0.00029910392372602731</ixz>
-          <iyy>0.0060013394099700237</iyy>
-          <iyz>-0.00083515091803384382</iyz>
-          <izz>0.0010991471651674461</izz>
+        <pose>-0.0037399999999999998 0.0223 -0.0327 0 0 0</pose>
+        <mass>1.1519999999999999</mass>
+        <inertia>
+          <ixx>0.0058399999999999997</ixx>
+          <ixy>-8.7200000000000005e-05</ixy>
+          <ixz>-0.00028899999999999998</ixz>
+          <iyy>0.0057999999999999996</iyy>
+          <iyz>-0.00080800000000000002</iyz>
+          <izz>0.0010300000000000001</izz>
         </inertia>
       </inertial>
@@ -433,5 +405,5 @@
         <geometry>
           <box>
-            <size>0.21299999999999999 0.024500000000000001 0.034000000000000002</size>
+            <size>0.11 0.024500000000000001 0.034000000000000002</size>
           </box>
         </geometry>
@@ -442,5 +414,5 @@
           <mesh>
             <scale>1 1 1</scale>
-            <uri>model://go2/dae/thigh_mirror.dae</uri>
+            <uri>model://go2w/dae/thigh_mirror.dae</uri>
           </mesh>
         </geometry>
@@ -460,6 +432,6 @@
           <lower>0.445059</lower>
           <upper>2.22529</upper>
-          <effort>45.43</effort>
-          <velocity>15.699999999999999</velocity>
+          <effort>35.549999999999997</effort>
+          <velocity>20.07</velocity>
         </limit>
         <dynamics>
@@ -472,13 +444,13 @@
       <pose relative_to='5'>0 0 0 0 0 0</pose>
       <inertial>
-        <pose>0.0043501030927835041 0.00077396907216494828 -0.13520618556701031 0 0 0</pose>
-        <mass>0.19400000000000001</mass>
-        <inertia>
-          <ixx>0.001394581937371134</ixx>
-          <ixy>-5.0965402061855686e-07</ixy>
-          <ixz>1.4759587628868399e-07</ixz>
-          <iyy>0.001415505295175258</iyy>
-          <iyz>-1.1313958762886591e-05</iyz>
-          <izz>4.3483727391752568e-05</izz>
+        <pose>0.0010548999999999999 -0.0078873125000000002 -0.20495550000000001 0 0 0</pose>
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
File: quad_simulator/spirit_description/models/spirit/spirit.sdf.xacro (robot description, xacro)
@@ -1,4 +1,5 @@
 <?xml version='1.0'?>
-<sdf version='1.6'>
+<sdf version='1.6' xmlns:xacro="http://www.ros.org/wiki/xacro">
+  <xacro:arg name="namespace" default="robot_1" />
   <model name='spirit'>
     <link name='body'>
@@ -1196,5 +1197,5 @@
           <parameters>/home/rml/ros2_ws/install/gazebo_scripts/share/gazebo_scripts/config/quad_control.yaml</parameters>
               <ros>
-                <namespace>robot_1</namespace>
+                <namespace>$(arg namespace)</namespace>
             </ros>
       </plugin>
