Commit message: Go1 added, All robot works with latest yaml convention update, Aesthetics upgrade on all robots

File: quad_simulator/a1_description/models/a1/a1.sdf.xacro (robot description, xacro)
@@ -1337,4 +1337,13 @@
     <joint name="imu_joint" type="fixed">
       <child>imu::link</child>
+      <parent>body</parent>
+    </joint>
+    <include>
+      <uri>model://cmu_text</uri>
+      <name>cmu_text</name>
+      <pose>0 0 0 0 0 0</pose>
+    </include>
+    <joint name="cmu_text_joint" type="fixed">
+      <child>cmu_text::text</child>
       <parent>body</parent>
     </joint>

File: quad_simulator/a1_description/models/a1/urdf/a1.urdf.xacro (robot description, xacro)
@@ -1182,3 +1182,20 @@
     </joint>
   </ros2_control>
+  <link name="cmu_text">
+    <visual>
+      <origin xyz="0 0 0" rpy="0 0 0" />
+      <geometry>
+        <mesh filename="package://objects_description/models/cmu_text/meshes/Spirit40_CMU_Text_transformed.stl" scale="1.3 1 1.3" />
+      </geometry>
+    </visual>
+    <inertial>
+      <mass value="0.0001" />
+      <inertia ixx="1e-08" ixy="0" ixz="0" iyy="1e-08" iyz="0" izz="1e-08" />
+    </inertial>
+  </link>
+  <joint name="cmu_text_joint" type="fixed">
+    <parent link="body" />
+    <child link="cmu_text" />
+    <origin xyz="0 0 -0.005" rpy="0 0 0" />
+  </joint>
 </robot>

File: quad_simulator/b2_description/models/b2/b2.sdf.xacro (robot description, xacro)
@@ -1447,4 +1447,13 @@
     <joint name="imu_joint" type="fixed">
       <child>imu::link</child>
+      <parent>body</parent>
+    </joint>
+    <include>
+      <uri>model://cmu_text</uri>
+      <name>cmu_text</name>
+      <pose>0 0 0 0 0 0</pose>
+    </include>
+    <joint name="cmu_text_joint" type="fixed">
+      <child>cmu_text::text</child>
       <parent>body</parent>
     </joint>

File: quad_simulator/b2_description/models/b2/urdf/b2.urdf.xacro (robot description, xacro)
@@ -1596,3 +1596,20 @@
     </joint>
   </ros2_control>
+  <link name="cmu_text">
+    <visual>
+      <origin xyz="0 0 0" rpy="0 0 0" />
+      <geometry>
+        <mesh filename="package://objects_description/models/cmu_text/meshes/Spirit40_CMU_Text_transformed.stl" scale="1.3 1 1.3" />
+      </geometry>
+    </visual>
+    <inertial>
+      <mass value="0.0001" />
+      <inertia ixx="1e-08" ixy="0" ixz="0" iyy="1e-08" iyz="0" izz="1e-08" />
+    </inertial>
+  </link>
+  <joint name="cmu_text_joint" type="fixed">
+    <parent link="body" />
+    <child link="cmu_text" />
+    <origin xyz="0 0 -0.005" rpy="0 0 0" />
+  </joint>
 </robot>

File: quad_simulator/go1_description/models/go1/go1.sdf.xacro (robot description, xacro)
@@ -75,4 +75,108 @@
         </geometry>
       </collision>
+      <collision name='trunk_fixed_joint_lump__camera_chin_collision_5'>
+        <pose>0.25219999999999998 0.012500000000000001 -0.0436 3.1415926535897931 1.5707963267948966 0</pose>
+        <geometry>
+          <box>
+            <size>0.001 0.001 0.001</size>
+          </box>
+        </geometry>
+        <surface>
+          <contact>
+            <ode/>
+          </contact>
+          <friction>
+            <ode/>
+          </friction>
+        </surface>
+      </collision>
+      <collision name='trunk_fixed_joint_lump__camera_face_collision_6'>
+        <pose>0.27850000000000003 0.012500000000000001 0.0167 3.1415926535897931 0 0</pose>
+        <geometry>
+          <box>
+            <size>0.001 0.001 0.001</size>
+          </box>
+        </geometry>
+        <surface>
+          <contact>
+            <ode/>
+          </contact>
+          <friction>
+            <ode/>
+          </friction>
+        </surface>
+      </collision>
+      <collision name='trunk_fixed_joint_lump__camera_left_collision_7'>
+        <pose>-0.066000000000000003 0.082000000000000003 -0.017600000000000001 3.1415926535897931 0.26179999999999998 1.5707963267948957</pose>
+        <geometry>
+          <box>
+            <size>0.001 0.001 0.001</size>
+          </box>
+        </geometry>
+        <surface>
+          <contact>
+            <ode/>
+          </contact>
+          <friction>
+            <ode/>
+          </friction>
+        </surface>
+      </collision>
+      <collision name='trunk_fixed_joint_lump__camera_rearDown_collision_8'>
+        <pose>-0.082500000000000004 0.012500000000000001 -0.043650000000000001 3.1415926535897931 1.5707963267948966 0</pose>
+        <geometry>
+          <box>
+            <size>0.001 0.001 0.001</size>
+          </box>
+        </geometry>
+        <surface>
+          <contact>
+            <ode/>
+          </contact>
+          <friction>
+            <ode/>
+          </friction>
+        </surface>
+      </collision>
+      <collision name='trunk_fixed_joint_lump__camera_right_collision_9'>
+        <pose>-0.041000000000000002 -0.082000000000000003 -0.017600000000000001 3.1415926535897931 0.26179999999999998 -1.570796326794897</pose>
+        <geometry>
+          <box>
+            <size>0.001 0.001 0.001</size>
+          </box>
+        </geometry>
+        <surface>
+          <contact>
+            <ode/>
+          </contact>
+          <friction>
+            <ode/>
+          </friction>
+        </surface>
+      </collision>
+      <collision name='trunk_fixed_joint_lump__ultraSound_face_collision_10'>
+        <pose>0.2747 0 -0.0088000000000000005 0 0 0</pose>
+        <geometry>
+          <box>
+            <size>0.001 0.001 0.001</size>
+          </box>
+        </geometry>
+      </collision>
+      <collision name='trunk_fixed_joint_lump__ultraSound_left_collision_11'>
+        <pose>-0.053499999999999999 0.082600000000000007 0.0086800000000000002 0 0.26179999999999998 1.570796326794897</pose>
+        <geometry>
+          <box>
+            <size>0.001 0.001 0.001</size>
+          </box>
+        </geometry>
+      </collision>
+      <collision name='trunk_fixed_joint_lump__ultraSound_right_collision_12'>
+        <pose>-0.053499999999999999 -0.082600000000000007 0.0086800000000000002 0 0.26179999999999998 -1.570796326794897</pose>
+        <geometry>
+          <box>
+            <size>0.001 0.001 0.001</size>
+          </box>
+        </geometry>
+      </collision>
       <visual name='trunk_visual'>
         <pose>0 0 0 0 0 0</pose>
@@ -80,5 +184,5 @@
           <mesh>
             <scale>1 1 1</scale>
-            <uri>model://go1/meshes/trunk.dae</uri>
+            <uri>model://go1/dae/trunk.dae</uri>
           </mesh>
         </geometry>
@@ -140,4 +244,188 @@
         </material>
       </visual>
+      <visual name='trunk_fixed_joint_lump__camera_chin_visual_5'>
+        <pose>0.25219999999999998 0.012500000000000001 -0.0436 3.1415926535897931 1.5707963267948966 0</pose>
+        <geometry>
+          <mesh>
+            <scale>1 1 1</scale>
+            <uri>model://go1/dae/depthCamera.dae</uri>
+          </mesh>
+        </geometry>
+        <material>
+          <diffuse>0.05 0.05 0.05 1</diffuse>
+          <ambient>0.05 0.05 0.05 1</ambient>
+        </material>
+      </visual>
+      <visual name='trunk_fixed_joint_lump__camera_face_visual_6'>
+        <pose>0.27850000000000003 0.012500000000000001 0.0167 3.1415926535897931 0 0</pose>
+        <geometry>
+          <mesh>
+            <scale>1 1 1</scale>
+            <uri>model://go1/dae/depthCamera.dae</uri>
+          </mesh>
+        </geometry>
+        <material>
+          <diffuse>0.05 0.05 0.05 1</diffuse>
+          <ambient>0.05 0.05 0.05 1</ambient>
+        </material>
+      </visual>
+      <visual name='trunk_fixed_joint_lump__camera_left_visual_7'>
+        <pose>-0.066000000000000003 0.082000000000000003 -0.017600000000000001 3.1415926535897931 0.26179999999999998 1.5707963267948957</pose>
+        <geometry>
+          <mesh>
+            <scale>1 1 1</scale>
+            <uri>model://go1/dae/depthCamera.dae</uri>
+          </mesh>
+        </geometry>
+        <material>
+          <diffuse>0.05 0.05 0.05 1</diffuse>
+          <ambient>0.05 0.05 0.05 1</ambient>
+        </material>
+      </visual>
+      <visual name='trunk_fixed_joint_lump__camera_rearDown_visual_8'>
+        <pose>-0.082500000000000004 0.012500000000000001 -0.043650000000000001 3.1415926535897931 1.5707963267948966 0</pose>
+        <geometry>
+          <mesh>
+            <scale>1 1 1</scale>
+            <uri>model://go1/dae/depthCamera.dae</uri>
+          </mesh>
+        </geometry>
+        <material>
+          <diffuse>0.05 0.05 0.05 1</diffuse>
+          <ambient>0.05 0.05 0.05 1</ambient>
+        </material>
+      </visual>
+      <visual name='trunk_fixed_joint_lump__camera_right_visual_9'>
+        <pose>-0.041000000000000002 -0.082000000000000003 -0.017600000000000001 3.1415926535897931 0.26179999999999998 -1.570796326794897</pose>
+        <geometry>
+          <mesh>
+            <scale>1 1 1</scale>
+            <uri>model://go1/dae/depthCamera.dae</uri>
+          </mesh>
+        </geometry>
+        <material>
+          <diffuse>0.05 0.05 0.05 1</diffuse>
+          <ambient>0.05 0.05 0.05 1</ambient>
+        </material>
+      </visual>
+      <visual name='trunk_fixed_joint_lump__ultraSound_face_visual_10'>
+        <pose>0.2747 0 -0.0088000000000000005 0 0 0</pose>
+        <geometry>
+          <mesh>
+            <scale>1 1 1</scale>
+            <uri>model://go1/dae/ultraSound.dae</uri>
+          </mesh>
+        </geometry>
+        <material>
+          <diffuse>0 0 0 1</diffuse>
+          <ambient>0 0 0 1</ambient>
+        </material>
+      </visual>
+      <visual name='trunk_fixed_joint_lump__ultraSound_left_visual_11'>
+        <pose>-0.053499999999999999 0.082600000000000007 0.0086800000000000002 0 0.26179999999999998 1.570796326794897</pose>
+        <geometry>
+          <mesh>
+            <scale>1 1 1</scale>
+            <uri>model://go1/dae/ultraSound.dae</uri>
+          </mesh>
+        </geometry>
+        <material>
+          <diffuse>0 0 0 1</diffuse>
+          <ambient>0 0 0 1</ambient>
+        </material>
+      </visual>
+      <visual name='trunk_fixed_joint_lump__ultraSound_right_visual_12'>
+        <pose>-0.053499999999999999 -0.082600000000000007 0.0086800000000000002 0 0.26179999999999998 -1.570796326794897</pose>
+        <geometry>
+          <mesh>
+            <scale>1 1 1</scale>
+            <uri>model://go1/dae/ultraSound.dae</uri>
+          </mesh>
+        </geometry>
+        <material>
+          <diffuse>0 0 0 1</diffuse>
+          <ambient>0 0 0 1</ambient>
+        </material>
+      </visual>
+      <sensor name='camera_chin_camera' type='depth'>
+        <update_rate>16</update_rate>
+        <camera>
+          <horizontal_fov>2.0939999999999999</horizontal_fov>
+          <image>
+            <width>928</width>
+            <height>800</height>
+            <format>R8G8B8</format>
+          </image>
+          <clip>
+            <near>0.10000000000000001</near>
+            <far>5</far>
+          </clip>
+        </camera>
+        <pose>0.25219999999999998 0.012500000000000001 -0.0436 3.1415926535897931 1.5707926536359933 2.6535897933410511e-06</pose>
+      </sensor>
+      <sensor name='camera_face_camera' type='depth'>
+        <update_rate>16</update_rate>
+        <camera>
+          <horizontal_fov>2.0939999999999999</horizontal_fov>
+          <image>
+            <width>928</width>
+            <height>800</height>
+            <format>R8G8B8</format>
+          </image>
+          <clip>
+            <near>0.10000000000000001</near>
+            <far>5</far>
+          </clip>
+        </camera>
+        <pose>0.27850000000000003 0.012500000000000001 0.0167 3.1415899999999999 0 0</pose>
+      </sensor>
+      <sensor name='camera_left_camera' type='depth'>
+        <update_rate>16</update_rate>
+        <camera>
+          <horizontal_fov>2.0939999999999999</horizontal_fov>
+          <image>
+            <width>928</width>
+            <height>800</height>
+            <format>R8G8B8</format>
+          </image>
+          <clip>
+            <near>0.10000000000000001</near>
+            <far>5</far>
+          </clip>
+        </camera>
+        <pose>-0.066000000000000003 0.082000000000000003 -0.017600000000000001 3.1415899999999999 0.26180000000000009 1.5708</pose>
+      </sensor>
+      <sensor name='camera_rearDown_camera' type='depth'>
+        <update_rate>16</update_rate>
+        <camera>
+          <horizontal_fov>2.0939999999999999</horizontal_fov>
+          <image>
+            <width>928</width>
+            <height>800</height>
+            <format>R8G8B8</format>
+          </image>
+          <clip>
+            <near>0.10000000000000001</near>
+            <far>5</far>
+          </clip>
+        </camera>
+        <pose>-0.082500000000000004 0.012500000000000001 -0.043650000000000001 3.1415926535897931 1.5707926536359933 2.6535897933410511e-06</pose>
+      </sensor>
+      <sensor name='camera_right_camera' type='depth'>
+        <update_rate>16</update_rate>
+        <camera>
+          <horizontal_fov>2.0939999999999999</horizontal_fov>
+          <image>
+            <width>928</width>
+            <height>800</height>
+            <format>R8G8B8</format>
+          </image>
+          <clip>
+            <near>0.10000000000000001</near>
+            <far>5</far>
+          </clip>
+        </camera>
+        <pose>-0.041000000000000002 -0.082000000000000003 -0.017600000000000001 3.1415899999999999 0.26179999999999998 -1.5707999999999998</pose>
+      </sensor>
     </link>
     <joint name='FL_hip_joint' type='revolute'>
@@ -209,5 +497,5 @@
           <mesh>
             <scale>1 1 1</scale>
-            <uri>model://go1/meshes/hip.dae</uri>
+            <uri>model://go1/dae/hip.dae</uri>
           </mesh>
         </geometry>
@@ -301,5 +589,5 @@
           <mesh>
             <scale>1 1 1</scale>
-            <uri>model://go1/meshes/thigh.dae</uri>
+            <uri>model://go1/dae/thigh.dae</uri>
           </mesh>
         </geometry>
@@ -382,5 +670,5 @@
           <mesh>
             <scale>1 1 1</scale>
-            <uri>model://go1/meshes/calf.dae</uri>
+            <uri>model://go1/dae/calf.dae</uri>
           </mesh>
         </geometry>
@@ -541,5 +829,5 @@
           <mesh>
             <scale>1 1 1</scale>
-            <uri>model://go1/meshes/hip.dae</uri>
+            <uri>model://go1/dae/hip.dae</uri>
           </mesh>
         </geometry>
@@ -633,5 +921,5 @@
           <mesh>
             <scale>1 1 1</scale>
-            <uri>model://go1/meshes/thigh_mirror.dae</uri>
+            <uri>model://go1/dae/thigh_mirror.dae</uri>
           </mesh>
         </geometry>
@@ -714,5 +1002,5 @@
           <mesh>
             <scale>1 1 1</scale>
-            <uri>model://go1/meshes/calf.dae</uri>
+            <uri>model://go1/dae/calf.dae</uri>
           </mesh>
         </geometry>
@@ -873,5 +1161,5 @@
           <mesh>
             <scale>1 1 1</scale>
-            <uri>model://go1/meshes/hip.dae</uri>
+            <uri>model://go1/dae/hip.dae</uri>
           </mesh>
         </geometry>
@@ -965,5 +1253,5 @@
           <mesh>
             <scale>1 1 1</scale>
-            <uri>model://go1/meshes/thigh.dae</uri>
+            <uri>model://go1/dae/thigh.dae</uri>
           </mesh>
         </geometry>
@@ -1046,5 +1334,5 @@
           <mesh>
             <scale>1 1 1</scale>
-            <uri>model://go1/meshes/calf.dae</uri>
+            <uri>model://go1/dae/calf.dae</uri>
           </mesh>
         </geometry>
@@ -1205,5 +1493,5 @@
           <mesh>
             <scale>1 1 1</scale>
-            <uri>model://go1/meshes/hip.dae</uri>
+            <uri>model://go1/dae/hip.dae</uri>
           </mesh>
         </geometry>
@@ -1297,5 +1585,5 @@
           <mesh>
             <scale>1 1 1</scale>
-            <uri>model://go1/meshes/thigh_mirror.dae</uri>
+            <uri>model://go1/dae/thigh_mirror.dae</uri>
           </mesh>
         </geometry>
@@ -1378,10 +1666,10 @@
           <mesh>
             <scale>1 1 1</scale>
-            <uri>model://go1/meshes/calf.dae</uri>
-          </mesh>
-        </geometry>
-        <material>
-          <diffuse>1.0 0.4235294117647059 0.0392156862745098 1</diffuse>
-          <ambient>1.0 0.4235294117647059 0.0392156862745098 1</ambient>
+            <uri>model://go1/dae/calf.dae</uri>
+          </mesh>
+        </geometry>
+        <material>
+          <diffuse>0.2 0.2 0.2 1</diffuse>
+          <ambient>0.2 0.2 0.2 1</ambient>
         </material>
       </visual>
@@ -1463,6 +1751,6 @@
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