Commit message: Go1 added, All robot works with latest yaml convention update, Aesthetics upgrade on all robots

File: quad_simulator/go1_description/models/go1/urdf/go1.urdf.xacro (robot description, xacro)
@@ -49,9 +49,7 @@
       <origin rpy="0 0 0" xyz="0 0 0"/>
       <geometry>
-        <mesh filename="package://go1_description/models/go1/meshes/trunk.dae" scale="1 1 1"/>
-      </geometry>
-      <material name="">
-        <color rgba="1.0 0.4235294117647059 0.0392156862745098 1.0"/>
-      </material>
+        <mesh filename="package://go1_description/models/go1/dae/trunk.dae" scale="1 1 1"/>
+      </geometry>
+      <!-- <material name="orange"/> -->
     </visual>
     <collision>
@@ -109,9 +107,7 @@
       <origin rpy="3.141592653589793 0 0" xyz="0 0 0"/>
       <geometry>
-        <mesh filename="package://go1_description/models/go1/meshes/hip.dae" scale="1 1 1"/>
-      </geometry>
-      <material name="">
-        <color rgba="1.0 0.4235294117647059 0.0392156862745098 1.0"/>
-      </material>
+        <mesh filename="package://go1_description/models/go1/dae/hip.dae" scale="1 1 1"/>
+      </geometry>
+      <!-- <material name="orange"/> -->
     </visual>
     <collision>
@@ -133,7 +129,5 @@
         <cylinder length="0.02" radius="0.035"/>
       </geometry>
-      <material name="">
-        <color rgba="0.0 0.8 0.0 1.0"/>
-      </material>
+      <material name="green"/>
     </visual>
     <collision>
@@ -166,9 +160,7 @@
       <origin rpy="0 0 0" xyz="0 0 0"/>
       <geometry>
-        <mesh filename="package://go1_description/models/go1/meshes/thigh_mirror.dae" scale="1 1 1"/>
-      </geometry>
-      <material name="">
-        <color rgba="1.0 0.4235294117647059 0.0392156862745098 1.0"/>
-      </material>
+        <mesh filename="package://go1_description/models/go1/dae/thigh_mirror.dae" scale="1 1 1"/>
+      </geometry>
+      <!-- <material name="orange"/> -->
     </visual>
     <collision>
@@ -190,7 +182,5 @@
         <cylinder length="0.02" radius="0.035"/>
       </geometry>
-      <material name="">
-        <color rgba="0.0 0.8 0.0 1.0"/>
-      </material>
+      <material name="green"/>
     </visual>
     <collision>
@@ -223,9 +213,7 @@
       <origin rpy="0 0 0" xyz="0 0 0"/>
       <geometry>
-        <mesh filename="package://go1_description/models/go1/meshes/calf.dae" scale="1 1 1"/>
-      </geometry>
-      <material name="">
-        <color rgba="1.0 0.4235294117647059 0.0392156862745098 1.0"/>
-      </material>
+        <mesh filename="package://go1_description/models/go1/dae/calf.dae" scale="1 1 1"/>
+      </geometry>
+      <!-- <material name="orange"/> -->
     </visual>
     <collision>
@@ -247,7 +235,5 @@
         <cylinder length="0.02" radius="0.035"/>
       </geometry>
-      <material name="">
-        <color rgba="0.0 0.8 0.0 1.0"/>
-      </material>
+      <material name="green"/>
     </visual>
     <collision>
@@ -274,7 +260,5 @@
         <sphere radius="0.01"/>
       </geometry>
-      <material name="">
-        <color rgba="1.0 0.4235294117647059 0.0392156862745098 1.0"/>
-      </material>
+      <!-- <material name="orange"/> -->
     </visual>
     <collision>
@@ -289,4 +273,34 @@
     </inertial>
   </link>
+  <transmission name="FR_hip_tran">
+    <type>transmission_interface/SimpleTransmission</type>
+    <joint name="FR_hip_joint">
+      <hardwareInterface>hardware_interface/EffortJointInterface</hardwareInterface>
+    </joint>
+    <actuator name="FR_hip_motor">
+      <hardwareInterface>hardware_interface/EffortJointInterface</hardwareInterface>
+      <mechanicalReduction>1</mechanicalReduction>
+    </actuator>
+  </transmission>
+  <transmission name="FR_thigh_tran">
+    <type>transmission_interface/SimpleTransmission</type>
+    <joint name="FR_thigh_joint">
+      <hardwareInterface>hardware_interface/EffortJointInterface</hardwareInterface>
+    </joint>
+    <actuator name="FR_thigh_motor">
+      <hardwareInterface>hardware_interface/EffortJointInterface</hardwareInterface>
+      <mechanicalReduction>1</mechanicalReduction>
+    </actuator>
+  </transmission>
+  <transmission name="FR_calf_tran">
+    <type>transmission_interface/SimpleTransmission</type>
+    <joint name="FR_calf_joint">
+      <hardwareInterface>hardware_interface/EffortJointInterface</hardwareInterface>
+    </joint>
+    <actuator name="FR_calf_motor">
+      <hardwareInterface>hardware_interface/EffortJointInterface</hardwareInterface>
+      <mechanicalReduction>1</mechanicalReduction>
+    </actuator>
+  </transmission>
   <joint name="FL_hip_joint" type="revolute">
     <origin rpy="0 0 0" xyz="0.1881 0.04675 0"/>
@@ -306,9 +320,7 @@
       <origin rpy="0 0 0" xyz="0 0 0"/>
       <geometry>
-        <mesh filename="package://go1_description/models/go1/meshes/hip.dae" scale="1 1 1"/>
-      </geometry>
-      <material name="">
-        <color rgba="1.0 0.4235294117647059 0.0392156862745098 1.0"/>
-      </material>
+        <mesh filename="package://go1_description/models/go1/dae/hip.dae" scale="1 1 1"/>
+      </geometry>
+      <!-- <material name="orange"/> -->
     </visual>
     <collision>
@@ -330,7 +342,5 @@
         <cylinder length="0.02" radius="0.035"/>
       </geometry>
-      <material name="">
-        <color rgba="0.0 0.8 0.0 1.0"/>
-      </material>
+      <material name="green"/>
     </visual>
     <collision>
@@ -363,9 +373,7 @@
       <origin rpy="0 0 0" xyz="0 0 0"/>
       <geometry>
-        <mesh filename="package://go1_description/models/go1/meshes/thigh.dae" scale="1 1 1"/>
-      </geometry>
-      <material name="">
-        <color rgba="1.0 0.4235294117647059 0.0392156862745098 1.0"/>
-      </material>
+        <mesh filename="package://go1_description/models/go1/dae/thigh.dae" scale="1 1 1"/>
+      </geometry>
+      <!-- <material name="orange"/> -->
     </visual>
     <collision>
@@ -387,7 +395,5 @@
         <cylinder length="0.02" radius="0.035"/>
       </geometry>
-      <material name="">
-        <color rgba="0.0 0.8 0.0 1.0"/>
-      </material>
+      <material name="green"/>
     </visual>
     <collision>
@@ -420,9 +426,7 @@
       <origin rpy="0 0 0" xyz="0 0 0"/>
       <geometry>
-        <mesh filename="package://go1_description/models/go1/meshes/calf.dae" scale="1 1 1"/>
-      </geometry>
-      <material name="">
-        <color rgba="1.0 0.4235294117647059 0.0392156862745098 1.0"/>
-      </material>
+        <mesh filename="package://go1_description/models/go1/dae/calf.dae" scale="1 1 1"/>
+      </geometry>
+      <!-- <material name="orange"/> -->
     </visual>
     <collision>
@@ -444,7 +448,5 @@
         <cylinder length="0.02" radius="0.035"/>
       </geometry>
-      <material name="">
-        <color rgba="0.0 0.8 0.0 1.0"/>
-      </material>
+      <material name="green"/>
     </visual>
     <collision>
@@ -471,7 +473,5 @@
         <sphere radius="0.01"/>
       </geometry>
-      <material name="">
-        <color rgba="1.0 0.4235294117647059 0.0392156862745098 1.0"/>
-      </material>
+      <!-- <material name="orange"/> -->
     </visual>
     <collision>
@@ -486,4 +486,34 @@
     </inertial>
   </link>
+  <transmission name="FL_hip_tran">
+    <type>transmission_interface/SimpleTransmission</type>
+    <joint name="FL_hip_joint">
+      <hardwareInterface>hardware_interface/EffortJointInterface</hardwareInterface>
+    </joint>
+    <actuator name="FL_hip_motor">
+      <hardwareInterface>hardware_interface/EffortJointInterface</hardwareInterface>
+      <mechanicalReduction>1</mechanicalReduction>
+    </actuator>
+  </transmission>
+  <transmission name="FL_thigh_tran">
+    <type>transmission_interface/SimpleTransmission</type>
+    <joint name="FL_thigh_joint">
+      <hardwareInterface>hardware_interface/EffortJointInterface</hardwareInterface>
+    </joint>
+    <actuator name="FL_thigh_motor">
+      <hardwareInterface>hardware_interface/EffortJointInterface</hardwareInterface>
+      <mechanicalReduction>1</mechanicalReduction>
+    </actuator>
+  </transmission>
+  <transmission name="FL_calf_tran">
+    <type>transmission_interface/SimpleTransmission</type>
+    <joint name="FL_calf_joint">
+      <hardwareInterface>hardware_interface/EffortJointInterface</hardwareInterface>
+    </joint>
+    <actuator name="FL_calf_motor">
+      <hardwareInterface>hardware_interface/EffortJointInterface</hardwareInterface>
+      <mechanicalReduction>1</mechanicalReduction>
+    </actuator>
+  </transmission>
   <joint name="RR_hip_joint" type="revolute">
     <origin rpy="0 0 0" xyz="-0.1881 -0.04675 0"/>
@@ -503,9 +533,7 @@
       <origin rpy="3.141592653589793 3.141592653589793 0" xyz="0 0 0"/>
       <geometry>
-        <mesh filename="package://go1_description/models/go1/meshes/hip.dae" scale="1 1 1"/>
-      </geometry>
-      <material name="">
-        <color rgba="1.0 0.4235294117647059 0.0392156862745098 1.0"/>
-      </material>
+        <mesh filename="package://go1_description/models/go1/dae/hip.dae" scale="1 1 1"/>
+      </geometry>
+      <!-- <material name="orange"/> -->
     </visual>
     <collision>
@@ -527,7 +555,5 @@
         <cylinder length="0.02" radius="0.035"/>
       </geometry>
-      <material name="">
-        <color rgba="0.0 0.8 0.0 1.0"/>
-      </material>
+      <material name="green"/>
     </visual>
     <collision>
@@ -560,9 +586,7 @@
       <origin rpy="0 0 0" xyz="0 0 0"/>
       <geometry>
-        <mesh filename="package://go1_description/models/go1/meshes/thigh_mirror.dae" scale="1 1 1"/>
-      </geometry>
-      <material name="">
-        <color rgba="1.0 0.4235294117647059 0.0392156862745098 1.0"/>
-      </material>
+        <mesh filename="package://go1_description/models/go1/dae/thigh_mirror.dae" scale="1 1 1"/>
+      </geometry>
+      <!-- <material name="orange"/> -->
     </visual>
     <collision>
@@ -584,7 +608,5 @@
         <cylinder length="0.02" radius="0.035"/>
       </geometry>
-      <material name="">
-        <color rgba="0.0 0.8 0.0 1.0"/>
-      </material>
+      <material name="green"/>
     </visual>
     <collision>
@@ -617,9 +639,7 @@
       <origin rpy="0 0 0" xyz="0 0 0"/>
       <geometry>
-        <mesh filename="package://go1_description/models/go1/meshes/calf.dae" scale="1 1 1"/>
-      </geometry>
-      <material name="">
-        <color rgba="1.0 0.4235294117647059 0.0392156862745098 1.0"/>
-      </material>
+        <mesh filename="package://go1_description/models/go1/dae/calf.dae" scale="1 1 1"/>
+      </geometry>
+      <!-- <material name="orange"/> -->
     </visual>
     <collision>
@@ -641,7 +661,5 @@
         <cylinder length="0.02" radius="0.035"/>
       </geometry>
-      <material name="">
-        <color rgba="0.0 0.8 0.0 1.0"/>
-      </material>
+      <material name="green"/>
     </visual>
     <collision>
@@ -668,7 +686,5 @@
         <sphere radius="0.01"/>
       </geometry>
-      <material name="">
-        <color rgba="1.0 0.4235294117647059 0.0392156862745098 1.0"/>
-      </material>
+      <!-- <material name="orange"/> -->
     </visual>
     <collision>
@@ -683,4 +699,34 @@
     </inertial>
   </link>
+  <transmission name="RR_hip_tran">
+    <type>transmission_interface/SimpleTransmission</type>
+    <joint name="RR_hip_joint">
+      <hardwareInterface>hardware_interface/EffortJointInterface</hardwareInterface>
+    </joint>
+    <actuator name="RR_hip_motor">
+      <hardwareInterface>hardware_interface/EffortJointInterface</hardwareInterface>
+      <mechanicalReduction>1</mechanicalReduction>
+    </actuator>
+  </transmission>
+  <transmission name="RR_thigh_tran">
+    <type>transmission_interface/SimpleTransmission</type>
+    <joint name="RR_thigh_joint">
+      <hardwareInterface>hardware_interface/EffortJointInterface</hardwareInterface>
+    </joint>
+    <actuator name="RR_thigh_motor">
+      <hardwareInterface>hardware_interface/EffortJointInterface</hardwareInterface>
+      <mechanicalReduction>1</mechanicalReduction>
+    </actuator>
+  </transmission>
+  <transmission name="RR_calf_tran">
+    <type>transmission_interface/SimpleTransmission</type>
+    <joint name="RR_calf_joint">
+      <hardwareInterface>hardware_interface/EffortJointInterface</hardwareInterface>
+    </joint>
+    <actuator name="RR_calf_motor">
+      <hardwareInterface>hardware_interface/EffortJointInterface</hardwareInterface>
+      <mechanicalReduction>1</mechanicalReduction>
+    </actuator>
+  </transmission>
   <joint name="RL_hip_joint" type="revolute">
     <origin rpy="0 0 0" xyz="-0.1881 0.04675 0"/>
@@ -700,9 +746,7 @@
       <origin rpy="0 3.141592653589793 0" xyz="0 0 0"/>
       <geometry>
-        <mesh filename="package://go1_description/models/go1/meshes/hip.dae" scale="1 1 1"/>
-      </geometry>
-      <material name="">
-        <color rgba="1.0 0.4235294117647059 0.0392156862745098 1.0"/>
-      </material>
+        <mesh filename="package://go1_description/models/go1/dae/hip.dae" scale="1 1 1"/>
+      </geometry>
+      <!-- <material name="orange"/> -->
     </visual>
     <collision>
@@ -724,7 +768,5 @@
         <cylinder length="0.02" radius="0.035"/>
       </geometry>
-      <material name="">
-        <color rgba="0.0 0.8 0.0 1.0"/>
-      </material>
+      <material name="green"/>
     </visual>
     <collision>
@@ -757,9 +799,7 @@
       <origin rpy="0 0 0" xyz="0 0 0"/>
       <geometry>
-        <mesh filename="package://go1_description/models/go1/meshes/thigh.dae" scale="1 1 1"/>
-      </geometry>
-      <material name="">
-        <color rgba="1.0 0.4235294117647059 0.0392156862745098 1.0"/>
-      </material>
+        <mesh filename="package://go1_description/models/go1/dae/thigh.dae" scale="1 1 1"/>
+      </geometry>
+      <!-- <material name="orange"/> -->
     </visual>
     <collision>
@@ -781,7 +821,5 @@
         <cylinder length="0.02" radius="0.035"/>
       </geometry>
-      <material name="">
-        <color rgba="0.0 0.8 0.0 1.0"/>
-      </material>
+      <material name="green"/>
     </visual>
     <collision>
@@ -814,9 +852,7 @@
       <origin rpy="0 0 0" xyz="0 0 0"/>
       <geometry>
-        <mesh filename="package://go1_description/models/go1/meshes/calf.dae" scale="1 1 1"/>
-      </geometry>
-      <material name="">
-        <color rgba="1.0 0.4235294117647059 0.0392156862745098 1.0"/>
-      </material>
+        <mesh filename="package://go1_description/models/go1/dae/calf.dae" scale="1 1 1"/>
+      </geometry>
+      <!-- <material name="orange"/> -->
     </visual>
     <collision>
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
File: quad_simulator/go2_description/models/go2/go2.sdf.xacro (robot description, xacro)
@@ -1391,4 +1391,13 @@
     <joint name="imu_joint" type="fixed">
       <child>imu::link</child>
+      <parent>body</parent>
+    </joint>
+    <include>
+      <uri>model://cmu_text</uri>
+      <name>cmu_text</name>
+      <pose>0 0 0 0 0 0</pose>
+    </include>
+    <joint name="cmu_text_joint" type="fixed">
+      <child>cmu_text::text</child>
       <parent>body</parent>
     </joint>

File: quad_simulator/go2_description/models/go2/urdf/go2.urdf.xacro (robot description, xacro)
@@ -1437,3 +1437,20 @@
     </joint>
   </ros2_control>
+  <link name="cmu_text">
+    <visual>
+      <origin xyz="0 0 0" rpy="0 0 0" />
+      <geometry>
+        <mesh filename="package://objects_description/models/cmu_text/meshes/Spirit40_CMU_Text_transformed.stl" scale="1.3 1 1.3" />
+      </geometry>
+    </visual>
+    <inertial>
+      <mass value="0.0001" />
+      <inertia ixx="1e-08" ixy="0" ixz="0" iyy="1e-08" iyz="0" izz="1e-08" />
+    </inertial>
+  </link>
+  <joint name="cmu_text_joint" type="fixed">
+    <parent link="body" />
+    <child link="cmu_text" />
+    <origin xyz="0 0 -0.005" rpy="0 0 0" />
+  </joint>
 </robot>

File: quad_simulator/go2w_description/models/go2w/go2w.sdf.xacro (robot description, xacro)
@@ -1195,4 +1195,13 @@
     <joint name="imu_joint" type="fixed">
       <child>imu::link</child>
+      <parent>body</parent>
+    </joint>
+    <include>
+      <uri>model://cmu_text</uri>
+      <name>cmu_text</name>
+      <pose>0 0 0 0 0 0</pose>
+    </include>
+    <joint name="cmu_text_joint" type="fixed">
+      <child>cmu_text::text</child>
       <parent>body</parent>
     </joint>

File: quad_simulator/go2w_description/models/go2w/urdf/go2w.urdf.xacro (robot description, xacro)
@@ -1439,3 +1439,20 @@
     </joint>
   </ros2_control>
+  <link name="cmu_text">
+    <visual>
+      <origin xyz="0 0 0" rpy="0 0 0" />
+      <geometry>
+        <mesh filename="package://objects_description/models/cmu_text/meshes/Spirit40_CMU_Text_transformed.stl" scale="1.3 1 1.3" />
+      </geometry>
+    </visual>
+    <inertial>
+      <mass value="0.0001" />
+      <inertia ixx="1e-08" ixy="0" ixz="0" iyy="1e-08" iyz="0" izz="1e-08" />
+    </inertial>
+  </link>
+  <joint name="cmu_text_joint" type="fixed">
+    <parent link="body" />
+    <child link="cmu_text" />
+    <origin xyz="0 0 -0.005" rpy="0 0 0" />
+  </joint>
 </robot>

File: quad_simulator/spot_description/models/spot/spot.sdf.xacro (robot description, xacro)
@@ -1259,4 +1259,13 @@
     <joint name="imu_joint" type="fixed">
       <child>imu::link</child>
+      <parent>body</parent>
+    </joint>
+    <include>
+      <uri>model://cmu_text</uri>
+      <name>cmu_text</name>
+      <pose>0 0 0 0 0 0</pose>
+    </include>
+    <joint name="cmu_text_joint" type="fixed">
+      <child>cmu_text::text</child>
       <parent>body</parent>
     </joint>

File: quad_simulator/spot_description/models/spot/urdf/spot.urdf.xacro (robot description, xacro)
@@ -807,3 +807,20 @@
     </joint>
   </ros2_control>
+  <link name="cmu_text">
+    <visual>
+      <origin xyz="0 0 0" rpy="0 0 0" />
+      <geometry>
+        <mesh filename="package://objects_description/models/cmu_text/meshes/Spirit40_CMU_Text_transformed.stl" scale="1.3 1 1.3" />
+      </geometry>
+    </visual>
+    <inertial>
+      <mass value="0.0001" />
+      <inertia ixx="1e-08" ixy="0" ixz="0" iyy="1e-08" iyz="0" izz="1e-08" />
+    </inertial>
+  </link>
+  <joint name="cmu_text_joint" type="fixed">
+    <parent link="body" />
+    <child link="cmu_text" />
+    <origin xyz="0 0 -0.005" rpy="0 0 0" />
+  </joint>
 </robot>

File: quad_simulator/vision60_description/models/vision60/urdf/vision60.urdf.xacro (robot description, xacro)
@@ -941,3 +941,20 @@
     </joint>
   </ros2_control>
+  <link name="cmu_text">
+    <visual>
+      <origin xyz="0 0 0" rpy="0 0 0" />
+      <geometry>
+        <mesh filename="package://objects_description/models/cmu_text/meshes/Spirit40_CMU_Text_transformed.stl" scale="1.3 1 1.3" />
+      </geometry>
+    </visual>
+    <inertial>
+      <mass value="0.0001" />
+      <inertia ixx="1e-08" ixy="0" ixz="0" iyy="1e-08" iyz="0" izz="1e-08" />
+    </inertial>
+  </link>
+  <joint name="cmu_text_joint" type="fixed">
+    <parent link="body" />
+    <child link="cmu_text" />
+    <origin xyz="0 0 -0.005" rpy="0 0 0" />
+  </joint>
 </robot>

File: quad_simulator/vision60_description/models/vision60/vision60.sdf.xacro (robot description, xacro)
@@ -1182,4 +1182,13 @@
     <joint name="imu_joint" type="fixed">
       <child>imu::link</child>
+      <parent>body</parent>
+    </joint>
+    <include>
+      <uri>model://cmu_text</uri>
+      <name>cmu_text</name>
+      <pose>0 0 0 0 0 0</pose>
+    </include>
+    <joint name="cmu_text_joint" type="fixed">
+      <child>cmu_text::text</child>
       <parent>body</parent>
     </joint>
