Commit message: Base Go2-W Support in Sim, Hardware Interface, RD Integration

File: quad_simulator/go2w_description/models/go2w/go2w.sdf.xacro (robot description, xacro)
@@ -287,4 +287,18 @@
           </mesh>
         </geometry>
+        <surface>
+          <contact>
+            <ode>
+              <kp>1e+06</kp>
+              <kd>1</kd>
+            </ode>
+          </contact>
+          <friction>
+            <ode>
+              <mu>1.0</mu>
+              <mu2>1.0</mu2>
+            </ode>
+          </friction>
+        </surface>
       </collision>
       <visual name='toe0_visual'>
@@ -546,4 +560,18 @@
           </mesh>
         </geometry>
+        <surface>
+          <contact>
+            <ode>
+              <kp>1e+06</kp>
+              <kd>1</kd>
+            </ode>
+          </contact>
+          <friction>
+            <ode>
+              <mu>1.0</mu>
+              <mu2>1.0</mu2>
+            </ode>
+          </friction>
+        </surface>
       </collision>
       <visual name='toe2_visual'>
@@ -805,4 +833,18 @@
           </mesh>
         </geometry>
+        <surface>
+          <contact>
+            <ode>
+              <kp>1e+06</kp>
+              <kd>1</kd>
+            </ode>
+          </contact>
+          <friction>
+            <ode>
+              <mu>1.0</mu>
+              <mu2>1.0</mu2>
+            </ode>
+          </friction>
+        </surface>
       </collision>
       <visual name='toe1_visual'>
@@ -1064,4 +1106,18 @@
           </mesh>
         </geometry>
+        <surface>
+          <contact>
+            <ode>
+              <kp>1e+06</kp>
+              <kd>1</kd>
+            </ode>
+          </contact>
+          <friction>
+            <ode>
+              <mu>1.0</mu>
+              <mu2>1.0</mu2>
+            </ode>
+          </friction>
+        </surface>
       </collision>
       <visual name='toe3_visual'>
@@ -1207,15 +1263,24 @@
     </joint>
     <!-- Setup ros control -->
-      <plugin
-          filename="libgz_ros2_control-system.so"
-          name="gz_ros2_control::GazeboSimROS2ControlPlugin">
-          <controlPeriod>0.001</controlPeriod>
-          <parameters>${controller_config_path}</parameters>
-              <ros>
-                <namespace>${namespace}</namespace>
-            </ros>
-      </plugin>
-    <!-- Publish ground truth state data -->
-    <plugin filename="libground_truth_estimator.so" name="ground_truth_estimator">
+    <plugin
+        filename="libgz_ros2_control-system.so"
+        name="gz_ros2_control::GazeboSimROS2ControlPlugin">
+        <controlPeriod>0.001</controlPeriod>
+        <parameters>$(arg controller_config_path)</parameters>
+            <ros>
+              <namespace>$(arg namespace)</namespace>
+          </ros>
+    </plugin>
+    <!-- Pin the body at its spawn pose for hold_duration seconds so that
+         controllers can come up and fold the legs into sit pose without
+         the body tipping. Mirrors the spawn_lock used on the go2 model.
+         Wheels articulate freely the whole time. -->
+    <plugin filename="libspawn_lock.so" name="spawn_lock">
+        <body_link>body</body_link>
+        <hold_duration>8.0</hold_duration>
+    </plugin>
+    <!-- Publish ground truth state data (wheel-aware variant: 12 leg
+         joints + 4 wheel joints in RobotState.joints). -->
+    <plugin filename="libquad_wheel_ground_truth_estimator.so" name="quad_wheel_ground_truth_estimator">
       <updateRateHZ>500.0</updateRateHZ>
       <ground_truth_state_topic>state/ground_truth</ground_truth_state_topic>

File: quad_simulator/go2w_description/models/go2w/urdf/go2w.urdf.xacro (robot description, xacro)
@@ -1438,4 +1438,27 @@
       <state_interface name="position" />
     </joint>
+    <!-- Wheel joints (continuous, axis y). Driven in velocity mode by
+         the QuadWheelController via the same effort command interface
+         used for the leg motors. -->
+    <joint name="jtoe0">
+      <command_interface name="effort" />
+      <state_interface name="velocity" />
+      <state_interface name="position" />
+    </joint>
+    <joint name="jtoe1">
+      <command_interface name="effort" />
+      <state_interface name="velocity" />
+      <state_interface name="position" />
+    </joint>
+    <joint name="jtoe2">
+      <command_interface name="effort" />
+      <state_interface name="velocity" />
+      <state_interface name="position" />
+    </joint>
+    <joint name="jtoe3">
+      <command_interface name="effort" />
+      <state_interface name="velocity" />
+      <state_interface name="position" />
+    </joint>
   </ros2_control>
   <link name="cmu_text">
