Commit message: Found bug in mesh files, debugging in progress

File: quad_simulator/quad_sim_scripts/worlds/parkour_local_min.xml.xacro (robot description, xacro)
@@ -1,10 +1,14 @@
-<mujoco model="parkour_local_min">
+<?xml version="1.0" encoding="utf-8"?>
+<mujoco model="parkour_local_min" xmlns:xacro="http://www.ros.org/wiki/xacro">
+  <xacro:arg name="meshdir" default=""/>
+  <xacro:arg name="mjcf_path" default=""/>
+  <xacro:arg name="terrain_mesh" default=""/>
   <compiler
     angle="radian"
-    meshdir="/home/rml/ros2_ws/install/go2_description/share/go2_description/models/go2/go2_mjc/assets"
+    meshdir="$(arg meshdir)"
     autolimits="true"/>
-  <include file="/home/rml/ros2_ws/install/go2_description/share/go2_description/models/go2/go2_mjc/go2.xml"/>
+  <include file="$(arg mjcf_path)"/>
   <asset>
-    <mesh name="terrain" file="/home/rml/ros2_ws/install/quad_sim_scripts/share/quad_sim_scripts/models/parkour_local_min/meshes/parkour_local_min.stl"/>
+    <mesh name="terrain" file="$(arg terrain_mesh)"/>
   </asset>
   <worldbody>

File: quad_simulator/quad_sim_scripts/worlds/step_25cm.xml.xacro (robot description, xacro)
@@ -1,14 +1,18 @@
-<mujoco model="step_25cm">
+<?xml version="1.0" encoding="utf-8"?>
+<mujoco model="step_25cm" xmlns:xacro="http://www.ros.org/wiki/xacro">
+  <xacro:arg name="meshdir" default=""/>
+  <xacro:arg name="mjcf_path" default=""/>
+  <xacro:arg name="terrain_mesh" default=""/>
   <compiler
     angle="radian"
-    meshdir="/home/rml/ros2_ws/install/go2_description/share/go2_description/models/go2/go2_mjc/assets"
+    meshdir="$(arg meshdir)"
     autolimits="true"/>
-  <include file="/home/rml/ros2_ws/install/go2_description/share/go2_description/models/go2/go2_mjc/go2.xml"/>
+  <include file="$(arg mjcf_path)"/>
   <asset>
-    <mesh name="terrain" file="/home/rml/ros2_ws/install/quad_sim_scripts/share/quad_sim_scripts/models/step_25cm/meshes/step_25cm.stl"/>
+    <mesh name="terrain" file="$(arg terrain_mesh)"/>
   </asset>
   <worldbody>
     <light directional="true" diffuse=".8 .8 .8" specular=".2 .2 .2" pos="0 0 5" dir="0 0 -1"/>
-    <geom name="floor" type="mesh" mesh="terrain" pos="-2 -2 -0.1" rgba="0.8 0.9 0.8 1"/>
+    <geom name="floor" type="mesh" mesh="terrain" pos="-2 -2 -0.25" rgba="0.8 0.9 0.8 1"/>
   </worldbody>
 </mujoco>
