Commit message: Tested and Documented Pinocchio Intergration, Added ROS2 Tests, Parameter Handling

File: quad_simulator/go2_description/models/go2/go2.sdf.xacro (robot description, xacro)
@@ -3,4 +3,5 @@
   <xacro:arg name="namespace" default="robot_1" />
   <xacro:arg name="controller_config_path" default="/path/quad_control.yaml" />
+  <xacro:arg name="robot_config_path" default="/path/go2.yaml" />
   <model name='go2'>
     <link name='body'>
@@ -112,12 +113,12 @@
     </link>
     <joint name='0' type='revolute'>
-      <pose relative_to='hip0'>0 0.095500000000000002 0 0 1.5708 0</pose>
+      <pose relative_to='hip0'>0 0.095500000000000002 0 0 0 0</pose>
       <parent>hip0</parent>
       <child>upper0</child>
       <axis>
-        <xyz>0 -1 0</xyz>
-        <limit>
-          <lower>-2.61799</lower>
-          <upper>2.61799</upper>
+        <xyz>0 1 0</xyz>
+        <limit>
+          <lower>-1.5708</lower>
+          <upper>3.4906999999999999</upper>
           <effort>23.699999999999999</effort>
           <velocity>30.100000000000001</velocity>
@@ -166,5 +167,5 @@
     </link>
     <joint name='1' type='revolute'>
-      <pose relative_to='upper0'>0 0 -0.21299999999999999 -3.14159 0 -3.14159</pose>
+      <pose relative_to='upper0'>0 0 -0.21299999999999999 0 0 0</pose>
       <parent>upper0</parent>
       <child>lower0</child>
@@ -172,6 +173,6 @@
         <xyz>0 1 0</xyz>
         <limit>
-          <lower>0.445059</lower>
-          <upper>2.22529</upper>
+          <lower>-2.7227000000000001</lower>
+          <upper>-0.83775999999999995</upper>
           <effort>45.43</effort>
           <velocity>15.699999999999999</velocity>
@@ -245,5 +246,5 @@
         </material>
       </visual>
-      <visual name='lower_fixed_joint_lump__FL_foot_visual_1'>
+      <visual name='lower0_fixed_joint_lump__FL_foot_visual_1'>
         <pose>0 0 -0.21299999999999999 0 0 0</pose>
         <geometry>
@@ -400,12 +401,12 @@
     </link>
     <joint name='4' type='revolute'>
-      <pose relative_to='hip2'>0 -0.095500000000000002 0 0 1.5708 0</pose>
+      <pose relative_to='hip2'>0 -0.095500000000000002 0 0 0 0</pose>
       <parent>hip2</parent>
       <child>upper2</child>
       <axis>
-        <xyz>0 -1 0</xyz>
-        <limit>
-          <lower>-2.61799</lower>
-          <upper>2.61799</upper>
+        <xyz>0 1 0</xyz>
+        <limit>
+          <lower>-1.5708</lower>
+          <upper>3.4906999999999999</upper>
           <effort>23.699999999999999</effort>
           <velocity>30.100000000000001</velocity>
@@ -454,5 +455,5 @@
     </link>
     <joint name='5' type='revolute'>
-      <pose relative_to='upper2'>0 0 -0.21299999999999999 -3.14159 0 -3.14159</pose>
+      <pose relative_to='upper2'>0 0 -0.21299999999999999 0 0 0</pose>
       <parent>upper2</parent>
       <child>lower2</child>
@@ -460,6 +461,6 @@
         <xyz>0 1 0</xyz>
         <limit>
-          <lower>0.445059</lower>
-          <upper>2.22529</upper>
+          <lower>-2.7227000000000001</lower>
+          <upper>-0.83775999999999995</upper>
           <effort>45.43</effort>
           <velocity>15.699999999999999</velocity>
@@ -689,12 +690,12 @@
     </link>
     <joint name='2' type='revolute'>
-      <pose relative_to='hip1'>0 0.095500000000000002 0 0 1.5708 0</pose>
+      <pose relative_to='hip1'>0 0.095500000000000002 0 0 0 0</pose>
       <parent>hip1</parent>
       <child>upper1</child>
       <axis>
-        <xyz>0 -1 0</xyz>
-        <limit>
-          <lower>-2.61799</lower>
-          <upper>2.61799</upper>
+        <xyz>0 1 0</xyz>
+        <limit>
+          <lower>-0.52359999999999995</lower>
+          <upper>4.5378999999999996</upper>
           <effort>23.699999999999999</effort>
           <velocity>30.100000000000001</velocity>
@@ -743,5 +744,5 @@
     </link>
     <joint name='3' type='revolute'>
-      <pose relative_to='upper1'>0 0 -0.21299999999999999 -3.14159 0 -3.14159</pose>
+      <pose relative_to='upper1'>0 0 -0.21299999999999999 0 0 0</pose>
       <parent>upper1</parent>
       <child>lower1</child>
@@ -749,6 +750,6 @@
         <xyz>0 1 0</xyz>
         <limit>
-          <lower>0.445059</lower>
-          <upper>2.22529</upper>
+          <lower>-2.7227000000000001</lower>
+          <upper>-0.83775999999999995</upper>
           <effort>45.43</effort>
           <velocity>15.699999999999999</velocity>
@@ -977,12 +978,12 @@
     </link>
     <joint name='6' type='revolute'>
-      <pose relative_to='hip3'>0 -0.095500000000000002 0 0 1.5708 0</pose>
+      <pose relative_to='hip3'>0 -0.095500000000000002 0 0 0 0</pose>
       <parent>hip3</parent>
       <child>upper3</child>
       <axis>
-        <xyz>0 -1 0</xyz>
-        <limit>
-          <lower>-2.61799</lower>
-          <upper>2.61799</upper>
+        <xyz>0 1 0</xyz>
+        <limit>
+          <lower>-0.52359999999999995</lower>
+          <upper>4.5378999999999996</upper>
           <effort>23.699999999999999</effort>
           <velocity>30.100000000000001</velocity>
@@ -1031,5 +1032,5 @@
     </link>
     <joint name='7' type='revolute'>
-      <pose relative_to='upper3'>0 0 -0.21299999999999999 -3.14159 0 -3.14159</pose>
+      <pose relative_to='upper3'>0 0 -0.21299999999999999 0 0 0</pose>
       <parent>upper3</parent>
       <child>lower3</child>
@@ -1037,6 +1038,6 @@
         <xyz>0 1 0</xyz>
         <limit>
-          <lower>0.445059</lower>
-          <upper>2.22529</upper>
+          <lower>-2.7227000000000001</lower>
+          <upper>-0.83775999999999995</upper>
           <effort>45.43</effort>
           <velocity>15.699999999999999</velocity>
@@ -1209,5 +1210,5 @@
       <self_collide>0</self_collide>
     </link>
-    <frame name='hip0_rotor_joint' attached_to='body'>
+     <frame name='hip0_rotor_joint' attached_to='body'>
       <pose>0.11215 0.04675 0 0 0 0</pose>
     </frame>
@@ -1394,13 +1395,13 @@
     </joint>
     <!-- Setup ros control -->
-      <plugin
-          filename="libgz_ros2_control-system.so"
-          name="gz_ros2_control::GazeboSimROS2ControlPlugin">
-          <controlPeriod>0.002</controlPeriod>
-          <parameters>$(arg controller_config_path)</parameters>
-              <ros>
-                <namespace>$(arg namespace)</namespace>
-            </ros>
-      </plugin>
+    <plugin
+        filename="libgz_ros2_control-system.so"
+        name="gz_ros2_control::GazeboSimROS2ControlPlugin">
+        <controlPeriod>0.002</controlPeriod>
+        <parameters>$(arg controller_config_path)</parameters>
+            <ros>
+              <namespace>$(arg namespace)</namespace>
+          </ros>
+    </plugin>
     <!-- Publish ground truth state data -->
     <plugin filename="libground_truth_estimator.so" name="ground_truth_estimator">
@@ -1408,4 +1409,5 @@
       <ground_truth_state_topic>state/ground_truth</ground_truth_state_topic>
       <ground_truth_body_frame_topic>state/ground_truth_body_frame</ground_truth_body_frame_topic>
+      <parameters>$(arg robot_config_path)</parameters>
       <ros>
         <parameter name="use_sim_time">true</parameter>

File: quad_simulator/go2_description/models/go2/urdf/go2.urdf.xacro (robot description, xacro)
@@ -227,5 +227,5 @@
     <origin
       xyz="0 0.0955 0"
-      rpy="0 1.57079632679 0" />
+      rpy="0 0 0" />
     <parent
       link="hip0" />
@@ -233,8 +233,8 @@
       link="upper0" />
     <axis
-      xyz="0 -1 0" />
+      xyz="0 1 0" />
     <limit
-      lower="-2.6179938779914944"
-      upper="2.6179938779914944"
+      lower="-1.5708"
+      upper="3.4907"
       effort="23.7"
       velocity="30.1" />
@@ -294,5 +294,5 @@
     <origin
       xyz="0 0 -0.213"
-      rpy="0 -3.14159265359 0" />
+      rpy="0 0 0" />
     <parent
       link="upper0" />
@@ -302,6 +302,6 @@
       xyz="0 1 0" />
     <limit
-      lower="0.445058959258554"
-      upper="2.2252947962927703"
+      lower="-2.7227"
+      upper="-0.83776"
       effort="45.43"
       velocity="15.70" />
@@ -522,5 +522,5 @@
     <origin
       xyz="0 -0.0955 0"
-      rpy="0 1.57079632679 0" />
+      rpy="0 0 0" />
     <parent
       link="hip2" />
@@ -528,8 +528,8 @@
       link="upper2" />
     <axis
-      xyz="0 -1 0" />
+      xyz="0 1 0" />
     <limit
-      lower="-2.6179938779914944"
-      upper="2.6179938779914944"
+      lower="-1.5708"
+      upper="3.4907"
       effort="23.7"
       velocity="30.1" />
@@ -589,5 +589,5 @@
     <origin
       xyz="0 0 -0.213"
-      rpy="0 -3.14159265359 0" />
+      rpy="0 0 0" />
     <parent
       link="upper2" />
@@ -597,6 +597,6 @@
       xyz="0 1 0" />
     <limit
-      lower="0.445058959258554"
-      upper="2.2252947962927703"
+      lower="-2.7227"
+      upper="-0.83776"
       effort="45.43"
       velocity="15.70" />
@@ -817,5 +817,5 @@
     <origin
       xyz="0 0.0955 0"
-      rpy="0 1.57079632679 0" />
+      rpy="0 0 0" />
     <parent
       link="hip1" />
@@ -823,8 +823,8 @@
       link="upper1" />
     <axis
-      xyz="0 -1 0" />
+      xyz="0 1 0" />
     <limit
-      lower="-2.6179938779914944"
-      upper="2.6179938779914944"
+      lower="-0.5236"
+      upper="4.5379"
       effort="23.7"
       velocity="30.1" />
@@ -884,5 +884,5 @@
     <origin
       xyz="0 0 -0.213"
-      rpy="0 -3.14159265359 0" />
+      rpy="0 0 0" />
     <parent
       link="upper1" />
@@ -892,6 +892,6 @@
       xyz="0 1 0" />
     <limit
-      lower="0.445058959258554"
-      upper="2.2252947962927703"
+      lower="-2.7227"
+      upper="-0.83776"
       effort="45.43"
       velocity="15.70" />
@@ -1112,5 +1112,5 @@
     <origin
       xyz="0 -0.0955 0"
-      rpy="0 1.57079632679 0" />
+      rpy="0 0 0" />
     <parent
       link="hip3" />
@@ -1118,8 +1118,8 @@
       link="upper3" />
     <axis
-      xyz="0 -1 0" />
+      xyz="0 1 0" />
     <limit
-      lower="-2.6179938779914944"
-      upper="2.6179938779914944"
+      lower="-0.5236"
+      upper="4.5379"
       effort="23.7"
       velocity="30.1" />
@@ -1179,5 +1179,5 @@
     <origin
       xyz="0 0 -0.213"
-      rpy="0 -3.14159265359 0" />
+      rpy="0 0 0" />
     <parent
       link="upper3" />
@@ -1187,6 +1187,6 @@
       xyz="0 1 0" />
     <limit
-      lower="0.445058959258554"
-      upper="2.2252947962927703"
+      lower="-2.7227"
+      upper="-0.83776"
       effort="45.43"
       velocity="15.70" />

File: quad_simulator/spirit_description/models/spirit/spirit.sdf.xacro (robot description, xacro)
@@ -3,4 +3,5 @@
   <xacro:arg name="namespace" default="robot_1" />
   <xacro:arg name="controller_config_path" default="/path/quad_control.yaml" />
+  <xacro:arg name="robot_config_path" default= "/path/spirit.yaml" />
   <model name='spirit'>
     <link name='body'>
@@ -1206,4 +1207,5 @@
       <ground_truth_state_topic>state/ground_truth</ground_truth_state_topic>
       <ground_truth_body_frame_topic>state/ground_truth_body_frame</ground_truth_body_frame_topic>
+      <parameters>$(arg robot_config_path)</parameters>
       <ros>
         <parameter name="use_sim_time">true</parameter>

Commit message: add learned go2 hardware support

File: quad_simulator/go2_description/models/go2/go2.sdf.xacro (robot description, xacro)
@@ -1403,13 +1403,4 @@
     <joint name="imu_joint" type="fixed">
       <child>imu::link</child>
-      <parent>body</parent>
-    </joint>
-    <include>
-      <uri>model://cmu_text</uri>
-      <name>cmu_text</name>
-      <pose>0 0 0 0 0 0</pose>
-    </include>
-    <joint name="cmu_text_joint" type="fixed">
-      <child>cmu_text::text</child>
       <parent>body</parent>
     </joint>

File: quad_simulator/go2_description/models/go2/urdf/go2.urdf.xacro (robot description, xacro)
@@ -1437,20 +1437,3 @@
     </joint>
   </ros2_control>
-  <link name="cmu_text">
-    <visual>
-      <origin xyz="0 0 0" rpy="0 0 0" />
-      <geometry>
-        <mesh filename="package://objects_description/models/cmu_text/meshes/Spirit40_CMU_Text_transformed.stl" scale="0.8 1 0.8" />
-      </geometry>
-    </visual>
-    <inertial>
-      <mass value="0.0001" />
-      <inertia ixx="1e-08" ixy="0" ixz="0" iyy="1e-08" iyz="0" izz="1e-08" />
-    </inertial>
-  </link>
-  <joint name="cmu_text_joint" type="fixed">
-    <parent link="body" />
-    <child link="cmu_text" />
-    <origin xyz="0 0 -0.005" rpy="0 0 0" />
-  </joint>
 </robot>

File: quad_simulator/go2_description/models/go2/urdf/go2_isaac_clean.urdf (robot description, URDF)
Before this commit: robot go2, 43 links, 42 joints
Links:
- removed link cmu_text
Joints:
- removed joint cmu_text_joint

File: quad_simulator/go2w_description/models/go2w/go2w.sdf.xacro (robot description, xacro)
@@ -1251,13 +1251,4 @@
     <joint name="imu_joint" type="fixed">
       <child>imu::link</child>
-      <parent>body</parent>
-    </joint>
-    <include>
-      <uri>model://cmu_text</uri>
-      <name>cmu_text</name>
-      <pose>0 0 0 0 0 0</pose>
-    </include>
-    <joint name="cmu_text_joint" type="fixed">
-      <child>cmu_text::text</child>
       <parent>body</parent>
     </joint>

File: quad_simulator/go2w_description/models/go2w/urdf/go2w.urdf.xacro (robot description, xacro)
@@ -1462,20 +1462,3 @@
     </joint>
   </ros2_control>
-  <link name="cmu_text">
-    <visual>
-      <origin xyz="0 0 0" rpy="0 0 0" />
-      <geometry>
-        <mesh filename="package://objects_description/models/cmu_text/meshes/Spirit40_CMU_Text_transformed.stl" scale="1.3 1 1.3" />
-      </geometry>
-    </visual>
-    <inertial>
-      <mass value="0.0001" />
-      <inertia ixx="1e-08" ixy="0" ixz="0" iyy="1e-08" iyz="0" izz="1e-08" />
-    </inertial>
-  </link>
-  <joint name="cmu_text_joint" type="fixed">
-    <parent link="body" />
-    <child link="cmu_text" />
-    <origin xyz="0 0 -0.005" rpy="0 0 0" />
-  </joint>
 </robot>
