Commit message: v115 gz deploy fixes: remove duplicate foot collisions (GRF was halved), zero SDF joint springs+damping, Go2HV envelope via yaml (launch no longer force-overrides), is_hardware gate for   clipped_effort, world-frame path follower w/ stance warmup
  Sim-only plant fixes + training-faithful actuation; hardware clipped_effort path unchanged (already applies Go2HV clip). Full record: underbrush docs/gazebo_v115_deploy_debug_ledger.md

File: quad_simulator/go2_description/models/go2/go2.sdf.xacro (robot description, xacro)
@@ -69,7 +69,7 @@
         </limit>
         <dynamics>
-          <damping>0.5</damping>
+          <damping>0</damping>
           <spring_reference>0</spring_reference>
-          <spring_stiffness>3</spring_stiffness>
+          <spring_stiffness>0</spring_stiffness>
         </dynamics>
       </axis>
@@ -125,7 +125,7 @@
         </limit>
         <dynamics>
-          <damping>0.5</damping>
+          <damping>0</damping>
           <spring_reference>1.36</spring_reference>
-          <spring_stiffness>3</spring_stiffness>
+          <spring_stiffness>0</spring_stiffness>
         </dynamics>
       </axis>
@@ -180,7 +180,7 @@
         </limit>
         <dynamics>
-          <damping>0.5</damping>
+          <damping>0</damping>
           <spring_reference>-2.65</spring_reference>
-          <spring_stiffness>3</spring_stiffness>
+          <spring_stiffness>0</spring_stiffness>
         </dynamics>
       </axis>
@@ -225,12 +225,4 @@
             <radius>0.0155</radius>
           </cylinder>
-        </geometry>
-      </collision>
-      <collision name='lower0_fixed_joint_lump__FL_foot_collision_3'>
-        <pose>-0.002 0 -0.21299999999999999 0 0 0</pose>
-        <geometry>
-          <sphere>
-            <radius>0.021999999999999999</radius>
-          </sphere>
         </geometry>
       </collision>
@@ -360,7 +352,7 @@
         </limit>
         <dynamics>
-          <damping>0.5</damping>
+          <damping>0</damping>
           <spring_reference>0</spring_reference>
-          <spring_stiffness>3</spring_stiffness>
+          <spring_stiffness>0</spring_stiffness>
         </dynamics>
       </axis>
@@ -416,7 +408,7 @@
         </limit>
         <dynamics>
-          <damping>0.5</damping>
+          <damping>0</damping>
           <spring_reference>1.36</spring_reference>
-          <spring_stiffness>3</spring_stiffness>
+          <spring_stiffness>0</spring_stiffness>
         </dynamics>
       </axis>
@@ -471,7 +463,7 @@
         </limit>
         <dynamics>
-          <damping>0.5</damping>
+          <damping>0</damping>
           <spring_reference>-2.65</spring_reference>
-          <spring_stiffness>3</spring_stiffness>
+          <spring_stiffness>0</spring_stiffness>
         </dynamics>
       </axis>
@@ -516,12 +508,4 @@
             <radius>0.0155</radius>
           </cylinder>
-        </geometry>
-      </collision>
-      <collision name='lower2_fixed_joint_lump__FR_foot_collision_3'>
-        <pose>-0.002 0 -0.21299999999999999 0 0 0</pose>
-        <geometry>
-          <sphere>
-            <radius>0.021999999999999999</radius>
-          </sphere>
         </geometry>
       </collision>
@@ -652,7 +636,7 @@
         </limit>
         <dynamics>
-          <damping>0.5</damping>
+          <damping>0</damping>
           <spring_reference>0</spring_reference>
-          <spring_stiffness>3</spring_stiffness>
+          <spring_stiffness>0</spring_stiffness>
         </dynamics>
       </axis>
@@ -708,7 +692,7 @@
         </limit>
         <dynamics>
-          <damping>0.5</damping>
+          <damping>0</damping>
           <spring_reference>1.36</spring_reference>
-          <spring_stiffness>3</spring_stiffness>
+          <spring_stiffness>0</spring_stiffness>
         </dynamics>
       </axis>
@@ -763,7 +747,7 @@
         </limit>
         <dynamics>
-          <damping>0.5</damping>
+          <damping>0</damping>
           <spring_reference>-2.65</spring_reference>
-          <spring_stiffness>3</spring_stiffness>
+          <spring_stiffness>0</spring_stiffness>
         </dynamics>
       </axis>
@@ -808,12 +792,4 @@
             <radius>0.0155</radius>
           </cylinder>
-        </geometry>
-      </collision>
-      <collision name='lower1_fixed_joint_lump__RL_foot_collision_3'>
-        <pose>-0.002 0 -0.21299999999999999 0 0 0</pose>
-        <geometry>
-          <sphere>
-            <radius>0.021999999999999999</radius>
-          </sphere>
         </geometry>
       </collision>
@@ -943,7 +919,7 @@
         </limit>
         <dynamics>
-          <damping>0.5</damping>
+          <damping>0</damping>
           <spring_reference>0</spring_reference>
-          <spring_stiffness>3</spring_stiffness>
+          <spring_stiffness>0</spring_stiffness>
         </dynamics>
       </axis>
@@ -999,7 +975,7 @@
         </limit>
         <dynamics>
-          <damping>0.5</damping>
+          <damping>0</damping>
           <spring_reference>1.36</spring_reference>
-          <spring_stiffness>3</spring_stiffness>
+          <spring_stiffness>0</spring_stiffness>
         </dynamics>
       </axis>
@@ -1054,7 +1030,7 @@
         </limit>
         <dynamics>
-          <damping>0.5</damping>
+          <damping>0</damping>
           <spring_reference>-2.65</spring_reference>
-          <spring_stiffness>3</spring_stiffness>
+          <spring_stiffness>0</spring_stiffness>
         </dynamics>
       </axis>
@@ -1099,12 +1075,4 @@
             <radius>0.0155</radius>
           </cylinder>
-        </geometry>
-      </collision>
-      <collision name='lower3_fixed_joint_lump__RR_foot_collision_3'>
-        <pose>-0.002 0 -0.21299999999999999 0 0 0</pose>
-        <geometry>
-          <sphere>
-            <radius>0.021999999999999999</radius>
-          </sphere>
         </geometry>
       </collision>
