Commit message: a1 working in sim, Corrected bugs in Underbrush Controller

File: quad_simulator/a1_description/models/a1/urdf/a1.urdf.xacro (robot description, xacro)
@@ -4,5 +4,7 @@
 <!-- |    EDITING THIS FILE BY HAND IS NOT RECOMMENDED                                 | -->
 <!-- =================================================================================== -->
-<robot name="a1_description">
+<robot name="a1_description" xmlns:xacro="http://www.ros.org/wiki/xacro">
+  <xacro:arg name="prefix" default=""/>
+  <xacro:property name="prefix" value="$(arg prefix)"/>
   <material name="black">
     <color rgba="0.0 0.0 0.0 1.0"/>
@@ -64,10 +66,10 @@
         </plugin>
     </gazebo> -->
-  <gazebo>
+  <!-- <gazebo>
     <plugin filename="libgazebo_ros_force.so" name="gazebo_ros_force">
       <bodyName>trunk</bodyName>
       <topicName>/apply_force/trunk</topicName>
     </plugin>
-  </gazebo>
+  </gazebo> -->
   <gazebo reference="imu_link">
     <gravity>true</gravity>
@@ -182,33 +184,4 @@
     </sensor>
   </gazebo>
-  <!-- Visualization of Foot contacts. -->
-  <!-- <gazebo reference="toe0">
-        <visual>
-            <plugin name="drawForcePlugin" filename="libunitreeDrawForcePlugin.so">
-                <topicName>FR_foot_contact</topicName>
-            </plugin>
-        </visual>
-    </gazebo>
-    <gazebo reference="toe1">
-        <visual>
-            <plugin name="drawForcePlugin" filename="libunitreeDrawForcePlugin.so">
-                <topicName>FL_foot_contact</topicName>
-            </plugin>
-        </visual>
-    </gazebo>
-    <gazebo reference="toe2">
-        <visual>
-            <plugin name="drawForcePlugin" filename="libunitreeDrawForcePlugin.so">
-                <topicName>RR_foot_contact</topicName>
-            </plugin>
-        </visual>
-    </gazebo>
-    <gazebo reference="toe3">
-        <visual>
-            <plugin name="drawForcePlugin" filename="libunitreeDrawForcePlugin.so">
-                <topicName>RL_foot_contact</topicName>
-            </plugin>
-        </visual>
-    </gazebo> -->
   <gazebo reference="body">
     <material>Gazebo/Green</material>
@@ -356,5 +329,5 @@
       <origin rpy="0 0 0" xyz="0 0 0"/>
       <geometry>
-        <mesh filename="package://a1_description/meshes/trunk.dae" scale="1 1 1"/>
+        <mesh filename="package://a1_description/models/a1/meshes/trunk.dae" scale="1 1 1"/>
       </geometry>
       <material name="orange"/>
@@ -401,5 +374,5 @@
       <origin rpy="0 0 0" xyz="0 0 0"/>
       <geometry>
-        <mesh filename="package://a1_description/meshes/hip.dae" scale="1 1 1"/>
+        <mesh filename="package://a1_description/models/a1/meshes/hip.dae" scale="1 1 1"/>
       </geometry>
       <material name="orange"/>
@@ -443,5 +416,5 @@
       <origin rpy="0 0 0" xyz="0 0 0"/>
       <geometry>
-        <mesh filename="package://a1_description/meshes/thigh.dae" scale="1 1 1"/>
+        <mesh filename="package://a1_description/models/a1/meshes/thigh.dae" scale="1 1 1"/>
       </geometry>
       <material name="orange"/>
@@ -471,5 +444,5 @@
       <origin rpy="0 0 0" xyz="0 0 0"/>
       <geometry>
-        <mesh filename="package://a1_description/meshes/calf.dae" scale="1 1 1"/>
+        <mesh filename="package://a1_description/models/a1/meshes/calf.dae" scale="1 1 1"/>
       </geometry>
       <material name="orange"/>
@@ -581,5 +554,5 @@
       <origin rpy="0 3.14159265359 0" xyz="0 0 0"/>
       <geometry>
-        <mesh filename="package://a1_description/meshes/hip.dae" scale="1 1 1"/>
+        <mesh filename="package://a1_description/models/a1/meshes/hip.dae" scale="1 1 1"/>
       </geometry>
       <material name="orange"/>
@@ -623,5 +596,5 @@
       <origin rpy="0 0 0" xyz="0 0 0"/>
       <geometry>
-        <mesh filename="package://a1_description/meshes/thigh.dae" scale="1 1 1"/>
+        <mesh filename="package://a1_description/models/a1/meshes/thigh.dae" scale="1 1 1"/>
       </geometry>
       <material name="orange"/>
@@ -651,5 +624,5 @@
       <origin rpy="0 0 0" xyz="0 0 0"/>
       <geometry>
-        <mesh filename="package://a1_description/meshes/calf.dae" scale="1 1 1"/>
+        <mesh filename="package://a1_description/models/a1/meshes/calf.dae" scale="1 1 1"/>
       </geometry>
       <material name="orange"/>
@@ -761,5 +734,5 @@
       <origin rpy="3.14159265359 0 0" xyz="0 0 0"/>
       <geometry>
-        <mesh filename="package://a1_description/meshes/hip.dae" scale="1 1 1"/>
+        <mesh filename="package://a1_description/models/a1/meshes/hip.dae" scale="1 1 1"/>
       </geometry>
       <material name="orange"/>
@@ -803,5 +776,5 @@
       <origin rpy="0 0 0" xyz="0 0 0"/>
       <geometry>
-        <mesh filename="package://a1_description/meshes/thigh_mirror.dae" scale="1 1 1"/>
+        <mesh filename="package://a1_description/models/a1/meshes/thigh_mirror.dae" scale="1 1 1"/>
       </geometry>
       <material name="orange"/>
@@ -831,5 +804,5 @@
       <origin rpy="0 0 0" xyz="0 0 0"/>
       <geometry>
-        <mesh filename="package://a1_description/meshes/calf.dae" scale="1 1 1"/>
+        <mesh filename="package://a1_description/models/a1/meshes/calf.dae" scale="1 1 1"/>
       </geometry>
       <material name="orange"/>
@@ -941,5 +914,5 @@
       <origin rpy="3.14159265359 3.14159265359 0" xyz="0 0 0"/>
       <geometry>
-        <mesh filename="package://a1_description/meshes/hip.dae" scale="1 1 1"/>
+        <mesh filename="package://a1_description/models/a1/meshes/hip.dae" scale="1 1 1"/>
       </geometry>
       <material name="orange"/>
@@ -983,5 +956,5 @@
       <origin rpy="0 0 0" xyz="0 0 0"/>
       <geometry>
-        <mesh filename="package://a1_description/meshes/thigh_mirror.dae" scale="1 1 1"/>
+        <mesh filename="package://a1_description/models/a1/meshes/thigh_mirror.dae" scale="1 1 1"/>
       </geometry>
       <material name="orange"/>
@@ -1011,5 +984,5 @@
       <origin rpy="0 0 0" xyz="0 0 0"/>
       <geometry>
-        <mesh filename="package://a1_description/meshes/calf.dae" scale="1 1 1"/>
+        <mesh filename="package://a1_description/models/a1/meshes/calf.dae" scale="1 1 1"/>
       </geometry>
       <material name="orange"/>
@@ -1144,3 +1117,68 @@
     <preserveFixedJoint>true</preserveFixedJoint>
   </gazebo>
+  <ros2_control name="GazeboSimSystem" type="system">
+    <hardware>
+      <plugin>gz_ros2_control/GazeboSimSystem</plugin>
+    </hardware>
+    <joint name="0">
+      <command_interface name="effort" />
+      <state_interface name="velocity" />
+      <state_interface name="position" />
+    </joint>
+    <joint name="1">
+      <command_interface name="effort" />
+      <state_interface name="velocity" />
+      <state_interface name="position" />
+    </joint>
+    <joint name="2">
+      <command_interface name="effort" />
+      <state_interface name="velocity" />
+      <state_interface name="position" />
+    </joint>
+    <joint name="3">
+      <command_interface name="effort" />
+      <state_interface name="velocity" />
+      <state_interface name="position" />
+    </joint>
+    <joint name="4">
+      <command_interface name="effort" />
+      <state_interface name="velocity" />
+      <state_interface name="position" />
+    </joint>
+    <joint name="5">
+      <command_interface name="effort" />
+      <state_interface name="velocity" />
+      <state_interface name="position" />
+    </joint>
+    <joint name="6">
+      <command_interface name="effort" />
+      <state_interface name="velocity" />
+      <state_interface name="position" />
+    </joint>
+    <joint name="7">
+      <command_interface name="effort" />
+      <state_interface name="velocity" />
+      <state_interface name="position" />
+    </joint>
+    <joint name="8">
+      <command_interface name="effort" />
+      <state_interface name="velocity" />
+      <state_interface name="position" />
+    </joint>
+    <joint name="9">
+      <command_interface name="effort" />
+      <state_interface name="velocity" />
+      <state_interface name="position" />
+    </joint>
+    <joint name="10">
+      <command_interface name="effort" />
+      <state_interface name="velocity" />
+      <state_interface name="position" />
+    </joint>
+    <joint name="11">
+      <command_interface name="effort" />
+      <state_interface name="velocity" />
+      <state_interface name="position" />
+    </joint>
+  </ros2_control>
 </robot>

File: quad_simulator/go2_description/models/go2/urdf/go2.urdf.xacro (robot description, xacro)
@@ -1372,3 +1372,68 @@
     name="front_camera">
   </link>
+  <ros2_control name="GazeboSimSystem" type="system">
+    <hardware>
+      <plugin>gz_ros2_control/GazeboSimSystem</plugin>
+    </hardware>
+    <joint name="0">
+      <command_interface name="effort" />
+      <state_interface name="velocity" />
+      <state_interface name="position" />
+    </joint>
+    <joint name="1">
+      <command_interface name="effort" />
+      <state_interface name="velocity" />
+      <state_interface name="position" />
+    </joint>
+    <joint name="2">
+      <command_interface name="effort" />
+      <state_interface name="velocity" />
+      <state_interface name="position" />
+    </joint>
+    <joint name="3">
+      <command_interface name="effort" />
+      <state_interface name="velocity" />
+      <state_interface name="position" />
+    </joint>
+    <joint name="4">
+      <command_interface name="effort" />
+      <state_interface name="velocity" />
+      <state_interface name="position" />
+    </joint>
+    <joint name="5">
+      <command_interface name="effort" />
+      <state_interface name="velocity" />
+      <state_interface name="position" />
+    </joint>
+    <joint name="6">
+      <command_interface name="effort" />
+      <state_interface name="velocity" />
+      <state_interface name="position" />
+    </joint>
+    <joint name="7">
+      <command_interface name="effort" />
+      <state_interface name="velocity" />
+      <state_interface name="position" />
+    </joint>
+    <joint name="8">
+      <command_interface name="effort" />
+      <state_interface name="velocity" />
+      <state_interface name="position" />
+    </joint>
+    <joint name="9">
+      <command_interface name="effort" />
+      <state_interface name="velocity" />
+      <state_interface name="position" />
+    </joint>
+    <joint name="10">
+      <command_interface name="effort" />
+      <state_interface name="velocity" />
+      <state_interface name="position" />
+    </joint>
+    <joint name="11">
+      <command_interface name="effort" />
+      <state_interface name="velocity" />
+      <state_interface name="position" />
+    </joint>
+  </ros2_control>
 </robot>

Commit message: fix cmu text pose, ready for pr

File: quad_simulator/a1_description/models/a1/urdf/a1.urdf.xacro (robot description, xacro)
@@ -1186,5 +1186,5 @@
       <origin xyz="0 0 0" rpy="0 0 0" />
       <geometry>
-        <mesh filename="package://objects_description/models/cmu_text/meshes/Spirit40_CMU_Text_transformed.stl" scale="1.3 1 1.3" />
+        <mesh filename="package://objects_description/models/cmu_text/meshes/Spirit40_CMU_Text_transformed.stl" scale="0.8 0.5 0.8" />
       </geometry>
     </visual>

File: quad_simulator/go2_description/models/go2/urdf/go2.urdf.xacro (robot description, xacro)
@@ -1441,5 +1441,5 @@
       <origin xyz="0 0 0" rpy="0 0 0" />
       <geometry>
-        <mesh filename="package://objects_description/models/cmu_text/meshes/Spirit40_CMU_Text_transformed.stl" scale="1.3 1 1.3" />
+        <mesh filename="package://objects_description/models/cmu_text/meshes/Spirit40_CMU_Text_transformed.stl" scale="0.8 1 0.8" />
       </geometry>
     </visual>

File: quad_simulator/vision60_description/models/vision60/urdf/vision60.urdf.xacro (robot description, xacro)
@@ -945,5 +945,5 @@
       <origin xyz="0 0 0" rpy="0 0 0" />
       <geometry>
-        <mesh filename="package://objects_description/models/cmu_text/meshes/Spirit40_CMU_Text_transformed.stl" scale="1.3 1 1.3" />
+        <mesh filename="package://objects_description/models/cmu_text/meshes/Spirit40_CMU_Text_transformed.stl" scale="0.8 1 0.8" />
       </geometry>
     </visual>

Commit message: removed commented code and cleaned up robot description files. Removed unnecessary mujoco scene generation and pngs included in copied unitree robot xml description as quad-sdk stores worlds in different location

File: quad_simulator/a1_description/models/a1/urdf/a1.urdf.xacro (robot description, xacro)
@@ -1,3 +1,7 @@
 <?xml version="1.0" encoding="utf-8"?>
+<!-- =================================================================================== -->
+<!-- |    This document was autogenerated by xacro from robot.xacro                    | -->
+<!-- |    EDITING THIS FILE BY HAND IS NOT RECOMMENDED                                 | -->
+<!-- =================================================================================== -->
 <robot
   name="a1">

File: quad_simulator/a2_description/models/a2/urdf/a2.urdf.xacro (robot description, xacro)
@@ -1,13 +1,8 @@
 <?xml version="1.0" encoding="utf-8"?>
+<!-- =================================================================================== -->
+<!-- |    This document was autogenerated by xacro from robot.xacro                    | -->
+<!-- |    EDITING THIS FILE BY HAND IS NOT RECOMMENDED                                 | -->
+<!-- =================================================================================== -->
 <robot name="a2" xmlns:xacro="http://www.ros.org/wiki/xacro">
-  <!-- [CAUTION] uncomment when convert to mujoco -->
-  <!-- <mujoco>
-    <compiler meshdir="../meshes" discardvisual="false" />
-  </mujoco>
-  <link name="world"></link>
-  <joint name="floating_base_joint" type="floating">
-    <parent link="world" />
-    <child link="base_link" />
-  </joint> -->
   <link
     name="base_link">

File: quad_simulator/b2_description/models/b2/urdf/b2.urdf.xacro (robot description, xacro)
@@ -1,6 +1,7 @@
 <?xml version="1.0" encoding="utf-8"?>
-<!-- This URDF was automatically created by SolidWorks to URDF Exporter! Originally created by Stephen Brawner (brawner@gmail.com)
-     Commit Version: 1.6.0-4-g7f85cfe  Build Version: 1.6.7995.38578
-     For more information, please see http://wiki.ros.org/sw_urdf_exporter -->
+<!-- =================================================================================== -->
+<!-- |    This document was autogenerated by xacro from robot.xacro                    | -->
+<!-- |    EDITING THIS FILE BY HAND IS NOT RECOMMENDED                                 | -->
+<!-- =================================================================================== -->
 <robot
   name="b2">
@@ -1269,10 +1270,4 @@
   </joint>
   <link name="upper3_rotor">
-    <!-- <visual>
-      <origin rpy="1.5707963267948966 0 0" xyz="0 0 0"/>
-      <geometry>
-        <cylinder length="0.02" radius="0.05"/>
-      </geometry>
-    </visual> -->
     <collision>
       <origin rpy="1.5707963267948966 0 0" xyz="0 0 0"/>
@@ -1441,27 +1436,4 @@
         izz="1.68E-27" />
     </inertial>
-    <!-- <visual>
-      <origin
-        xyz="0 0 0"
-        rpy="0 0 0" />
-      <geometry>
-        <mesh
-          filename="package://b2_description/models/b2/meshes/f_oc_link.STL" />
-      </geometry>
-      <material
-        name="">
-        <color
-          rgba="1 1 1 1" />
-      </material>
-    </visual>
-    <collision>
-      <origin
-        xyz="0 0 0"
-        rpy="0 0 0" />
-      <geometry>
-        <mesh
-          filename="package://b2_description/models/b2/meshes/f_oc_link.STL" />
-      </geometry>
-    </collision> -->
   </link>
   <joint
@@ -1494,27 +1466,4 @@
         izz="1.68E-22" />
     </inertial>
-    <!-- <visual>
-      <origin
-        xyz="0 0 0"
-        rpy="0 0 0" />
-      <geometry>
-        <mesh
-          filename="package://b2_description/models/b2/meshes/r_oc_link.STL" />
-      </geometry>
-      <material
-        name="">
-        <color
-          rgba="1 1 1 1" />
-      </material>
-    </visual>
-    <collision>
-      <origin
-        xyz="0 0 0"
-        rpy="0 0 0" />
-      <geometry>
-        <mesh
-          filename="package://b2_description/models/b2/meshes/r_oc_link.STL" />
-      </geometry>
-    </collision> -->
   </link>
   <joint

File: quad_simulator/go1_description/models/go1/urdf/go1.urdf.xacro (robot description, xacro)
@@ -31,18 +31,5 @@
   <material name="white">
     <color rgba="1.0 1.0 1.0 1.0"/>
-  </material>
-  <!-- <xacro:include filename="$(find go1_gazebo)/launch/stairs.urdf.xacro"/> -->
-  <!-- <xacro:stairs stairs="15" xpos="0" ypos="0" zpos="0" /> -->
-  <!-- Rotor related joint and link is only for demonstrate location. -->
-  <!-- Actually, the rotor will rotate and the joint is not fixed. Reduction ratio should be considered. -->
-  <!-- Debug mode will hung up the robot, use "true" or "false" to switch it. -->
-  <!-- <xacro:if value="$(arg DEBUG)">
-        <link name="world"/>
-        <joint name="base_static_joint" type="fixed">
-            <origin rpy="0 0 0" xyz="0 0 0"/>
-            <parent link="world"/>
-            <child link="trunk"/>
-        </joint>
-    </xacro:if>  -->
+  </material>S
   <link name="trunk">
     <visual>

File: quad_simulator/go2_description/models/go2/urdf/go2.urdf.xacro (robot description, xacro)
@@ -1,7 +1,7 @@
 <?xml version="1.0" encoding="utf-8"?>
-<!-- This URDF was automatically created by SolidWorks to URDF Exporter! Originally created by
-Stephen Brawner (brawner@gmail.com)
-     Commit Version: 1.6.0-4-g7f85cfe  Build Version: 1.6.7995.38578
-     For more information, please see http://wiki.ros.org/sw_urdf_exporter -->
+<!-- =================================================================================== -->
+<!-- |    This document was autogenerated by xacro from robot.xacro                    | -->
+<!-- |    EDITING THIS FILE BY HAND IS NOT RECOMMENDED                                 | -->
+<!-- =================================================================================== -->
 <robot name="go2" xmlns:xacro="http://www.ros.org/wiki/xacro">
   <link

File: quad_simulator/go2w_description/models/go2w/urdf/go2w.urdf.xacro (robot description, xacro)
@@ -1,7 +1,7 @@
 <?xml version="1.0" encoding="utf-8"?>
-<!-- This URDF was automatically created by SolidWorks to URDF Exporter! Originally created by
-Stephen Brawner (brawner@gmail.com)
-     Commit Version: 1.6.0-4-g7f85cfe  Build Version: 1.6.7995.38578
-     For more information, please see http://wiki.ros.org/sw_urdf_exporter -->
+<!-- =================================================================================== -->
+<!-- |    This document was autogenerated by xacro from robot.xacro                    | -->
+<!-- |    EDITING THIS FILE BY HAND IS NOT RECOMMENDED                                 | -->
+<!-- =================================================================================== -->
 <robot name="go2w" xmlns:xacro="http://www.ros.org/wiki/xacro">
   <link
